File: hardware/boards/key-board-lh/key-board-lh.kicad_sch (KiCad schematic)
At the start: 8 parts, among them J1 12-way

Commit message: Remove the key boards' test pads; SMD pads join the ground pour solid
The owner decided this: a one-off build is probed by hand, so the six
bring-up test pads (TP-CHAIN) come off both key boards. That means their
symbols (with the power symbols and labels stacked on them), the BOM row,
the layout.yaml placements and the silk legend. The bring-up steps now probe
J1's pin tails, with the key-board pin map in the README. carrier.md's
proposed TP-*/LK-* row is marked not fitted, and the main board's open item
is gone.

tools/pcb_route.py pours ground with ZONE_CONNECTION_THT_THERMAL: thermal
spokes on hand-soldered through-hole pads, solid on reflowed SMD pads. Once
the pads were gone, the register's boxed-in ground pin (U1.15) kept tripping
KiCad's starved_thermal.

Key board LH is re-laid out and rendered: 0 check errors, and every net
routes on the first pass. The key-chain simulation and both key boards'
simulations are re-run and pass.

STILL RED: key board RH is not yet re-laid out. That layout search is
running.

Co-Authored-By: Claude Opus 5.5 <noreply@anthropic.com>
Claude-Session: https://claude.ai/code/session_01LmB4muFXnoLprWX4JzuJ5A
Parts:
- removed TP1, TP2, TP3, TP4, TP5, TP6: test pad, TestPoint:TestPoint_Pad_D1.0mm, symbol Connector:TestPoint
Changed lines of the file:
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@@
     (instances (project "key-board-lh" (path "/a2d77fad-366b-59d5-8d08-ccdc7dd94a07" (page "8"))))
   )
-  (symbol (lib_id "Connector:TestPoint") (at 27.94 152.4 0) (unit 1)
-    (in_bom no) (on_board yes) (dnp no)
-    (property "Reference" "TP6" (at 27.94 144.78 90) (effects (font (size 1.27 1.27)) (justify left)))
-    (property "Probe" "3V3" (at 0 0 0) (effects (font (size 1.27 1.27)) hide))
-    (property "Value" "test pad" (at 30.48 144.78 90) (effects (font (size 1.27 1.27)) (justify left)))
-    (property "Footprint" "TestPoint:TestPoint_Pad_D1.0mm" (at 27.94 152.4 0) (effects (font (size 1.27 1.27)) hide))
-    (property "Datasheet" "" (at 27.94 152.4 0) (effects (font (size 1.27 1.27)) hide))
-    (property "Row" "TP-CHAIN" (at 27.94 152.4 0) (effects (font (size 1.27 1.27)) hide))
-    (property "Pins" "1=1" (at 27.94 152.4 0) (effects (font (size 1.27 1.27)) hide))
-    (property "Note" "bring-up test pad: the chain's 3V3 at this board (hardware/boards/key-board-lh/README.md)" (at 27.94 152.4 0) (effects (font (size 1.27 1.27)) hide))
-    (property "Assembly" "none" (at 27.94 152.4 0) (effects (font (size 1.27 1.27)) hide))
-    (pin "1")
-    (instances (project "key-board-lh" (path "/a2d77fad-366b-59d5-8d08-ccdc7dd94a07" (reference "TP6") (unit 1))))
-  )
-  (symbol (lib_id "power:+3V3") (at 27.94 152.4 0) (unit 1)
-    (in_bom yes) (on_board yes) (dnp no)
-    (property "Reference" "#PWR25" (at 27.94 158.75 0) (effects (font (size 1.27 1.27)) hide))
-    (property "Value" "V3V3_CHAIN_LH" (at 27.94 156.21 0) (effects (font (size 1.27 1.27))))
-    (property "Footprint" "" (at 27.94 152.4 0) (effects (font (size 1.27 1.27)) hide))
-    (property "Datasheet" "" (at 27.94 152.4 0) (effects (font (size 1.27 1.27)) hide))
-    (pin "1")
-    (instances (project "key-board-lh" (path "/a2d77fad-366b-59d5-8d08-ccdc7dd94a07" (reference "#PWR25") (unit 1))))
-  )
-  (symbol (lib_id "Connector:TestPoint") (at 38.1 152.4 0) (unit 1)
-    (in_bom no) (on_board yes) (dnp no)
-    (property "Reference" "TP3" (at 38.1 144.78 90) (effects (font (size 1.27 1.27)) (justify left)))
-    (property "Probe" "GND" (at 0 0 0) (effects (font (size 1.27 1.27)) hide))
-    (property "Value" "test pad" (at 40.64 144.78 90) (effects (font (size 1.27 1.27)) (justify left)))
-    (property "Footprint" "TestPoint:TestPoint_Pad_D1.0mm" (at 38.1 152.4 0) (effects (font (size 1.27 1.27)) hide))
-    (property "Datasheet" "" (at 38.1 152.4 0) (effects (font (size 1.27 1.27)) hide))
-    (property "Row" "TP-CHAIN" (at 38.1 152.4 0) (effects (font (size 1.27 1.27)) hide))
-    (property "Pins" "1=1" (at 38.1 152.4 0) (effects (font (size 1.27 1.27)) hide))
-    (property "Note" "bring-up test pad: ground (hardware/boards/key-board-lh/README.md)" (at 38.1 152.4 0) (effects (font (size 1.27 1.27)) hide))
-    (property "Assembly" "none" (at 38.1 152.4 0) (effects (font (size 1.27 1.27)) hide))
-    (pin "1")
-    (instances (project "key-board-lh" (path "/a2d77fad-366b-59d5-8d08-ccdc7dd94a07" (reference "TP3") (unit 1))))
-  )
-  (symbol (lib_id "power:GND") (at 38.1 152.4 0) (unit 1)
-    (in_bom yes) (on_board yes) (dnp no)
-    (property "Reference" "#PWR26" (at 38.1 158.75 0) (effects (font (size 1.27 1.27)) hide))
-    (property "Value" "GND_CHAIN" (at 38.1 156.21 0) (effects (font (size 1.27 1.27))))
-    (property "Footprint" "" (at 38.1 152.4 0) (effects (font (size 1.27 1.27)) hide))
-    (property "Datasheet" "" (at 38.1 152.4 0) (effects (font (size 1.27 1.27)) hide))
-    (pin "1")
-    (instances (project "key-board-lh" (path "/a2d77fad-366b-59d5-8d08-ccdc7dd94a07" (reference "#PWR26") (unit 1))))
-  )
-  (symbol (lib_id "Connector:TestPoint") (at 48.26 152.4 0) (unit 1)
-    (in_bom no) (on_board yes) (dnp no)
-    (property "Reference" "TP4" (at 48.26 144.78 90) (effects (font (size 1.27 1.27)) (justify left)))
-    (property "Probe" "SCK" (at 0 0 0) (effects (font (size 1.27 1.27)) hide))
-    (property "Value" "test pad" (at 50.8 144.78 90) (effects (font (size 1.27 1.27)) (justify left)))
-    (property "Footprint" "TestPoint:TestPoint_Pad_D1.0mm" (at 48.26 152.4 0) (effects (font (size 1.27 1.27)) hide))
-    (property "Datasheet" "" (at 48.26 152.4 0) (effects (font (size 1.27 1.27)) hide))
-    (property "Row" "TP-CHAIN" (at 48.26 152.4 0) (effects (font (size 1.27 1.27)) hide))
-    (property "Pins" "1=1" (at 48.26 152.4 0) (effects (font (size 1.27 1.27)) hide))
-    (property "Note" "bring-up test pad: the chain's clock (hardware/boards/key-board-lh/README.md)" (at 48.26 152.4 0) (effects (font (size 1.27 1.27)) hide))
-    (property "Assembly" "none" (at 48.26 152.4 0) (effects (font (size 1.27 1.27)) hide))
-    (pin "1")
-    (instances (project "key-board-lh" (path "/a2d77fad-366b-59d5-8d08-ccdc7dd94a07" (reference "TP4") (unit 1))))
-  )
-  (label "CHAIN_SCK" (at 48.26 152.4 270) (fields_autoplaced) (effects (font (size 1.27 1.27)) (justify right bottom)))
-  (symbol (lib_id "Connector:TestPoint") (at 58.42 152.4 0) (unit 1)
-    (in_bom no) (on_board yes) (dnp no)
-    (property "Reference" "TP5" (at 58.42 144.78 90) (effects (font (size 1.27 1.27)) (justify left)))
-    (property "Probe" "SH/LD" (at 0 0 0) (effects (font (size 1.27 1.27)) hide))
-    (property "Value" "test pad" (at 60.96 144.78 90) (effects (font (size 1.27 1.27)) (justify left)))
-    (property "Footprint" "TestPoint:TestPoint_Pad_D1.0mm" (at 58.42 152.4 0) (effects (font (size 1.27 1.27)) hide))
-    (property "Datasheet" "" (at 58.42 152.4 0) (effects (font (size 1.27 1.27)) hide))
-    (property "Row" "TP-CHAIN" (at 58.42 152.4 0) (effects (font (size 1.27 1.27)) hide))
-    (property "Pins" "1=1" (at 58.42 152.4 0) (effects (font (size 1.27 1.27)) hide))
-    (property "Note" "bring-up test pad: the chain's shift/load (hardware/boards/key-board-lh/README.md)" (at 58.42 152.4 0) (effects (font (size 1.27 1.27)) hide))
-    (property "Assembly" "none" (at 58.42 152.4 0) (effects (font (size 1.27 1.27)) hide))
-    (pin "1")
-    (instances (project "key-board-lh" (path "/a2d77fad-366b-59d5-8d08-ccdc7dd94a07" (reference "TP5") (unit 1))))
-  )
-  (label "CHAIN_SHLD" (at 58.42 152.4 270) (fields_autoplaced) (effects (font (size 1.27 1.27)) (justify right bottom)))
-  (symbol (lib_id "Connector:TestPoint") (at 68.58 152.4 0) (unit 1)
-    (in_bom no) (on_board yes) (dnp no)
-    (property "Reference" "TP1" (at 68.58 144.78 90) (effects (font (size 1.27 1.27)) (justify left)))
-    (property "Probe" "QH" (at 0 0 0) (effects (font (size 1.27 1.27)) hide))
-    (property "Value" "test pad" (at 71.12 144.78 90) (effects (font (size 1.27 1.27)) (justify left)))
-    (property "Footprint" "TestPoint:TestPoint_Pad_D1.0mm" (at 68.58 152.4 0) (effects (font (size 1.27 1.27)) hide))
-    (property "Datasheet" "" (at 68.58 152.4 0) (effects (font (size 1.27 1.27)) hide))
-    (property "Row" "TP-CHAIN" (at 68.58 152.4 0) (effects (font (size 1.27 1.27)) hide))
-    (property "Pins" "1=1" (at 68.58 152.4 0) (effects (font (size 1.27 1.27)) hide))
-    (property "Note" "bring-up test pad: this board's serial output (QH) (hardware/boards/key-board-lh/README.md)" (at 68.58 152.4 0) (effects (font (size 1.27 1.27)) hide))
-    (property "Assembly" "none" (at 68.58 152.4 0) (effects (font (size 1.27 1.27)) hide))
-    (pin "1")
-    (instances (project "key-board-lh" (path "/a2d77fad-366b-59d5-8d08-ccdc7dd94a07" (reference "TP1") (unit 1))))
-  )
-  (label "HOP_LH_LT" (at 68.58 152.4 270) (fields_autoplaced) (effects (font (size 1.27 1.27)) (justify right bottom)))
-  (symbol (lib_id "Connector:TestPoint") (at 78.74 152.4 0) (unit 1)
-    (in_bom no) (on_board yes) (dnp no)
-    (property "Reference" "TP2" (at 78.74 144.78 90) (effects (font (size 1.27 1.27)) (justify left)))
-    (property "Probe" "SER" (at 0 0 0) (effects (font (size 1.27 1.27)) hide))
-    (property "Value" "test pad" (at 81.28 144.78 90) (effects (font (size 1.27 1.27)) (justify left)))
-    (property "Footprint" "TestPoint:TestPoint_Pad_D1.0mm" (at 78.74 152.4 0) (effects (font (size 1.27 1.27)) hide))
-    (property "Datasheet" "" (at 78.74 152.4 0) (effects (font (size 1.27 1.27)) hide))
-    (property "Row" "TP-CHAIN" (at 78.74 152.4 0) (effects (font (size 1.27 1.27)) hide))
-    (property "Pins" "1=1" (at 78.74 152.4 0) (effects (font (size 1.27 1.27)) hide))
-    (property "Note" "bring-up test pad: this board's serial input (SER), driven by the next board up the chain - tie it to TP-GND or TP-3V3 on the bench, where nothing drives it (hardware/boards/key-board-lh/README.md)" (at 78.74 152.4 0) (effects (font (size 1.27 1.27)) hide))
-    (property "Assembly" "none" (at 78.74 152.4 0) (effects (font (size 1.27 1.27)) hide))
-    (pin "1")
-    (instances (project "key-board-lh" (path "/a2d77fad-366b-59d5-8d08-ccdc7dd94a07" (reference "TP2") (unit 1))))
-  )
-  (label "CHAIN_SER_LH" (at 78.74 152.4 270) (fields_autoplaced) (effects (font (size 1.27 1.27)) (justify right bottom)))
   (symbol (lib_id "Device:C") (at 93.98 152.4 0) (unit 1)
     (in_bom yes) (on_board yes) (dnp no)
