File: hardware/boards/key-board-rh/key-board-rh.kicad_sch (KiCad schematic)
At the start: 8 parts

Commit message: Key boards: numeric references on every part, silkscreen readable with parts fitted
Owner, 2026-09-28: 'resistors should all be R1, R2, R3 etc. Everything should
be properly numeric and labeled on the silk screen', and 'make sure silk
screens will still be visible even when components are placed'.

- Sheets: the key boards' instance references renumbered (SWn, R(2n-1)
  series, R(2n) pull-up, Cn per key; then the free pull-up, decoupler,
  bulk cap, U1, J1, TP1-TP6). Circuit-level row names are unchanged; each
  part's BOM row stays its Row field. Test pads carry a Probe field.
- Tools find parts by row and sheet, not by name: pcb.py ref_of (placement,
  the network T, check_cad), kicad.py's allocation and chain checks. The
  allocation check now fails a board with no register instead of passing it
  by finding none. The board export records each part's sheet.
- Silkscreen: every part's reference, sized by its real width in KiCad's
  font (text_w; the old per-character guess ran 15-35 % short); network
  resistors' references read along the parts; switches 'SW1 LH1'; a
  test-pad legend (TP1 QH ...). check_silk now fails any placed mark under a
  part's courtyard, proven on a scratch copy on both sides.
- KS-33 footprint courtyard +-7.0 -> +-7.75: the switch is 15 x 15, and the
  old courtyard let labels sit under its housing.
- Straight-down plan renders of both sides (pcb-plan-top/-bottom.png).
- LH board re-laid out: check 0 errors; README and tooling.md follow.

Co-Authored-By: Claude Opus 5.5 <noreply@anthropic.com>
Claude-Session: https://claude.ai/code/session_01LmB4muFXnoLprWX4JzuJ5A
Parts:
- TP1: renamed from TP-QH-RH; Probe (none) -> QH
- TP2: renamed from TP-SER-RH; Probe (none) -> SER
- TP3: renamed from TP-GND-RH; Probe (none) -> GND
- TP4: renamed from TP-SCK-RH; Probe (none) -> SCK
- TP5: renamed from TP-SHLD-RH; Probe (none) -> SH/LD
- TP6: renamed from TP-3V3-RH; Probe (none) -> 3V3
- renumbered C-BULK-CHAIN-RH to C8, J-CHAIN to J1
Changed lines of the file:
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@@
   (symbol (lib_id "Connector_Generic:Conn_01x12") (at 45.72 101.6 0) (unit 1)
     (in_bom yes) (on_board yes) (dnp no)
-    (property "Reference" "J-CHAIN" (at 45.72 86.36 0) (effects (font (size 1.27 1.27))))
+    (property "Reference" "J1" (at 45.72 86.36 0) (effects (font (size 1.27 1.27))))
     (property "Value" "12-way" (at 45.72 119.38 0) (effects (font (size 1.27 1.27))))
     (property "Footprint" "woody:IDC-Header_2x06_P1.27mm_Samtec_SHF_Horizontal" (at 45.72 101.6 0) (effects (font (size 1.27 1.27)) hide))
@@
     (pin "8")
     (pin "9")
-    (instances (project "key-board-rh" (path "/0d798814-7e94-52b0-a143-b50dd4dde890" (reference "J-CHAIN") (unit 1))))
+    (instances (project "key-board-rh" (path "/0d798814-7e94-52b0-a143-b50dd4dde890" (reference "J1") (unit 1))))
   )
   (wire (pts (xy 40.64 114.30) (xy 38.1 114.30)) (stroke (width 0) (type default)))
@@
   (symbol (lib_id "Connector:TestPoint") (at 27.94 152.4 0) (unit 1)
     (in_bom no) (on_board yes) (dnp no)
-    (property "Reference" "TP-3V3-RH" (at 27.94 144.78 90) (effects (font (size 1.27 1.27)) (justify left)))
+    (property "Reference" "TP6" (at 27.94 144.78 90) (effects (font (size 1.27 1.27)) (justify left)))
+    (property "Probe" "3V3" (at 0 0 0) (effects (font (size 1.27 1.27)) hide))
     (property "Value" "test pad" (at 30.48 144.78 90) (effects (font (size 1.27 1.27)) (justify left)))
     (property "Footprint" "TestPoint:TestPoint_Pad_D1.0mm" (at 27.94 152.4 0) (effects (font (size 1.27 1.27)) hide))
@@
     (property "Assembly" "none" (at 27.94 152.4 0) (effects (font (size 1.27 1.27)) hide))
     (pin "1")
-    (instances (project "key-board-rh" (path "/0d798814-7e94-52b0-a143-b50dd4dde890" (reference "TP-3V3-RH") (unit 1))))
+    (instances (project "key-board-rh" (path "/0d798814-7e94-52b0-a143-b50dd4dde890" (reference "TP6") (unit 1))))
   )
   (symbol (lib_id "power:+3V3") (at 27.94 152.4 0) (unit 1)
@@
   (symbol (lib_id "Connector:TestPoint") (at 38.1 152.4 0) (unit 1)
     (in_bom no) (on_board yes) (dnp no)
-    (property "Reference" "TP-GND-RH" (at 38.1 144.78 90) (effects (font (size 1.27 1.27)) (justify left)))
+    (property "Reference" "TP3" (at 38.1 144.78 90) (effects (font (size 1.27 1.27)) (justify left)))
+    (property "Probe" "GND" (at 0 0 0) (effects (font (size 1.27 1.27)) hide))
     (property "Value" "test pad" (at 40.64 144.78 90) (effects (font (size 1.27 1.27)) (justify left)))
     (property "Footprint" "TestPoint:TestPoint_Pad_D1.0mm" (at 38.1 152.4 0) (effects (font (size 1.27 1.27)) hide))
@@
     (property "Assembly" "none" (at 38.1 152.4 0) (effects (font (size 1.27 1.27)) hide))
     (pin "1")
-    (instances (project "key-board-rh" (path "/0d798814-7e94-52b0-a143-b50dd4dde890" (reference "TP-GND-RH") (unit 1))))
+    (instances (project "key-board-rh" (path "/0d798814-7e94-52b0-a143-b50dd4dde890" (reference "TP3") (unit 1))))
   )
   (symbol (lib_id "power:GND") (at 38.1 152.4 0) (unit 1)
@@
   (symbol (lib_id "Connector:TestPoint") (at 48.26 152.4 0) (unit 1)
     (in_bom no) (on_board yes) (dnp no)
-    (property "Reference" "TP-SCK-RH" (at 48.26 144.78 90) (effects (font (size 1.27 1.27)) (justify left)))
+    (property "Reference" "TP4" (at 48.26 144.78 90) (effects (font (size 1.27 1.27)) (justify left)))
+    (property "Probe" "SCK" (at 0 0 0) (effects (font (size 1.27 1.27)) hide))
     (property "Value" "test pad" (at 50.8 144.78 90) (effects (font (size 1.27 1.27)) (justify left)))
     (property "Footprint" "TestPoint:TestPoint_Pad_D1.0mm" (at 48.26 152.4 0) (effects (font (size 1.27 1.27)) hide))
@@
     (property "Assembly" "none" (at 48.26 152.4 0) (effects (font (size 1.27 1.27)) hide))
     (pin "1")
-    (instances (project "key-board-rh" (path "/0d798814-7e94-52b0-a143-b50dd4dde890" (reference "TP-SCK-RH") (unit 1))))
+    (instances (project "key-board-rh" (path "/0d798814-7e94-52b0-a143-b50dd4dde890" (reference "TP4") (unit 1))))
   )
   (label "CHAIN_SCK" (at 48.26 152.4 270) (fields_autoplaced) (effects (font (size 1.27 1.27)) (justify right bottom)))
   (symbol (lib_id "Connector:TestPoint") (at 58.42 152.4 0) (unit 1)
     (in_bom no) (on_board yes) (dnp no)
-    (property "Reference" "TP-SHLD-RH" (at 58.42 144.78 90) (effects (font (size 1.27 1.27)) (justify left)))
+    (property "Reference" "TP5" (at 58.42 144.78 90) (effects (font (size 1.27 1.27)) (justify left)))
+    (property "Probe" "SH/LD" (at 0 0 0) (effects (font (size 1.27 1.27)) hide))
     (property "Value" "test pad" (at 60.96 144.78 90) (effects (font (size 1.27 1.27)) (justify left)))
     (property "Footprint" "TestPoint:TestPoint_Pad_D1.0mm" (at 58.42 152.4 0) (effects (font (size 1.27 1.27)) hide))
@@
     (property "Assembly" "none" (at 58.42 152.4 0) (effects (font (size 1.27 1.27)) hide))
     (pin "1")
-    (instances (project "key-board-rh" (path "/0d798814-7e94-52b0-a143-b50dd4dde890" (reference "TP-SHLD-RH") (unit 1))))
+    (instances (project "key-board-rh" (path "/0d798814-7e94-52b0-a143-b50dd4dde890" (reference "TP5") (unit 1))))
   )
   (label "CHAIN_SHLD" (at 58.42 152.4 270) (fields_autoplaced) (effects (font (size 1.27 1.27)) (justify right bottom)))
   (symbol (lib_id "Connector:TestPoint") (at 68.58 152.4 0) (unit 1)
     (in_bom no) (on_board yes) (dnp no)
-    (property "Reference" "TP-QH-RH" (at 68.58 144.78 90) (effects (font (size 1.27 1.27)) (justify left)))
+    (property "Reference" "TP1" (at 68.58 144.78 90) (effects (font (size 1.27 1.27)) (justify left)))
+    (property "Probe" "QH" (at 0 0 0) (effects (font (size 1.27 1.27)) hide))
     (property "Value" "test pad" (at 71.12 144.78 90) (effects (font (size 1.27 1.27)) (justify left)))
     (property "Footprint" "TestPoint:TestPoint_Pad_D1.0mm" (at 68.58 152.4 0) (effects (font (size 1.27 1.27)) hide))
@@
     (property "Assembly" "none" (at 68.58 152.4 0) (effects (font (size 1.27 1.27)) hide))
     (pin "1")
-    (instances (project "key-board-rh" (path "/0d798814-7e94-52b0-a143-b50dd4dde890" (reference "TP-QH-RH") (unit 1))))
+    (instances (project "key-board-rh" (path "/0d798814-7e94-52b0-a143-b50dd4dde890" (reference "TP1") (unit 1))))
   )
   (label "HOP_RH_RT" (at 68.58 152.4 270) (fields_autoplaced) (effects (font (size 1.27 1.27)) (justify right bottom)))
   (symbol (lib_id "Connector:TestPoint") (at 78.74 152.4 0) (unit 1)
     (in_bom no) (on_board yes) (dnp no)
-    (property "Reference" "TP-SER-RH" (at 78.74 144.78 90) (effects (font (size 1.27 1.27)) (justify left)))
+    (property "Reference" "TP2" (at 78.74 144.78 90) (effects (font (size 1.27 1.27)) (justify left)))
+    (property "Probe" "SER" (at 0 0 0) (effects (font (size 1.27 1.27)) hide))
     (property "Value" "test pad" (at 81.28 144.78 90) (effects (font (size 1.27 1.27)) (justify left)))
     (property "Footprint" "TestPoint:TestPoint_Pad_D1.0mm" (at 78.74 152.4 0) (effects (font (size 1.27 1.27)) hide))
@@
     (property "Assembly" "none" (at 78.74 152.4 0) (effects (font (size 1.27 1.27)) hide))
     (pin "1")
-    (instances (project "key-board-rh" (path "/0d798814-7e94-52b0-a143-b50dd4dde890" (reference "TP-SER-RH") (unit 1))))
+    (instances (project "key-board-rh" (path "/0d798814-7e94-52b0-a143-b50dd4dde890" (reference "TP2") (unit 1))))
   )
   (label "HOP_LT_RH" (at 78.74 152.4 270) (fields_autoplaced) (effects (font (size 1.27 1.27)) (justify right bottom)))
   (symbol (lib_id "Device:C") (at 93.98 152.4 0) (unit 1)
     (in_bom no) (on_board yes) (dnp yes)
-    (property "Reference" "C-BULK-CHAIN-RH" (at 96.52000000000001 151.13 0) (effects (font (size 1.27 1.27)) (justify left)))
+    (property "Reference" "C8" (at 96.52000000000001 151.13 0) (effects (font (size 1.27 1.27)) (justify left)))
     (property "Value" "10uF DNP" (at 96.52000000000001 153.67000000000002 0) (effects (font (size 1.27 1.27)) (justify left)))
     (property "Footprint" "Capacitor_SMD:C_0805_2012Metric" (at 93.98 152.4 0) (effects (font (size 1.27 1.27)) hide))
@@
     (pin "1")
     (pin "2")
-    (instances (project "key-board-rh" (path "/0d798814-7e94-52b0-a143-b50dd4dde890" (reference "C-BULK-CHAIN-RH") (unit 1))))
+    (instances (project "key-board-rh" (path "/0d798814-7e94-52b0-a143-b50dd4dde890" (reference "C8") (unit 1))))
   )
   (symbol (lib_id "power:+3V3") (at 93.98 148.59 0) (unit 1)

Commit message: Fit C-BULK-CHAIN on both key boards instead of leaving it empty
The 10uF reservoir on each key board's 3V3 (C7 on the left-hand board,
C8 on the right) was a do-not-fit footprint, to be fitted at bring-up
only if the rail rang. It costs cents, so it is now a fitted,
machine-placed part (owner, 2026-09-28): Samsung CL21A106KAYNNNE, LCSC
C15850, a JLC Basic part.

The key-chain simulation now calls the fitted board "as ordered":
- rail-as-ordered: 5 mV peak to peak on the key board's 3V3.
- rail-impedance-as-ordered: a 2.2 ohm peak.
- The new rail-without-bulk holds the same limits with it left off
  (72 mV). A board built without the part still works; the part makes
  the rail quieter.
- rail-impedance-without-bulk (176-217 ohm peak) replaces
  rail-impedance-with-bulk; edge-droop-as-ordered is renamed
  edge-droop-decoupler-alone, since it models the decoupler with the
  bulk capacitor off.
Both boards' own simulations now include the part.

The sheets, the BOM row, the loom page, cluster-boards.md and both
board READMEs no longer treat it as optional. Both boards are re-laid
out (no DNP mark), checked at 0 errors and re-rendered, and the part
is in each board's JLC BOM and CPL.

Co-Authored-By: Claude Opus 5.5 <noreply@anthropic.com>
Claude-Session: https://claude.ai/code/session_01LmB4muFXnoLprWX4JzuJ5A
Parts:
- C8: value 10uF DNP -> 10uF; Assembly none -> machine; LCSC (none) -> C15850; MPN (none) -> CL21A106KAYNNNE; Manufacturer (none) -> Samsung; Note DO NOT FIT unless the rail rings: FB-CHAIN and C-DECOUPLE-1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 -> the rail's reservoir, beside J-CHAIN's 3V3 pin: FB-CHAIN an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; now fitted; now in the parts list
Changed lines of the file:
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@@
   (label "HOP_LT_RH" (at 78.74 152.4 270) (fields_autoplaced) (effects (font (size 1.27 1.27)) (justify right bottom)))
   (symbol (lib_id "Device:C") (at 93.98 152.4 0) (unit 1)
-    (in_bom no) (on_board yes) (dnp yes)
+    (in_bom yes) (on_board yes) (dnp no)
     (property "Reference" "C8" (at 96.52000000000001 151.13 0) (effects (font (size 1.27 1.27)) (justify left)))
-    (property "Value" "10uF DNP" (at 96.52000000000001 153.67000000000002 0) (effects (font (size 1.27 1.27)) (justify left)))
+    (property "Value" "10uF" (at 96.52000000000001 153.67000000000002 0) (effects (font (size 1.27 1.27)) (justify left)))
     (property "Footprint" "Capacitor_SMD:C_0805_2012Metric" (at 93.98 152.4 0) (effects (font (size 1.27 1.27)) hide))
     (property "Datasheet" "" (at 93.98 152.4 0) (effects (font (size 1.27 1.27)) hide))
     (property "Row" "C-BULK-CHAIN" (at 93.98 152.4 0) (effects (font (size 1.27 1.27)) hide))
     (property "Pins" "1=1 2=2" (at 93.98 152.4 0) (effects (font (size 1.27 1.27)) hide))
-    (property "Note" "DO NOT FIT unless the rail rings: FB-CHAIN and C-DECOUPLE-165 make an LC near 0.5 MHz, half the chain clock. Scope this board's VCC while shifting at bring-up; if it rings, fit a 10uF X5R 0805 here, whose ESR damps it (FB-CHAIN row, key-chain-loom/bom.csv)" (at 93.98 152.4 0) (effects (font (size 1.27 1.27)) hide))
-    (property "Assembly" "none" (at 93.98 152.4 0) (effects (font (size 1.27 1.27)) hide))
+    (property "Note" "the rail's reservoir, beside J-CHAIN's 3V3 pin: FB-CHAIN and C-DECOUPLE-165 make a lightly damped LC near 0.5 MHz, half the chain clock, and this 10uF's ESR damps it (C-BULK-CHAIN row, key-chain-loom/bom.csv; the simulation, key-chain-loom/sim, rail-as-ordered)" (at 93.98 152.4 0) (effects (font (size 1.27 1.27)) hide))
+    (property "Manufacturer" "Samsung" (at 93.98 152.4 0) (effects (font (size 1.27 1.27)) hide))
+    (property "MPN" "CL21A106KAYNNNE" (at 93.98 152.4 0) (effects (font (size 1.27 1.27)) hide))
+    (property "LCSC" "C15850" (at 93.98 152.4 0) (effects (font (size 1.27 1.27)) hide))
+    (property "Assembly" "machine" (at 93.98 152.4 0) (effects (font (size 1.27 1.27)) hide))
     (pin "1")
     (pin "2")
