File: hardware/cluster/key-marker-and-bits/key-marker-and-bits.kicad_sch (KiCad schematic)
At the start: 1 part

Commit message: First PCB: the left-hand key board, placed from the body CAD and routed
- tools/pcb.py: a board's first layout from its KiCad sheets (netlist,
  footprints) and the body CAD's new exports (key-board outline DXF,
  switch and ribbon-connector positions); then the .kicad_pcb is source.
  check = KiCad DRC with schematic parity + switches where the CAD puts
  them; render = 3D both sides, 2D copper, and fab/ (Gerbers, drill,
  placement), ledgered in hardware/SHEETS.csv. tools/kicad.py check runs it.
- tools/pcb_route.py: a small two-layer grid router for simple boards;
  ground routed as a net plus pours and stitching vias.
- key-board-lh: 24 parts, all nets routed; KiCad DRC 0 errors, schematic
  parity clean (one stock-footprint silkscreen warning). Tested: a switch
  moved 1 mm fails the check.
- Footprints on the sheets; hardware/lib/woody.pretty holds the KS-33
  footprint (marbastlib, banked) with Gateron's STEP lifted by
  switch.pcb_below_seat. J-CHAIN's stand-in is Molex 200528-0120.
- Findings, recorded in tooling.md §4 and DESIGN.md: the ribbon connector
  needs 6.7 mm, the CAD envelope is 5.5; KS-33 pins show only ~0.1 mm
  below a 1.6 mm board (1.2 mm would leave ~0.5).
- setup-env.sh installs footprints, rsvg, shapely and repairs an empty
  global fp-lib-table.

Co-Authored-By: Claude Opus 5.5 <noreply@anthropic.com>
Claude-Session: https://claude.ai/code/session_01LmB4muFXnoLprWX4JzuJ5A
Parts:
- R-KEY-PU-FREE: footprint (none) -> Resistor_SMD:R_0805_2012Metric
Changed lines of the file:
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@@
     (property "Reference" "R-KEY-PU-FREE" (at 104.14 100.33 0) (effects (font (size 1.27 1.27)) (justify left)))
     (property "Value" "2k2 1%" (at 104.14 102.87 0) (effects (font (size 1.27 1.27)) (justify left)))
-    (property "Footprint" "" (at 100.33 101.6 0) (effects (font (size 1.27 1.27)) hide))
+    (property "Footprint" "Resistor_SMD:R_0805_2012Metric" (at 100.33 101.6 0) (effects (font (size 1.27 1.27)) hide))
     (property "Datasheet" "" (at 101.6 101.6 0) (effects (font (size 1.27 1.27)) hide))
     (property "Row" "R-KEY-PU" (at 101.6 101.6 0) (effects (font (size 1.27 1.27)) hide))

Commit message: LH key board as the worked example: orderable, labelled, testable
- Samtec full prints banked (SHF header, FFSD cable); the header's true
  dimensions replace the catalogue estimates (body.yaml boards.chain_*), and
  the cable is ordered -RN2 (notch reversed on the key-board end): both
  sockets' cables leave downward, the ribbon runs flat, and key-board pin =
  13 - main-board pin. The same-day 12-n/14-n map was wrong and is undone in
  the sheets, the interface netlist and the docs (history in notes.md).
- Model: the hairpin's legs follow the cable's real exit - the main board's
  on the board, clear of the thumb switches' poles; 0 DRC FAILs, 0 clashes.
- Sheets: Manufacturer/MPN/LCSC/Assembly fields from JLC's parts API (JLC
  and LCSC pages banked in datasheets/fab and the manifest); five bring-up
  test pads per key board (TP-CHAIN, copper only).
- pcb.py: JLC's limits in the DRC (layout.yaml fab:), which grew the vias
  and J-CHAIN's pads to the 0.18 mm ring; HASL lead-free in the stackup and
  Gerber job; a generated parts-side silkscreen; the JLC BOM, CPL and
  hand-assembly list in fab/, ledgered against board and sheets.
- Router: a real rip-up (blockers removed too); plated holes no longer wall
  off their own pads.
- hardware/boards/key-board-lh/README.md: sources, ordering, hand assembly,
  bring-up, open items. tooling.md and lib README follow.
All checks pass: CAD, DRC (0/0), KiCad, staleness, BOM, netlist, datasheets.

Co-Authored-By: Claude Opus 5.5 <noreply@anthropic.com>
Claude-Session: https://claude.ai/code/session_01LmB4muFXnoLprWX4JzuJ5A
Parts:
- R-KEY-PU-FREE: Assembly (none) -> machine; LCSC (none) -> C17520; MPN (none) -> 0805W8F2201T5E; Manufacturer (none) -> UNI-ROYAL
Changed lines of the file:
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@@
     (property "Pins" "1=1 2=2" (at 101.6 101.6 0) (effects (font (size 1.27 1.27)) hide))
     (property "Note" "One per FREE bit. The same part the key networks use, and the reason 'free' bits are not free: each one costs the same static draw as a key" (at 101.6 101.6 0) (effects (font (size 1.27 1.27)) hide))
+    (property "Manufacturer" "UNI-ROYAL" (at 101.6 101.6 0) (effects (font (size 1.27 1.27)) hide))
+    (property "MPN" "0805W8F2201T5E" (at 101.6 101.6 0) (effects (font (size 1.27 1.27)) hide))
+    (property "LCSC" "C17520" (at 101.6 101.6 0) (effects (font (size 1.27 1.27)) hide))
+    (property "Assembly" "machine" (at 101.6 101.6 0) (effects (font (size 1.27 1.27)) hide))
     (pin "1")
     (pin "2")

Commit message: WIP: layout-side fixes (networks as T, via-in-pad, segment merge, silk, stackup, TP-SER, drills)
Co-Authored-By: Claude Opus 5.5 <noreply@anthropic.com>
Claude-Session: https://claude.ai/code/session_01LmB4muFXnoLprWX4JzuJ5A
Parts:
- R-KEY-PU-FREE: Note One per FREE bit. The same part the key networks use, and t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 -> One per FREE bit, holding its unswitched input high. The sa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
Changed lines of the file:
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@@
     (property "Row" "R-KEY-PU" (at 101.6 101.6 0) (effects (font (size 1.27 1.27)) hide))
     (property "Pins" "1=1 2=2" (at 101.6 101.6 0) (effects (font (size 1.27 1.27)) hide))
-    (property "Note" "One per FREE bit. The same part the key networks use, and the reason 'free' bits are not free: each one costs the same static draw as a key" (at 101.6 101.6 0) (effects (font (size 1.27 1.27)) hide))
+    (property "Note" "One per FREE bit, holding its unswitched input high. The same part the key networks use; with no switch on the bit it draws only the input's leakage, so what a free bit costs is a part and a placement, not current" (at 101.6 101.6 0) (effects (font (size 1.27 1.27)) hide))
     (property "Manufacturer" "UNI-ROYAL" (at 101.6 101.6 0) (effects (font (size 1.27 1.27)) hide))
     (property "MPN" "0805W8F2201T5E" (at 101.6 101.6 0) (effects (font (size 1.27 1.27)) hide))
