File: hardware/cluster/key-switch-network/key-switch-network.kicad_sch (KiCad schematic)
At the start: 4 parts, among them SW1-n KS-33

Commit message: First PCB: the left-hand key board, placed from the body CAD and routed
- tools/pcb.py: a board's first layout from its KiCad sheets (netlist,
  footprints) and the body CAD's new exports (key-board outline DXF,
  switch and ribbon-connector positions); then the .kicad_pcb is source.
  check = KiCad DRC with schematic parity + switches where the CAD puts
  them; render = 3D both sides, 2D copper, and fab/ (Gerbers, drill,
  placement), ledgered in hardware/SHEETS.csv. tools/kicad.py check runs it.
- tools/pcb_route.py: a small two-layer grid router for simple boards;
  ground routed as a net plus pours and stitching vias.
- key-board-lh: 24 parts, all nets routed; KiCad DRC 0 errors, schematic
  parity clean (one stock-footprint silkscreen warning). Tested: a switch
  moved 1 mm fails the check.
- Footprints on the sheets; hardware/lib/woody.pretty holds the KS-33
  footprint (marbastlib, banked) with Gateron's STEP lifted by
  switch.pcb_below_seat. J-CHAIN's stand-in is Molex 200528-0120.
- Findings, recorded in tooling.md §4 and DESIGN.md: the ribbon connector
  needs 6.7 mm, the CAD envelope is 5.5; KS-33 pins show only ~0.1 mm
  below a 1.6 mm board (1.2 mm would leave ~0.5).
- setup-env.sh installs footprints, rsvg, shapely and repairs an empty
  global fp-lib-table.

Co-Authored-By: Claude Opus 5.5 <noreply@anthropic.com>
Claude-Session: https://claude.ai/code/session_01LmB4muFXnoLprWX4JzuJ5A
Parts:
- C-KEY: footprint (none) -> Capacitor_SMD:C_0805_2012Metric
- R-KEY-PU, R-KEY-SER: footprint (none) -> Resistor_SMD:R_0805_2012Metric
- SW1-n: footprint (none) -> woody:SW_Gateron_KS33_1u
Changed lines of the file:
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@@
     (property "Reference" "R-KEY-PU" (at 104.14 90.17 0) (effects (font (size 1.27 1.27)) (justify left)))
     (property "Value" "2k2 1%" (at 104.14 92.71 0) (effects (font (size 1.27 1.27)) (justify left)))
-    (property "Footprint" "" (at 100.33 91.44 0) (effects (font (size 1.27 1.27)) hide))
+    (property "Footprint" "Resistor_SMD:R_0805_2012Metric" (at 100.33 91.44 0) (effects (font (size 1.27 1.27)) hide))
     (property "Datasheet" "" (at 101.6 91.44 0) (effects (font (size 1.27 1.27)) hide))
     (property "Row" "R-KEY-PU" (at 101.6 91.44 0) (effects (font (size 1.27 1.27)) hide))
@@
     (property "Reference" "C-KEY" (at 104.14 110.49 0) (effects (font (size 1.27 1.27)) (justify left)))
     (property "Value" "47nF" (at 104.14 113.03 0) (effects (font (size 1.27 1.27)) (justify left)))
-    (property "Footprint" "" (at 102.87 115.57 0) (effects (font (size 1.27 1.27)) hide))
+    (property "Footprint" "Capacitor_SMD:C_0805_2012Metric" (at 102.87 115.57 0) (effects (font (size 1.27 1.27)) hide))
     (property "Datasheet" "" (at 101.6 111.76 0) (effects (font (size 1.27 1.27)) hide))
     (property "Row" "C-KEY" (at 101.6 111.76 0) (effects (font (size 1.27 1.27)) hide))
@@
     (property "Reference" "R-KEY-SER" (at 109.22 99.06 90) (effects (font (size 1.27 1.27))))
     (property "Value" "100R 1%" (at 109.22 104.14 90) (effects (font (size 1.27 1.27))))
-    (property "Footprint" "" (at 109.22 102.87 0) (effects (font (size 1.27 1.27)) hide))
+    (property "Footprint" "Resistor_SMD:R_0805_2012Metric" (at 109.22 102.87 0) (effects (font (size 1.27 1.27)) hide))
     (property "Datasheet" "" (at 109.22 101.6 0) (effects (font (size 1.27 1.27)) hide))
     (property "Row" "R-KEY-SER" (at 109.22 101.6 0) (effects (font (size 1.27 1.27)) hide))
@@
     (property "Reference" "SW1-n" (at 123.19 107.95 270) (effects (font (size 1.27 1.27)) (justify right)))
     (property "Value" "KS-33" (at 123.19 110.49 270) (effects (font (size 1.27 1.27)) (justify right)))
-    (property "Footprint" "" (at 125.73 109.22 0) (effects (font (size 1.27 1.27)) hide))
+    (property "Footprint" "woody:SW_Gateron_KS33_1u" (at 125.73 109.22 0) (effects (font (size 1.27 1.27)) hide))
     (property "Datasheet" "" (at 125.73 109.22 0) (effects (font (size 1.27 1.27)) hide))
     (property "Row" "SW1-n" (at 120.65 109.22 0) (effects (font (size 1.27 1.27)) hide))

Commit message: LH key board as the worked example: orderable, labelled, testable
- Samtec full prints banked (SHF header, FFSD cable); the header's true
  dimensions replace the catalogue estimates (body.yaml boards.chain_*), and
  the cable is ordered -RN2 (notch reversed on the key-board end): both
  sockets' cables leave downward, the ribbon runs flat, and key-board pin =
  13 - main-board pin. The same-day 12-n/14-n map was wrong and is undone in
  the sheets, the interface netlist and the docs (history in notes.md).
- Model: the hairpin's legs follow the cable's real exit - the main board's
  on the board, clear of the thumb switches' poles; 0 DRC FAILs, 0 clashes.
- Sheets: Manufacturer/MPN/LCSC/Assembly fields from JLC's parts API (JLC
  and LCSC pages banked in datasheets/fab and the manifest); five bring-up
  test pads per key board (TP-CHAIN, copper only).
- pcb.py: JLC's limits in the DRC (layout.yaml fab:), which grew the vias
  and J-CHAIN's pads to the 0.18 mm ring; HASL lead-free in the stackup and
  Gerber job; a generated parts-side silkscreen; the JLC BOM, CPL and
  hand-assembly list in fab/, ledgered against board and sheets.
- Router: a real rip-up (blockers removed too); plated holes no longer wall
  off their own pads.
- hardware/boards/key-board-lh/README.md: sources, ordering, hand assembly,
  bring-up, open items. tooling.md and lib README follow.
All checks pass: CAD, DRC (0/0), KiCad, staleness, BOM, netlist, datasheets.

Co-Authored-By: Claude Opus 5.5 <noreply@anthropic.com>
Claude-Session: https://claude.ai/code/session_01LmB4muFXnoLprWX4JzuJ5A
Parts:
- C-KEY: Assembly (none) -> machine; LCSC (none) -> C53134; MPN (none) -> CL21B473KBCNNNC; Manufacturer (none) -> Samsung
- R-KEY-PU: Assembly (none) -> machine; LCSC (none) -> C17520; MPN (none) -> 0805W8F2201T5E; Manufacturer (none) -> UNI-ROYAL
- R-KEY-SER: Assembly (none) -> machine; LCSC (none) -> C17408; MPN (none) -> 0805W8F1000T5E; Manufacturer (none) -> UNI-ROYAL
- SW1-n: Assembly (none) -> hand; MPN (none) -> KS-33 Red (linear) - bought, BOM row SW1-n; Manufacturer (none) -> Gateron
Changed lines of the file:
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@@
     (property "Pins" "1=1 2=2" (at 101.6 91.44 0) (effects (font (size 1.27 1.27)) hide))
     (property "Note" "Pulls the register input to 3V3. It is also what makes the static draw a live trade rather than a free one - the same rail is the MCP3202's reference" (at 101.6 91.44 0) (effects (font (size 1.27 1.27)) hide))
+    (property "Manufacturer" "UNI-ROYAL" (at 101.6 91.44 0) (effects (font (size 1.27 1.27)) hide))
+    (property "MPN" "0805W8F2201T5E" (at 101.6 91.44 0) (effects (font (size 1.27 1.27)) hide))
+    (property "LCSC" "C17520" (at 101.6 91.44 0) (effects (font (size 1.27 1.27)) hide))
+    (property "Assembly" "machine" (at 101.6 91.44 0) (effects (font (size 1.27 1.27)) hide))
     (pin "1")
     (pin "2")
@@
     (property "Pins" "1=1 2=2" (at 101.6 111.76 0) (effects (font (size 1.27 1.27)) hide))
     (property "Note" "Also AT the register input - automatic, because every register sits beside its own switches (main board or key board)" (at 101.6 111.76 0) (effects (font (size 1.27 1.27)) hide))
+    (property "Manufacturer" "Samsung" (at 101.6 111.76 0) (effects (font (size 1.27 1.27)) hide))
+    (property "MPN" "CL21B473KBCNNNC" (at 101.6 111.76 0) (effects (font (size 1.27 1.27)) hide))
+    (property "LCSC" "C53134" (at 101.6 111.76 0) (effects (font (size 1.27 1.27)) hide))
+    (property "Assembly" "machine" (at 101.6 111.76 0) (effects (font (size 1.27 1.27)) hide))
     (pin "1")
     (pin "2")
@@
     (property "Pins" "1=1 2=2" (at 109.22 101.6 0) (effects (font (size 1.27 1.27)) hide))
     (property "Note" "Between the switch and the input node. AT the register input, millimetres from the switch" (at 109.22 101.6 0) (effects (font (size 1.27 1.27)) hide))
+    (property "Manufacturer" "UNI-ROYAL" (at 109.22 101.6 0) (effects (font (size 1.27 1.27)) hide))
+    (property "MPN" "0805W8F1000T5E" (at 109.22 101.6 0) (effects (font (size 1.27 1.27)) hide))
+    (property "LCSC" "C17408" (at 109.22 101.6 0) (effects (font (size 1.27 1.27)) hide))
+    (property "Assembly" "machine" (at 109.22 101.6 0) (effects (font (size 1.27 1.27)) hide))
     (pin "1")
     (pin "2")
@@
     (property "Pins" "1=1 2=2" (at 120.65 109.22 0) (effects (font (size 1.27 1.27)) hide))
     (property "Note" "Two electrical contacts. The row calls the part 3-pin, and the third is a locating post rather than a net - so it is not netted here" (at 120.65 109.22 0) (effects (font (size 1.27 1.27)) hide))
+    (property "Assembly" "hand" (at 120.65 109.22 0) (effects (font (size 1.27 1.27)) hide))
+    (property "Manufacturer" "Gateron" (at 120.65 109.22 0) (effects (font (size 1.27 1.27)) hide))
+    (property "MPN" "KS-33 Red (linear) - bought, BOM row SW1-n" (at 120.65 109.22 0) (effects (font (size 1.27 1.27)) hide))
     (pin "1")
     (pin "2")

Commit message: WIP: layout-side fixes (networks as T, via-in-pad, segment merge, silk, stackup, TP-SER, drills)
Co-Authored-By: Claude Opus 5.5 <noreply@anthropic.com>
Claude-Session: https://claude.ai/code/session_01LmB4muFXnoLprWX4JzuJ5A
Parts:
- C-KEY: Note Also AT the register input - automatic, because every regis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 -> Beside its own switch, with R-KEY-SER and R-KEY-PU: the nod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
- R-KEY-SER: Note Between the switch and the input node. AT the register inpu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 -> Between the switch and the input node, beside the switch. I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
Changed lines of the file:
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@@
     (property "Row" "C-KEY" (at 101.6 111.76 0) (effects (font (size 1.27 1.27)) hide))
     (property "Pins" "1=1 2=2" (at 101.6 111.76 0) (effects (font (size 1.27 1.27)) hide))
-    (property "Note" "Also AT the register input - automatic, because every register sits beside its own switches (main board or key board)" (at 101.6 111.76 0) (effects (font (size 1.27 1.27)) hide))
+    (property "Note" "Beside its own switch, with R-KEY-SER and R-KEY-PU: the node's RC is local to the contact that disturbs it, and the trace on to the register input carries a slow edge" (at 101.6 111.76 0) (effects (font (size 1.27 1.27)) hide))
     (property "Manufacturer" "Samsung" (at 101.6 111.76 0) (effects (font (size 1.27 1.27)) hide))
     (property "MPN" "CL21B473KBCNNNC" (at 101.6 111.76 0) (effects (font (size 1.27 1.27)) hide))
@@
     (property "Row" "R-KEY-SER" (at 109.22 101.6 0) (effects (font (size 1.27 1.27)) hide))
     (property "Pins" "1=1 2=2" (at 109.22 101.6 0) (effects (font (size 1.27 1.27)) hide))
-    (property "Note" "Between the switch and the input node. AT the register input, millimetres from the switch" (at 109.22 101.6 0) (effects (font (size 1.27 1.27)) hide))
+    (property "Note" "Between the switch and the input node, beside the switch. It sets the pressed node's divider with R-KEY-PU and limits C-KEY's discharge into the contact (key-switch-network.md section 2)" (at 109.22 101.6 0) (effects (font (size 1.27 1.27)) hide))
     (property "Manufacturer" "UNI-ROYAL" (at 109.22 101.6 0) (effects (font (size 1.27 1.27)) hide))
     (property "MPN" "0805W8F1000T5E" (at 109.22 101.6 0) (effects (font (size 1.27 1.27)) hide))

Commit message: Wave r2 fixes, part 2: board README, tooling.md, ordering
- README: assembly for the through-wood mount; the layout-only keys
  (R5-10); what check fails on (R5-9, R6-10); ordering: FFSD length code
  zero-padded (R4-1), Samtec header's thin US stock (R4-6), the switch's
  order code and why -Y24 not -Y31 (R4-3), C-BULK's part (R4-7), US
  resistor equivalents (R4-8), the RH board has no layout yet (R4-4);
  the assembly-drawing claim dropped (R3-5); J-CHAIN ring in Open (R3-10);
  the test pads' order stated as it is (R3-9).
- tooling.md section 4: every check and router rule; which generated files
  are not byte-stable (R6-11).
- SW1-n carries its MPN on the sheet; hand-assembly list regenerated.
- pcb_route.py docstring: stitching skips pads on the ground tree.

Co-Authored-By: Claude Opus 5.5 <noreply@anthropic.com>
Claude-Session: https://claude.ai/code/session_01LmB4muFXnoLprWX4JzuJ5A
Parts:
- SW1-n: MPN KS-33 Red (linear) - bought, BOM row SW1-n -> KS-33H10B050NN-Y24
Changed lines of the file:
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@@
     (property "Assembly" "hand" (at 120.65 109.22 0) (effects (font (size 1.27 1.27)) hide))
     (property "Manufacturer" "Gateron" (at 120.65 109.22 0) (effects (font (size 1.27 1.27)) hide))
-    (property "MPN" "KS-33 Red (linear) - bought, BOM row SW1-n" (at 120.65 109.22 0) (effects (font (size 1.27 1.27)) hide))
+    (property "MPN" "KS-33H10B050NN-Y24" (at 120.65 109.22 0) (effects (font (size 1.27 1.27)) hide))
     (pin "1")
     (pin "2")
