File: hardware/module/mod-channels/mod-channels.jack.kicad_sch (KiCad schematic)
At the start: 4 parts

Commit message: WIP module schematics: footprints, bought-part fields, and the two board projects (module-main, module-jack)
Recovered from a container restart; not yet exported or checked.

Co-Authored-By: Claude Opus 5.5 <noreply@anthropic.com>
Claude-Session: https://claude.ai/code/session_01LmB4muFXnoLprWX4JzuJ5A
Parts:
- J-CV-MOD1, J-CV-MOD2, J-CV-MOD3, J-CV-MOD4: footprint (none) -> Connector_Audio:Jack_3.5mm_QingPu_WQP-PJ398SM_Vertical_CircularHoles; Assembly (none) -> hand; MPN (none) -> PJ398SM; Manufacturer (none) -> Thonk
Changed lines of the file:
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@@
     (property "Reference" "J-CV-MOD1" (at 43.18 49.53 0) (effects (font (size 1.27 1.27)) (justify left)))
     (property "Value" "PJ398SM" (at 43.18 52.07 0) (effects (font (size 1.27 1.27)) (justify left)))
-    (property "Footprint" "" (at 40.64 50.8 0) (effects (font (size 1.27 1.27)) hide))
+    (property "Footprint" "Connector_Audio:Jack_3.5mm_QingPu_WQP-PJ398SM_Vertical_CircularHoles" (at 40.64 50.8 0) (effects (font (size 1.27 1.27)) hide))
     (property "Datasheet" "" (at 40.64 50.8 0) (effects (font (size 1.27 1.27)) hide))
     (property "Row" "J-CV" (at 40.64 50.8 0) (effects (font (size 1.27 1.27)) hide))
     (property "Pins" "TIP=T(~) SLEEVE=S(~)" (at 40.64 50.8 0) (effects (font (size 1.27 1.27)) hide))
     (property "Pins_source" "datasheets/connectors/PJ398SM.kicad_mod pad names T, TN, S; datasheets/connectors/PJ398SM-drawing.jpg: 3 tip, 2 normalling contact, 1 sleeve. TN is not on this symbol: unused, not netted" (at 40.64 50.8 0) (effects (font (size 1.27 1.27)) hide))
+    (property "Manufacturer" "Thonk" (at 40.64 50.8 0) (effects (font (size 1.27 1.27)) hide))
+    (property "MPN" "PJ398SM" (at 40.64 50.8 0) (effects (font (size 1.27 1.27)) hide))
+    (property "LCSC" "" (at 40.64 50.8 0) (effects (font (size 1.27 1.27)) hide))
+    (property "Assembly" "hand" (at 40.64 50.8 0) (effects (font (size 1.27 1.27)) hide))
     (pin "S")
     (pin "T")
-    (instances (project "mod-channels.jack" (path "/78e948b4-b72c-521f-91bf-99d3fb72fc5f" (reference "J-CV-MOD1") (unit 1))) (project "mod-channels" (path "/cbc0bf1c-8023-50b5-8559-bb6234a2b622/c20288e6-dbab-5bd0-8a13-eb6772e93998" (reference "J-CV-MOD1") (unit 1))))
+    (instances (project "module-jack" (path "/f69c67ba-c380-5393-90d5-6d2847e300fb/7ec3a694-47c1-564c-a449-ea2fb8fdb831" (reference "J3") (unit 1))) (project "mod-channels.jack" (path "/78e948b4-b72c-521f-91bf-99d3fb72fc5f" (reference "J-CV-MOD1") (unit 1))) (project "mod-channels" (path "/cbc0bf1c-8023-50b5-8559-bb6234a2b622/c20288e6-dbab-5bd0-8a13-eb6772e93998" (reference "J-CV-MOD1") (unit 1))))
   )
   (symbol (lib_id "Connector_Audio:AudioJack2") (at 91.44 50.8 0) (unit 1)
@@
     (property "Reference" "J-CV-MOD2" (at 93.98 49.53 0) (effects (font (size 1.27 1.27)) (justify left)))
     (property "Value" "PJ398SM" (at 93.98 52.07 0) (effects (font (size 1.27 1.27)) (justify left)))
-    (property "Footprint" "" (at 91.44 50.8 0) (effects (font (size 1.27 1.27)) hide))
+    (property "Footprint" "Connector_Audio:Jack_3.5mm_QingPu_WQP-PJ398SM_Vertical_CircularHoles" (at 91.44 50.8 0) (effects (font (size 1.27 1.27)) hide))
     (property "Datasheet" "" (at 91.44 50.8 0) (effects (font (size 1.27 1.27)) hide))
     (property "Row" "J-CV" (at 91.44 50.8 0) (effects (font (size 1.27 1.27)) hide))
     (property "Pins" "TIP=T(~) SLEEVE=S(~)" (at 91.44 50.8 0) (effects (font (size 1.27 1.27)) hide))
     (property "Pins_source" "datasheets/connectors/PJ398SM.kicad_mod pad names T, TN, S; datasheets/connectors/PJ398SM-drawing.jpg: 3 tip, 2 normalling contact, 1 sleeve. TN is not on this symbol: unused, not netted" (at 91.44 50.8 0) (effects (font (size 1.27 1.27)) hide))
+    (property "Manufacturer" "Thonk" (at 91.44 50.8 0) (effects (font (size 1.27 1.27)) hide))
+    (property "MPN" "PJ398SM" (at 91.44 50.8 0) (effects (font (size 1.27 1.27)) hide))
+    (property "LCSC" "" (at 91.44 50.8 0) (effects (font (size 1.27 1.27)) hide))
+    (property "Assembly" "hand" (at 91.44 50.8 0) (effects (font (size 1.27 1.27)) hide))
     (pin "S")
     (pin "T")
-    (instances (project "mod-channels.jack" (path "/78e948b4-b72c-521f-91bf-99d3fb72fc5f" (reference "J-CV-MOD2") (unit 1))) (project "mod-channels" (path "/cbc0bf1c-8023-50b5-8559-bb6234a2b622/c20288e6-dbab-5bd0-8a13-eb6772e93998" (reference "J-CV-MOD2") (unit 1))))
+    (instances (project "module-jack" (path "/f69c67ba-c380-5393-90d5-6d2847e300fb/7ec3a694-47c1-564c-a449-ea2fb8fdb831" (reference "J4") (unit 1))) (project "mod-channels.jack" (path "/78e948b4-b72c-521f-91bf-99d3fb72fc5f" (reference "J-CV-MOD2") (unit 1))) (project "mod-channels" (path "/cbc0bf1c-8023-50b5-8559-bb6234a2b622/c20288e6-dbab-5bd0-8a13-eb6772e93998" (reference "J-CV-MOD2") (unit 1))))
   )
   (symbol (lib_id "Connector_Audio:AudioJack2") (at 142.24 50.8 0) (unit 1)
@@
     (property "Reference" "J-CV-MOD3" (at 144.78 49.53 0) (effects (font (size 1.27 1.27)) (justify left)))
     (property "Value" "PJ398SM" (at 144.78 52.07 0) (effects (font (size 1.27 1.27)) (justify left)))
-    (property "Footprint" "" (at 142.24 50.8 0) (effects (font (size 1.27 1.27)) hide))
+    (property "Footprint" "Connector_Audio:Jack_3.5mm_QingPu_WQP-PJ398SM_Vertical_CircularHoles" (at 142.24 50.8 0) (effects (font (size 1.27 1.27)) hide))
     (property "Datasheet" "" (at 142.24 50.8 0) (effects (font (size 1.27 1.27)) hide))
     (property "Row" "J-CV" (at 142.24 50.8 0) (effects (font (size 1.27 1.27)) hide))
     (property "Pins" "TIP=T(~) SLEEVE=S(~)" (at 142.24 50.8 0) (effects (font (size 1.27 1.27)) hide))
     (property "Pins_source" "datasheets/connectors/PJ398SM.kicad_mod pad names T, TN, S; datasheets/connectors/PJ398SM-drawing.jpg: 3 tip, 2 normalling contact, 1 sleeve. TN is not on this symbol: unused, not netted" (at 142.24 50.8 0) (effects (font (size 1.27 1.27)) hide))
+    (property "Manufacturer" "Thonk" (at 142.24 50.8 0) (effects (font (size 1.27 1.27)) hide))
+    (property "MPN" "PJ398SM" (at 142.24 50.8 0) (effects (font (size 1.27 1.27)) hide))
+    (property "LCSC" "" (at 142.24 50.8 0) (effects (font (size 1.27 1.27)) hide))
+    (property "Assembly" "hand" (at 142.24 50.8 0) (effects (font (size 1.27 1.27)) hide))
     (pin "S")
     (pin "T")
-    (instances (project "mod-channels.jack" (path "/78e948b4-b72c-521f-91bf-99d3fb72fc5f" (reference "J-CV-MOD3") (unit 1))) (project "mod-channels" (path "/cbc0bf1c-8023-50b5-8559-bb6234a2b622/c20288e6-dbab-5bd0-8a13-eb6772e93998" (reference "J-CV-MOD3") (unit 1))))
+    (instances (project "module-jack" (path "/f69c67ba-c380-5393-90d5-6d2847e300fb/7ec3a694-47c1-564c-a449-ea2fb8fdb831" (reference "J5") (unit 1))) (project "mod-channels.jack" (path "/78e948b4-b72c-521f-91bf-99d3fb72fc5f" (reference "J-CV-MOD3") (unit 1))) (project "mod-channels" (path "/cbc0bf1c-8023-50b5-8559-bb6234a2b622/c20288e6-dbab-5bd0-8a13-eb6772e93998" (reference "J-CV-MOD3") (unit 1))))
   )
   (symbol (lib_id "Connector_Audio:AudioJack2") (at 193.04 50.8 0) (unit 1)
@@
     (property "Reference" "J-CV-MOD4" (at 195.58 49.53 0) (effects (font (size 1.27 1.27)) (justify left)))
     (property "Value" "PJ398SM" (at 195.58 52.07 0) (effects (font (size 1.27 1.27)) (justify left)))
-    (property "Footprint" "" (at 193.04 50.8 0) (effects (font (size 1.27 1.27)) hide))
+    (property "Footprint" "Connector_Audio:Jack_3.5mm_QingPu_WQP-PJ398SM_Vertical_CircularHoles" (at 193.04 50.8 0) (effects (font (size 1.27 1.27)) hide))
     (property "Datasheet" "" (at 193.04 50.8 0) (effects (font (size 1.27 1.27)) hide))
     (property "Row" "J-CV" (at 193.04 50.8 0) (effects (font (size 1.27 1.27)) hide))
     (property "Pins" "TIP=T(~) SLEEVE=S(~)" (at 193.04 50.8 0) (effects (font (size 1.27 1.27)) hide))
     (property "Pins_source" "datasheets/connectors/PJ398SM.kicad_mod pad names T, TN, S; datasheets/connectors/PJ398SM-drawing.jpg: 3 tip, 2 normalling contact, 1 sleeve. TN is not on this symbol: unused, not netted" (at 193.04 50.8 0) (effects (font (size 1.27 1.27)) hide))
+    (property "Manufacturer" "Thonk" (at 193.04 50.8 0) (effects (font (size 1.27 1.27)) hide))
+    (property "MPN" "PJ398SM" (at 193.04 50.8 0) (effects (font (size 1.27 1.27)) hide))
+    (property "LCSC" "" (at 193.04 50.8 0) (effects (font (size 1.27 1.27)) hide))
+    (property "Assembly" "hand" (at 193.04 50.8 0) (effects (font (size 1.27 1.27)) hide))
     (pin "S")
     (pin "T")
-    (instances (project "mod-channels.jack" (path "/78e948b4-b72c-521f-91bf-99d3fb72fc5f" (reference "J-CV-MOD4") (unit 1))) (project "mod-channels" (path "/cbc0bf1c-8023-50b5-8559-bb6234a2b622/c20288e6-dbab-5bd0-8a13-eb6772e93998" (reference "J-CV-MOD4") (unit 1))))
+    (instances (project "module-jack" (path "/f69c67ba-c380-5393-90d5-6d2847e300fb/7ec3a694-47c1-564c-a449-ea2fb8fdb831" (reference "J6") (unit 1))) (project "mod-channels.jack" (path "/78e948b4-b72c-521f-91bf-99d3fb72fc5f" (reference "J-CV-MOD4") (unit 1))) (project "mod-channels" (path "/cbc0bf1c-8023-50b5-8559-bb6234a2b622/c20288e6-dbab-5bd0-8a13-eb6772e93998" (reference "J-CV-MOD4") (unit 1))))
   )
   (wire (pts (xy 45.72 50.8) (xy 48.26 50.8)) (stroke (width 0) (type default)))
