File: hardware/module/mod-channels/mod-channels.main.kicad_sch (KiCad schematic)
At the start: 39 parts

Commit message: WIP module schematics: footprints, bought-part fields, and the two board projects (module-main, module-jack)
Recovered from a container restart; not yet exported or checked.

Co-Authored-By: Claude Opus 5.5 <noreply@anthropic.com>
Claude-Session: https://claude.ai/code/session_01LmB4muFXnoLprWX4JzuJ5A
Parts:
- C-DEC-MODA-NEG, C-DEC-MODA-POS, C-DEC-MODB-NEG, C-DEC-MODB-POS, C-DEC-MODC-NEG, C-DEC-MODC-POS: footprint (none) -> Capacitor_SMD:C_0805_2012Metric; Assembly (none) -> machine; LCSC (none) -> C49678; MPN (none) -> CC0805KRX7R9BB104; Manufacturer (none) -> YAGEO
- C-FILT-MOD-1, C-FILT-MOD-2, C-FILT-MOD-3, C-FILT-MOD-4: footprint (none) -> Capacitor_SMD:C_1206_3216Metric; Assembly (none) -> machine; LCSC (none) -> C97947; MPN (none) -> GRM31C5C1H823JA01L; Manufacturer (none) -> Murata
- D-JACK-CLAMP-1, D-JACK-CLAMP-2, D-JACK-CLAMP-3, D-JACK-CLAMP-4: footprint (none) -> Package_TO_SOT_SMD:SOT-23; Assembly (none) -> machine; LCSC (none) -> C2500; MPN (none) -> BAV99,215; Manufacturer (none) -> Nexperia
- R-BIAS-DAC-1, R-BIAS-DAC-2, R-BIAS-DAC-3, R-BIAS-DAC-4, R-BIAS-DAC-CH7: footprint (none) -> Resistor_SMD:R_0805_2012Metric; Assembly (none) -> machine; LCSC (none) -> C149504; MPN (none) -> 0805W8F1003T5E; Manufacturer (none) -> UNI-ROYAL(Uniroyal Elec)
- R-OPAMP-IN-1, R-OPAMP-IN-2, R-OPAMP-IN-3, R-OPAMP-IN-4, R-OPAMP-IN-REF: footprint (none) -> Resistor_SMD:R_0805_2012Metric; Assembly (none) -> machine; LCSC (none) -> C17513; MPN (none) -> 0805W8F1001T5E; Manufacturer (none) -> UNI-ROYAL(Uniroyal Elec)
- R-OUT-PROT-1, R-OUT-PROT-2, R-OUT-PROT-3, R-OUT-PROT-4: footprint (none) -> Resistor_SMD:R_1206_3216Metric; Assembly (none) -> machine; LCSC (none) -> C4261071; MPN (none) -> ERJ-P08F1001V; Manufacturer (none) -> Panasonic
- R1-1, R1-2, R1-3, R1-4: footprint (none) -> Resistor_SMD:R_0805_2012Metric; Assembly (none) -> machine; LCSC (none) -> C110775; MPN (none) -> RT0805BRD0710KL; Manufacturer (none) -> YAGEO
- R2-1, R2-2, R2-3, R2-4: footprint (none) -> Resistor_SMD:R_0805_2012Metric; Assembly (none) -> machine; LCSC (none) -> C728649; MPN (none) -> RT0805BRD0730KL; Manufacturer (none) -> YAGEO
- U-MOD-A, U-MOD-B, U-MOD-C: footprint (none) -> Package_SO:SOIC-8_3.9x4.9mm_P1.27mm; Assembly (none) -> machine; LCSC (none) -> C139363; MPN (none) -> OPA2197IDR; Manufacturer (none) -> Texas Instruments

Commit message: Mod gain resistors specified 0.1 % (A2-12, owner): sheet values, BOM rows, page tolerance table, mod-jack-range re-derived, sim re-run
Co-Authored-By: Claude Opus 5.5 <noreply@anthropic.com>
Claude-Session: https://claude.ai/code/session_01LmB4muFXnoLprWX4JzuJ5A
Parts:
- R1-1, R1-2, R1-3, R1-4: value 10k 1% -> 10k 0.1%
- R2-1, R2-2, R2-3, R2-4: value 30k 1% -> 30k 0.1%
Changed lines of the file:
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@@
     (in_bom yes) (on_board yes) (dnp no)
     (property "Reference" "R1-1" (at 551.18 278.13 0) (effects (font (size 1.27 1.27)) (justify left)))
-    (property "Value" "10k 1%" (at 551.18 280.67 0) (effects (font (size 1.27 1.27)) (justify left)))
+    (property "Value" "10k 0.1%" (at 551.18 280.67 0) (effects (font (size 1.27 1.27)) (justify left)))
     (property "Footprint" "Resistor_SMD:R_0805_2012Metric" (at 547.37 279.4 0) (effects (font (size 1.27 1.27)) hide))
     (property "Datasheet" "" (at 548.64 279.4 0) (effects (font (size 1.27 1.27)) hide))
@@
     (in_bom yes) (on_board yes) (dnp no)
     (property "Reference" "R2-1" (at 601.98 278.13 0) (effects (font (size 1.27 1.27)) (justify left)))
-    (property "Value" "30k 1%" (at 601.98 280.67 0) (effects (font (size 1.27 1.27)) (justify left)))
+    (property "Value" "30k 0.1%" (at 601.98 280.67 0) (effects (font (size 1.27 1.27)) (justify left)))
     (property "Footprint" "Resistor_SMD:R_0805_2012Metric" (at 598.17 279.4 0) (effects (font (size 1.27 1.27)) hide))
     (property "Datasheet" "" (at 599.44 279.4 0) (effects (font (size 1.27 1.27)) hide))
@@
     (in_bom yes) (on_board yes) (dnp no)
     (property "Reference" "R1-2" (at 195.58 323.85 0) (effects (font (size 1.27 1.27)) (justify left)))
-    (property "Value" "10k 1%" (at 195.58 326.39 0) (effects (font (size 1.27 1.27)) (justify left)))
+    (property "Value" "10k 0.1%" (at 195.58 326.39 0) (effects (font (size 1.27 1.27)) (justify left)))
     (property "Footprint" "Resistor_SMD:R_0805_2012Metric" (at 191.77 325.12 0) (effects (font (size 1.27 1.27)) hide))
     (property "Datasheet" "" (at 193.04 325.12 0) (effects (font (size 1.27 1.27)) hide))
@@
     (in_bom yes) (on_board yes) (dnp no)
     (property "Reference" "R2-2" (at 246.38 323.85 0) (effects (font (size 1.27 1.27)) (justify left)))
-    (property "Value" "30k 1%" (at 246.38 326.39 0) (effects (font (size 1.27 1.27)) (justify left)))
+    (property "Value" "30k 0.1%" (at 246.38 326.39 0) (effects (font (size 1.27 1.27)) (justify left)))
     (property "Footprint" "Resistor_SMD:R_0805_2012Metric" (at 242.57 325.12 0) (effects (font (size 1.27 1.27)) hide))
     (property "Datasheet" "" (at 243.84 325.12 0) (effects (font (size 1.27 1.27)) hide))
@@
     (in_bom yes) (on_board yes) (dnp no)
     (property "Reference" "R1-3" (at 601.98 323.85 0) (effects (font (size 1.27 1.27)) (justify left)))
-    (property "Value" "10k 1%" (at 601.98 326.39 0) (effects (font (size 1.27 1.27)) (justify left)))
+    (property "Value" "10k 0.1%" (at 601.98 326.39 0) (effects (font (size 1.27 1.27)) (justify left)))
     (property "Footprint" "Resistor_SMD:R_0805_2012Metric" (at 598.17 325.12 0) (effects (font (size 1.27 1.27)) hide))
     (property "Datasheet" "" (at 599.44 325.12 0) (effects (font (size 1.27 1.27)) hide))
@@
     (in_bom yes) (on_board yes) (dnp no)
     (property "Reference" "R2-3" (at 652.78 323.85 0) (effects (font (size 1.27 1.27)) (justify left)))
-    (property "Value" "30k 1%" (at 652.78 326.39 0) (effects (font (size 1.27 1.27)) (justify left)))
+    (property "Value" "30k 0.1%" (at 652.78 326.39 0) (effects (font (size 1.27 1.27)) (justify left)))
     (property "Footprint" "Resistor_SMD:R_0805_2012Metric" (at 648.97 325.12 0) (effects (font (size 1.27 1.27)) hide))
     (property "Datasheet" "" (at 650.24 325.12 0) (effects (font (size 1.27 1.27)) hide))
@@
     (in_bom yes) (on_board yes) (dnp no)
     (property "Reference" "R1-4" (at 297.18 369.57 0) (effects (font (size 1.27 1.27)) (justify left)))
-    (property "Value" "10k 1%" (at 297.18 372.11 0) (effects (font (size 1.27 1.27)) (justify left)))
+    (property "Value" "10k 0.1%" (at 297.18 372.11 0) (effects (font (size 1.27 1.27)) (justify left)))
     (property "Footprint" "Resistor_SMD:R_0805_2012Metric" (at 293.37 370.84 0) (effects (font (size 1.27 1.27)) hide))
     (property "Datasheet" "" (at 294.64 370.84 0) (effects (font (size 1.27 1.27)) hide))
@@
     (in_bom yes) (on_board yes) (dnp no)
     (property "Reference" "R2-4" (at 347.98 369.57 0) (effects (font (size 1.27 1.27)) (justify left)))
-    (property "Value" "30k 1%" (at 347.98 372.11 0) (effects (font (size 1.27 1.27)) (justify left)))
+    (property "Value" "30k 0.1%" (at 347.98 372.11 0) (effects (font (size 1.27 1.27)) (justify left)))
     (property "Footprint" "Resistor_SMD:R_0805_2012Metric" (at 344.17 370.84 0) (effects (font (size 1.27 1.27)) hide))
     (property "Datasheet" "" (at 345.44 370.84 0) (effects (font (size 1.27 1.27)) hide))
