File: hardware/module/power-entry/power-entry.kicad_sch (KiCad schematic)
At the start: 32 parts

Commit message: U-ISO is the in-stock RECOM RPA20-2412SAW (owner correction), not the RP20
Footprint Converter_DCDC_RECOM_RPA20-RP20-xxxxSAW_THT: RPA20 numbering
(4 -Vout, 5 Trim, 6 +Vout; no CTRL), and its descr records that the RP20
drops into the same holes with 4/6 swapped. Trim is a no-connect again.
BOM rows and sim params from RECOM-RPA20-AW.pdf: +/-3.1 %, 0.007 ohm,
eta 0.82, 1.1 nF. Sims: 198 runs/5 asserts and 20 runs/23 asserts, 0 failed.

Co-Authored-By: Claude Opus 5.5 <noreply@anthropic.com>
Claude-Session: https://claude.ai/code/session_01LmB4muFXnoLprWX4JzuJ5A
Parts:
- C-ISO-IN: Note Across U-ISO's input pins, beside them: the ceramic half of the input filter (RECOM's Class B C1 for the RP20-24xxSAW, 4.7uF MLCC, PD-6; 50 V here because it sits across both rails) -> Across U-ISO's input pins, beside them: the ceramic half of the input filter (the RPA20 datasheet names no ceramic, PD-7; 4.7uF 50 V beside the pins takes the switching current off C2)
- C-ISO-OUT: Note U-ISO's output capacitor, 100uF/25V: well inside the RP20-2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 -> U-ISO's output capacitor, 100uF/25V: well inside the RPA20-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
- C-ISO-Y: Note Across the isolation barrier AT the converter, ISO_VIN_POS to PWR_GND: gives the switching common-mode current a 1 nF path home beside U-ISO instead of round the star and the ribbon (RECOM's Class B filter puts 470pF across the barrier on each side, C4/C5, PD-6; one 1 nF here). On the +12 V side so PTC-ISO covers it if it fails short -> Across the isolation barrier AT the converter, ISO_VIN_POS to PWR_GND: gives the switching common-mode current a 1 nF path home beside U-ISO instead of round the star and the ribbon (RECOM's RPA20 filter has no Y-capacitor, PD-7; one 1 nF here against its 1100pF isolation capacitance, PD-5). On the +12 V side so PTC-ISO covers it if it fails short
- C2: Note U-ISO's input bulk, ACROSS its input (ISO_VIN_POS to ISO_VIN_NEG, 24 V): the external input electrolytic RECOM asks for (RECOM-RP20-AW.pdf PD-5 Note 11, which suggests 220uF/100V where a surge test applies; 100uF/50V here, on the rack's rails). An electrolytic with real ESR, because it damps L-ISO-IN (power-entry.md) -> U-ISO's input bulk, ACROSS its input (ISO_VIN_POS to ISO_VIN_NEG, 24 V): RECOM's input electrolytic (RECOM-RPA20-AW.pdf PD-7 filter: C1 47uF/50V; 100uF/50V here). An electrolytic with real ESR, because it damps L-ISO-IN (power-entry.md)
- PTC-ISO: Note The converter branch's fuse, in its +12 V leg ahead of D2, and the input fuse RECOM requires (RECOM-RP20-AW.pdf PD-4 Note 8: 'not internally fused. An input line fuse must always be used'): the load switch is on U-ISO's output and cannot see a fault in U-ISO or its input network. One leg is enough - the branch is a series loop, +12 through U-ISO to -12, and C-ISO-Y hangs on the +12 side of it. power-entry.md, 'Fuses on the rails' -> The converter branch's fuse, in its +12 V leg ahead of D2, and the input fuse RECOM recommends (RECOM-RPA20-AW.pdf PD-5 Note 5: 3A slow blow, 'refer to local safety regulations'; F1 in the PD-7 filter): the load switch is on U-ISO's output and cannot see a fault in U-ISO or its input network. One leg is enough - the branch is a series loop, +12 through U-ISO to -12, and C-ISO-Y hangs on the +12 side of it. power-entry.md, 'Fuses on the rails'
- U-ISO: value RP20-2412SAW -> RPA20-2412SAW; footprint woody:Converter_DCDC_RECOM_RP20-xxxxSAW_THT -> woody:Converter_DCDC_RECOM_RPA20-RP20-xxxxSAW_THT; symbol woody:RP20-xxxxSAW -> woody:RPA20-xxxxSAW; MPN RP20-2412SAW -> RPA20-2412SAW; Note THE INSTRUMENT'S SUPPLY, ISOLATED (ADR 0027): input across the rack's +12 V and -12 V, so the instrument's current loops rail to rail and never enters the rack's ground; output +12 V to the load switch, return on PWR_GND, which meets the module's grounds only through NT-UMB-MOD and NT-DIG-MOD. The standard RP20-2412SAW has no CTRL and no Trim pin (PD-1 Note 3): always on, 12 V nominal. RECOM requires an input fuse (PD-4 Note 8): PTC-ISO -> THE INSTRUMENT'S SUPPLY, ISOLATED (ADR 0027): input across the rack's +12 V and -12 V, so the instrument's current loops rail to rail and never enters the rack's ground; output +12 V to the load switch, return on PWR_GND, which meets the module's grounds only through NT-UMB-MOD and NT-DIG-MOD. The standard RPA20-2412SAW has no CTRL pin (PD-1 Note 2): always on; Trim open = 12 V nominal. Input fuse per RECOM's PD-5 Note 5: PTC-ISO. The RP20-2412SAW drops into the same holes (footprint's descr); Pins VIN=1(+Vin) GND=2(-Vin) VO=4(+Vout) 0V=6(-Vout) -> VIN=1(+Vin) GND=2(-Vin) 0V=4(-Vout) TRIM=5(Trim) VO=6(+Vout); Pins_source datasheets/discrete-and-power/RECOM-RP20-AW.pdf PD-6 Pinnin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 -> datasheets/discrete-and-power/RECOM-RPA20-AW.pdf PD-8 Pin C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
Connections:
- net ISO_POS12: now also U-ISO.6 (+Vout); no longer U-ISO.4 (+Vout)
- net PWR_GND: now also U-ISO.4 (-Vout); no longer U-ISO.6 (-Vout)
- no-connect marks 6 -> 7
