File: hardware/module/power-entry/power-entry.kicad_sch (KiCad schematic)
At the start: 34 parts

Commit message: DAC rail: LT3042 set by R-SET-DAC 52.3k 0.1 % replaces the LM317L and TRIM-DAC-RAIL (owner, 2026-10-01); sheet, export, renders, BOM, figures, sims (WIP: pages follow)
Co-Authored-By: Claude Opus 5.5 <noreply@anthropic.com>
Claude-Session: https://claude.ai/code/session_01LmB4muFXnoLprWX4JzuJ5A
Parts:
- removed C-REG-ADJ: 10uF, Capacitor_SMD:C_0805_2012Metric, symbol Device:C
- removed R-REG-SET-HI: 150R 0.1%, Resistor_SMD:R_0805_2012Metric, symbol Device:R
- removed R-REG-SET-LO: 523R 0.1%, Resistor_SMD:R_0805_2012Metric, symbol Device:R
- removed TRIM-DAC-RAIL: 50R, Potentiometer_SMD:Potentiometer_Bourns_3224W_Vertical, symbol Device:R_Potentiometer_Trim
- removed U-REG-DAC: LM317LZ, Package_TO_SOT_THT:TO-92_Inline, symbol Regulator_Linear:LM317L_TO92
- added C-REG-IN: 10uF, Capacitor_SMD:C_1206_3216Metric, symbol Device:C
- added C-SET-DAC: 100nF, Capacitor_SMD:C_1206_3216Metric, symbol Device:C
- added R-SET-DAC: 52.3k 0.1%, Resistor_SMD:R_0805_2012Metric, symbol Device:R
- added U-REG-DAC: LT3042EMSE, Package_SO:MSOP-10-1EP_3x3mm_P0.5mm_EP1.68x1.88mm, symbol Regulator_Linear:LT3042xMSE
- C-DEC-REG-IN: Note At the LM317's input pin. One of the board-wide C-DECOUPLE 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 -> At U-REG-DAC's (LT3042) IN pins, beside C-REG-IN: the HF pa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
- C-REG-OUT: value 1uF -> 10uF; footprint Capacitor_SMD:C_0805_2012Metric -> Capacitor_SMD:C_1206_3216Metric; Drawn_as C -> (none); LCSC C28323 -> C531431; MPN CL21B105KBFNNNE -> CGA5L1X7R1H106KT0Y0N; Manufacturer Samsung Electro-Mechanics -> TDK; Note (none) -> U-REG-DAC's (LT3042) output capacitor, at OUT with OUTS Kel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; Row C-REG-OUT -> C-REG-DAC
Connections:
- net AGND_MOD: now also C-REG-IN.2, C-SET-DAC.2, R-SET-DAC.2, U-REG-DAC.11 (GND), U-REG-DAC.5 (ILIM), U-REG-DAC.8 (GND)
- net DAC_AVDD: now also U-REG-DAC.10 (OUT), U-REG-DAC.9 (OUTS)
- net MODULE_ANALOG_POS12: now also C-REG-IN.1, U-REG-DAC.1 (IN), U-REG-DAC.2 (IN), U-REG-DAC.3 (EN/UV), U-REG-DAC.6 (PGFB)
- new net DAC_REG_SET: C-SET-DAC.1, R-SET-DAC.1, U-REG-DAC.7 (SET)
- no-connect marks 7 -> 8
Other:
- note added: "FROM THE HAND-WRITTEN NETLIST THIS SHEET REPLACES (verbatim; the part notes are on each part's Note field): AUTHORITATIVE for connectivity. The drawing in power-entry.md is a representation of this file. SCOPE. This circuit owns the rail entry and its fuses, the bead-and-bulk branches, the DAC rail (U-REG-DAC), the logic 5 V and the instrument's isolated supply up to ISO_POS12 and PWR_GND. The lo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"
- note added: "REPLACED 2026-10-01 (owner: a precision-set LDO, no trimmer): U-REG-DAC is the LT3042, DAC_AVDD = I_SET x R-SET-DAC with nothing to adjust. EN/UV and PGFB on IN, PG open, ILIM on AGND_MOD. C-SET-DAC (NP0) across R-SET-DAC; C-REG-IN and C-REG-OUT at its pins, OUTS Kelvin to C-REG-OUT. power-entry.md, The DAC rail"
- note removed: "FROM THE HAND-WRITTEN NETLIST THIS SHEET REPLACES (verbatim; the part notes are on each part's Note field): AUTHORITATIVE for connectivity. The drawing in power-entry.md is a representation of this file. SCOPE. This circuit owns the rail entry and its fuses, the bead-and-bulk branches, the LM317, the logic 5 V and the instrument's isolated supply up to ISO_POS12 and PWR_GND. The load switch those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"
