File: hardware/module/power-entry/power-entry.main.kicad_sch (KiCad schematic)
At the start: 26 parts

Commit message: #19 #8: thirteen LEDs (tail-end LED removed, owner); C-STRIP-BULK two 6.3x7.7 polymer cans; J-MCU at 262.27
The owner, 2026-10-03: "remove that bottom led again" / "Keep current
layout, remove bottom one". ADR 0028 second amendment of 2026-10-03.

- lighting.led_count 14 -> 13; new lighting.led_slots 14 keeps LED2-14
  where they stood (pitch 19.869, x 24.55 ... 262.98), now LED1-13;
  drc.echo 'LED row on the main board' prints count and places.
- led-strip-drive sheet: D-LED-1 / C-LED-1 (D7 / C25) removed, the chain
  renumbered from the tail with every part's UUID kept; new D-LED-1's DIN2
  grounded; BOM qty 13.
- Figures by the three-step rule (the 14-LED spellings grepped first, moved
  into forbidden; the 13-LED spellings that are correct again taken out):
  led-row-current 170-195 mA, umbilical-current 359 mA, hotplug-iso-ocp
  0.49-0.54 A / 3.4x, instrument-input-z-margin 55x / 159x, led-pwm-rail-ripple
  5.6 mV / 0.00088 cents, led-pwm-pitch 0.0034 / 0.011 cents,
  diode-split-rationale back at 0.22 A.
- C10 replacement (coordinator-approved, all four criteria hold):
  C-STRIP-BULK is two MA25V220M6X8 (JIERR, LCSC C46550464), 220 uF 25 V
  polymer, 6.3 x 7.7 mm, in parallel (C10, C44): 14 mohm at 100 kHz
  (<= 0.16), ripple 2.9 A x 0.3 at 1-10 kHz per can vs a 0.367 A swing,
  440 uF; every sim that takes the bulk now takes the pair (c_strip,
  r_strip) and passes. Datasheet and EasyEDA footprint banked (fragment
  R52), JLC rotation row by pin function (0).
- Sims re-run, not scaled, 0 failed: led-strip-drive, power-entry-instrument,
  umbilical-load-switch, panel-led, digital-and-supervision, power-entry,
  interfaces/system, breath-adc, breath-output-stage.
- ADR 0005, 0014, 0016, 0021, 0027, 0028 (amendment), firmware README
  (13 pixels), led-strip-drive, power-entry-instrument, power-entry,
  umbilical-load-switch pages and sim READMEs follow.
- boards.mcu_conn_at [262.27, 12.29, 90] (the owner's option 1; the
  Matrix branch carries the same line); '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
Parts:
- FB2: Note U-ISO's +12 V input leg; FB4 is its -12 V leg. They carry the converter's input, ~0.23 A in typical play, which puts them between the bias curve's 0 and 250 mA traces (ferrite-bias-impedance): the two of the four where DC bias matters - see the FB-IN row. ORDERED AS MI1206K601R-10: JLC sources it through Global Sourcing / consignment (owner, 2026-10-01), so it stays machine-placed though LCSC lists 0 - see the FB-IN row -> U-ISO's +12 V input leg; FB4 is its -12 V leg. They carry the converter's input, ~0.22 A in typical play, which puts them between the bias curve's 0 and 250 mA traces (ferrite-bias-impedance): the two of the four where DC bias matters - see the FB-IN row. ORDERED AS MI1206K601R-10: JLC sources it through Global Sourcing / consignment (owner, 2026-10-01), so it stays machine-placed though LCSC lists 0 - see the FB-IN row
Changed lines of the file:
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@@
     (property "Pins" "1=1 2=2" (at 243.84 142.24 0) (effects (font (size 1.27 1.27)) hide))
     (property "Drawn_as" "FB2" (at 243.84 142.24 0) (effects (font (size 1.27 1.27)) hide))
-    (property "Note" "U-ISO's +12 V input leg; FB4 is its -12 V leg. They carry the converter's input, ~0.23 A in typical play, which puts them between the bias curve's 0 and 250 mA traces (ferrite-bias-impedance): the two of the four where DC bias matters - see the FB-IN row. ORDERED AS MI1206K601R-10: JLC sources it through Global Sourcing / consignment (owner, 2026-10-01), so it stays machine-placed though LCSC lists 0 - see the FB-IN row" (at 243.84 142.24 0) (effects (font (size 1.27 1.27)) hide))
+    (property "Note" "U-ISO's +12 V input leg; FB4 is its -12 V leg. They carry the converter's input, ~0.22 A in typical play, which puts them between the bias curve's 0 and 250 mA traces (ferrite-bias-impedance): the two of the four where DC bias matters - see the FB-IN row. ORDERED AS MI1206K601R-10: JLC sources it through Global Sourcing / consignment (owner, 2026-10-01), so it stays machine-placed though LCSC lists 0 - see the FB-IN row" (at 243.84 142.24 0) (effects (font (size 1.27 1.27)) hide))
     (property "Manufacturer" "Laird" (at 243.84 142.24 0) (effects (font (size 1.27 1.27)) hide))
     (property "MPN" "MI1206K601R-10" (at 243.84 142.24 0) (effects (font (size 1.27 1.27)) hide))
