File: hardware/boards/main-board/main-board.kicad_sch (KiCad schematic)
At the start: 15 parts, among them J4 12-way, J5 12-way, J6 8-way 2.54mm right-angle pin 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, U10 MPXV4006DP, U9 SP0504BAHTG 4-channel 5V array

Commit message: Clamp the REF5050's input; bank the main board's chosen-part datasheets
The rail's TVS clamps at up to 24.4 V, and the REF5050's VIN absolute maximum
is 18 V. The reference is now fed through R-REF-IN (330R) and held by
D-REF-CLAMP (MMSZ5245B 15 V zener) on a new REF_VIN node. At the TVS clamp
the zener holds VIN at about 16.1 V or less. In normal running the drop is
0.4 V.

- The breath-excitation-reference sheet is rebuilt from its netlist and
  re-exported, with a PWR_FLAG on REF_VIN.
- The page gains a derivation section, and carrier.md's drawing shows the
  clamp.
- The main board re-places the sheets; the reference table is regenerated.
  R and D references after the new parts shift by one.
- Board ERC is clean, and key-board fab is re-rendered (fingerprints only).
- Fragments R24/R25 bank the parts agents' datasheets, 196 verified.

Co-Authored-By: Claude Opus 5.5 <noreply@anthropic.com>
Claude-Session: https://claude.ai/code/session_01LmB4muFXnoLprWX4JzuJ5A
Parts:
- renumbered D4 to D5, D5 to D6, R33 to R34, R34 to R35, R35 to R36, R36 to R37, R37 to R38, R38 to R39
Changed lines of the file:
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@@
   (title_block
     (title "Woody main board (hardware/boards/main-board)")
+    (comment 7 "title: Main board")
     (date "")
     (rev "")
     (company "Woody")
-    (comment 1 "SOURCE for this board - edit in KiCad 9. board-netlist.yaml is exported: python3 tools/kicad.py export hardware/boards/main-board")
-    (comment 2 "Each block is a circuit sheet placed once per instance; the root draws the interface circuits' main-board parts")
-    (comment 3 "ADR 0017, ADR 0018, ADR 0019, ADR 0021, ADR 0022")
-    (comment 4 "Register inputs must match allocation.yaml, J-CHAIN the loom's J-CHAIN-MAIN - tools/kicad.py check")
+    (comment 1 "SOURCE (written once by the main board's migration) - edit in KiCad; connectivity: hardware/boards/main-board/netlist.yaml")
+    (comment 2 "placement: schematic.yaml; checked against netlist.yaml by kicad-cli netlist export")
+    (comment 3 "SOURCE - edit in KiCad 9; tools/kicad.py exports board-netlist.yaml")
+    (comment 4 "fingerprint source - verify: python3 tools/sch.py check hardware/boards/main-board")
   )
   (symbol (lib_id "Connector_Generic:Conn_01x12") (at 106.68 63.5 0) (unit 1)
@@
   (symbol (lib_id "Device:R") (at 106.68 152.4 0) (unit 1)
     (in_bom yes) (on_board yes) (dnp no)
-    (property "Reference" "R33" (at 109.22 151.13 0) (effects (font (size 1.27 1.27)) (justify left)))
+    (property "Reference" "R34" (at 109.22 151.13 0) (effects (font (size 1.27 1.27)) (justify left)))
     (property "Value" "100R 1%" (at 109.22 153.67 0) (effects (font (size 1.27 1.27)) (justify left)))
     (property "Footprint" "" (at 105.41 152.4 0) (effects (font (size 1.27 1.27)) hide))
@@
     (pin "1")
     (pin "2")
-    (instances (project "main-board" (path "/b12a49ac-ffa0-5078-b2ba-e15d161f1936" (reference "R33") (unit 1))))
+    (instances (project "main-board" (path "/b12a49ac-ffa0-5078-b2ba-e15d161f1936" (reference "R34") (unit 1))))
   )
   (symbol (lib_id "Device:R") (at 106.68 182.88 0) (unit 1)
     (in_bom yes) (on_board yes) (dnp no)
-    (property "Reference" "R34" (at 109.22 181.61 0) (effects (font (size 1.27 1.27)) (justify left)))
+    (property "Reference" "R35" (at 109.22 181.61 0) (effects (font (size 1.27 1.27)) (justify left)))
     (property "Value" "100R 1%" (at 109.22 184.15 0) (effects (font (size 1.27 1.27)) (justify left)))
     (property "Footprint" "" (at 105.41 182.88 0) (effects (font (size 1.27 1.27)) hide))
@@
     (pin "1")
     (pin "2")
-    (instances (project "main-board" (path "/b12a49ac-ffa0-5078-b2ba-e15d161f1936" (reference "R34") (unit 1))))
+    (instances (project "main-board" (path "/b12a49ac-ffa0-5078-b2ba-e15d161f1936" (reference "R35") (unit 1))))
   )
   (symbol (lib_id "Device:R") (at 106.68 213.36 0) (unit 1)
     (in_bom yes) (on_board yes) (dnp no)
-    (property "Reference" "R35" (at 109.22 212.09 0) (effects (font (size 1.27 1.27)) (justify left)))
+    (property "Reference" "R36" (at 109.22 212.09 0) (effects (font (size 1.27 1.27)) (justify left)))
     (property "Value" "100R 1%" (at 109.22 214.63 0) (effects (font (size 1.27 1.27)) (justify left)))
     (property "Footprint" "" (at 105.41 213.36 0) (effects (font (size 1.27 1.27)) hide))
@@
     (pin "1")
     (pin "2")
-    (instances (project "main-board" (path "/b12a49ac-ffa0-5078-b2ba-e15d161f1936" (reference "R35") (unit 1))))
+    (instances (project "main-board" (path "/b12a49ac-ffa0-5078-b2ba-e15d161f1936" (reference "R36") (unit 1))))
   )
   (symbol (lib_id "Device:R") (at 106.68 243.84 0) (unit 1)
     (in_bom yes) (on_board yes) (dnp no)
-    (property "Reference" "R36" (at 109.22 242.57 0) (effects (font (size 1.27 1.27)) (justify left)))
+    (property "Reference" "R37" (at 109.22 242.57 0) (effects (font (size 1.27 1.27)) (justify left)))
     (property "Value" "10k" (at 109.22 245.11 0) (effects (font (size 1.27 1.27)) (justify left)))
     (property "Footprint" "" (at 105.41 243.84 0) (effects (font (size 1.27 1.27)) hide))
@@
     (pin "1")
     (pin "2")
-    (instances (project "main-board" (path "/b12a49ac-ffa0-5078-b2ba-e15d161f1936" (reference "R36") (unit 1))))
+    (instances (project "main-board" (path "/b12a49ac-ffa0-5078-b2ba-e15d161f1936" (reference "R37") (unit 1))))
   )
   (symbol (lib_id "Device:FerriteBead") (at 106.68 274.32 0) (unit 1)
@@
   (symbol (lib_id "Device:R") (at 106.68 396.24 0) (unit 1)
     (in_bom yes) (on_board yes) (dnp no)
-    (property "Reference" "R37" (at 109.22 394.97 0) (effects (font (size 1.27 1.27)) (justify left)))
+    (property "Reference" "R38" (at 109.22 394.97 0) (effects (font (size 1.27 1.27)) (justify left)))
     (property "Value" "1k 1%" (at 109.22 397.51 0) (effects (font (size 1.27 1.27)) (justify left)))
     (property "Footprint" "" (at 105.41 396.24 0) (effects (font (size 1.27 1.27)) hide))
@@
     (pin "1")
     (pin "2")
-    (instances (project "main-board" (path "/b12a49ac-ffa0-5078-b2ba-e15d161f1936" (reference "R37") (unit 1))))
+    (instances (project "main-board" (path "/b12a49ac-ffa0-5078-b2ba-e15d161f1936" (reference "R38") (unit 1))))
   )
   (symbol (lib_id "Device:R") (at 106.68 426.72 0) (unit 1)
     (in_bom yes) (on_board yes) (dnp no)
-    (property "Reference" "R38" (at 109.22 425.45 0) (effects (font (size 1.27 1.27)) (justify left)))
+    (property "Reference" "R39" (at 109.22 425.45 0) (effects (font (size 1.27 1.27)) (justify left)))
     (property "Value" "1k 1%" (at 109.22 427.99 0) (effects (font (size 1.27 1.27)) (justify left)))
     (property "Footprint" "" (at 105.41 426.72 0) (effects (font (size 1.27 1.27)) hide))
@@
     (pin "1")
     (pin "2")
-    (instances (project "main-board" (path "/b12a49ac-ffa0-5078-b2ba-e15d161f1936" (reference "R38") (unit 1))))
+    (instances (project "main-board" (path "/b12a49ac-ffa0-5078-b2ba-e15d161f1936" (reference "R39") (unit 1))))
   )
   (symbol (lib_id "Device:D_Zener") (at 106.68 457.2 0) (unit 1)
     (in_bom yes) (on_board yes) (dnp no)
-    (property "Reference" "D4" (at 106.68 454.66 0) (effects (font (size 1.27 1.27))))
+    (property "Reference" "D5" (at 106.68 454.66 0) (effects (font (size 1.27 1.27))))
     (property "Value" "PESD12VS1UB or equivalent 12V-standoff ESD diode" (at 106.68 459.74 0) (effects (font (size 1.27 1.27))))
     (property "Footprint" "" (at 106.68 457.2 0) (effects (font (size 1.27 1.27)) hide))
@@
     (pin "1")
     (pin "2")
-    (instances (project "main-board" (path "/b12a49ac-ffa0-5078-b2ba-e15d161f1936" (reference "D4") (unit 1))))
+    (instances (project "main-board" (path "/b12a49ac-ffa0-5078-b2ba-e15d161f1936" (reference "D5") (unit 1))))
   )
   (symbol (lib_id "Device:D_Zener") (at 106.68 487.68 0) (unit 1)
     (in_bom yes) (on_board yes) (dnp no)
-    (property "Reference" "D5" (at 106.68 485.14 0) (effects (font (size 1.27 1.27))))
+    (property "Reference" "D6" (at 106.68 485.14 0) (effects (font (size 1.27 1.27))))
     (property "Value" "PESD12VS1UB or equivalent 12V-standoff ESD diode" (at 106.68 490.22 0) (effects (font (size 1.27 1.27))))
     (property "Footprint" "" (at 106.68 487.68 0) (effects (font (size 1.27 1.27)) hide))
@@
     (pin "1")
     (pin "2")
-    (instances (project "main-board" (path "/b12a49ac-ffa0-5078-b2ba-e15d161f1936" (reference "D5") (unit 1))))
+    (instances (project "main-board" (path "/b12a49ac-ffa0-5078-b2ba-e15d161f1936" (reference "D6") (unit 1))))
   )
   (symbol (lib_id "Connector_Generic:Conn_01x08") (at 106.68 530.86 0) (unit 1)

Commit message: Main board: apply the chosen parts to every symbol and row
Every main-board and adapter symbol now carries Footprint, Manufacturer,
MPN, LCSC and Assembly. The values come from the selections whose
datasheets are banked. The BOM rows follow those choices:

- D-USBOR is the SS14 (SMA).
- J-LED is four solder pads, not a connector.
- L-BUCK-IN is 22 uH, C-BUCK-IN is a UCM electrolytic, C-STRIP-BULK is
  470 uF 25 V.
- D-TVS-BREATH is the PESD12VS1UA (SOD-323); the UB is SOD523.
- J-UMB is the hanxia header. Its posts go through the adapter and its
  tails through the tongue; the old wording had them swapped.
- U-BUCK and U-BREATH say where to buy.
- C-ADC-BULK is 1206 if fitted.

The body and geometry follow the chosen parts:

- The J-UMB and J-MCU envelopes in config/body.yaml are now read off the
  parts' drawings.
- J-MCU is longer, so the regulator block moved and the right-hand ribbon
  header followed it by 1.5 mm. The RH key board is re-laid out, with C8
  moving with the header's 3V3 pin. It checks clean.
- A mount candidate is now nudged by up to 3 mm before it is dropped. All
  seven main-board mounts hold.

New footprints and pages:

- New woody.pretty footprints: the MPXV4006DP (case 1351-01) from
  breath-sense-link.md's land pattern, and the NE8FAV from Neutrik's
  layout, mirrored to the top view.
- The input-LC derivation uses the chosen capacitor's banked ESR: Q is at
  most 1.8, and the margin is 120x worst case.
- The main-board README lists what is still open before layout.

Co-Authored-By: Claude Opus 5.5 <noreply@anthropic.com>
Claude-Session: https://claude.ai/code/session_01LmB4muFXnoLprWX4JzuJ5A
Parts:
- D5, D6: value PESD12VS1UB or equivalent 12V-standoff ESD diode -> PESD12VS1UA or equivalent 12V-standoff ESD diode; footprint (none) -> Diode_SMD:D_SOD-323; Assembly (none) -> machine; LCSC (none) -> C131084; MPN (none) -> PESD12VS1UA,115; Manufacturer (none) -> Nexperia
- FB1, FB2: footprint (none) -> Inductor_SMD:L_0805_2012Metric; Assembly (none) -> machine; LCSC (none) -> C3716677; MPN (none) -> BLM21SP601SN1D; Manufacturer (none) -> Murata
- J4, J5: footprint (none) -> woody:IDC-Header_2x06_P1.27mm_Samtec_SHF_Horizontal; Assembly (none) -> hand; MPN (none) -> SHF-106-01-L-D-RA; Manufacturer (none) -> Samtec
- J6: footprint (none) -> Connector_PinHeader_2.54mm:PinHeader_1x08_P2.54mm_Horizontal; Assembly (none) -> hand; LCSC (none) -> C32713267; MPN (none) -> HX PZ2.54-1x8P WZ; Manufacturer (none) -> hanxia
- R34, R35, R36: footprint (none) -> Resistor_SMD:R_0805_2012Metric; Assembly (none) -> machine; LCSC (none) -> C17408; MPN (none) -> 0805W8F1000T5E; Manufacturer (none) -> UNI-ROYAL
- R37: footprint (none) -> Resistor_SMD:R_0805_2012Metric; Assembly (none) -> machine; LCSC (none) -> C17414; MPN (none) -> 0805W8F1002T5E; Manufacturer (none) -> UNI-ROYAL
- R38, R39: footprint (none) -> Resistor_SMD:R_1206_3216Metric; Assembly (none) -> machine; LCSC (none) -> C4410; MPN (none) -> 1206W4F1001T5E; Manufacturer (none) -> UNI-ROYAL
- U10: footprint (none) -> woody:NXP_Case1351-01_SOP-8_P2.54mm; Assembly (none) -> hand; LCSC (none) -> C5190605; MPN (none) -> MPXV4006DP; Manufacturer (none) -> NXP
- U9: footprint (none) -> Package_TO_SOT_SMD:SOT-23-5; Assembly (none) -> machine; LCSC (none) -> C10675; MPN (none) -> SP0504BAHTG; Manufacturer (none) -> Littelfuse

Commit message: Series resistors on the main board to 1206 1/4 W; fix a render-ledger prefix bug
R-SPI-SER and R-CHAIN-SER (three each) now use UNI-ROYAL 1206W4F1000T5E
(LCSC C17901). A sustained output fault dissipates 109 mW in them. That is
87 % of an 0805's rating and 44 % of this part's. The banked UNI-ROYAL
datasheet covers the 1206 size. The owner approved the change, keeping the
parts surface-mounted.

tools/kicad.py ledger_set matched on a path prefix. Rendering
hardware/carrier therefore dropped the ledger rows of the five circuits
nested under it. It now matches the directory and its fab/ only.

Co-Authored-By: Claude Opus 5.5 <noreply@anthropic.com>
Claude-Session: https://claude.ai/code/session_01LmB4muFXnoLprWX4JzuJ5A
Parts:
- R34, R35, R36: footprint Resistor_SMD:R_0805_2012Metric -> Resistor_SMD:R_1206_3216Metric; LCSC C17408 -> C17901; MPN 0805W8F1000T5E -> 1206W4F1000T5E
Changed lines of the file:
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@@
     (property "Reference" "R34" (at 109.22 151.13 0) (effects (font (size 1.27 1.27)) (justify left)))
     (property "Value" "100R 1%" (at 109.22 153.67 0) (effects (font (size 1.27 1.27)) (justify left)))
-    (property "Footprint" "Resistor_SMD:R_0805_2012Metric" (at 105.41 152.4 0) (effects (font (size 1.27 1.27)) hide))
+    (property "Footprint" "Resistor_SMD:R_1206_3216Metric" (at 105.41 152.4 0) (effects (font (size 1.27 1.27)) hide))
     (property "Datasheet" "" (at 106.68 152.4 0) (effects (font (size 1.27 1.27)) hide))
     (property "Row" "R-CHAIN-SER" (at 106.68 152.4 0) (effects (font (size 1.27 1.27)) hide))
@@
     (property "Note" "At the DRIVING end, where the MCU's pins arrive on the main board" (at 106.68 152.4 0) (effects (font (size 1.27 1.27)) hide))
     (property "Manufacturer" "UNI-ROYAL" (at 106.68 152.4 0) (effects (font (size 1.27 1.27)) hide))
-    (property "MPN" "0805W8F1000T5E" (at 106.68 152.4 0) (effects (font (size 1.27 1.27)) hide))
-    (property "LCSC" "C17408" (at 106.68 152.4 0) (effects (font (size 1.27 1.27)) hide))
+    (property "MPN" "1206W4F1000T5E" (at 106.68 152.4 0) (effects (font (size 1.27 1.27)) hide))
+    (property "LCSC" "C17901" (at 106.68 152.4 0) (effects (font (size 1.27 1.27)) hide))
     (property "Assembly" "machine" (at 106.68 152.4 0) (effects (font (size 1.27 1.27)) hide))
     (pin "1")
@@
     (property "Reference" "R35" (at 109.22 181.61 0) (effects (font (size 1.27 1.27)) (justify left)))
     (property "Value" "100R 1%" (at 109.22 184.15 0) (effects (font (size 1.27 1.27)) (justify left)))
-    (property "Footprint" "Resistor_SMD:R_0805_2012Metric" (at 105.41 182.88 0) (effects (font (size 1.27 1.27)) hide))
+    (property "Footprint" "Resistor_SMD:R_1206_3216Metric" (at 105.41 182.88 0) (effects (font (size 1.27 1.27)) hide))
     (property "Datasheet" "" (at 106.68 182.88 0) (effects (font (size 1.27 1.27)) hide))
     (property "Row" "R-CHAIN-SER" (at 106.68 182.88 0) (effects (font (size 1.27 1.27)) hide))
     (property "Pins" "1=1 2=2" (at 106.68 182.88 0) (effects (font (size 1.27 1.27)) hide))
     (property "Manufacturer" "UNI-ROYAL" (at 106.68 182.88 0) (effects (font (size 1.27 1.27)) hide))
-    (property "MPN" "0805W8F1000T5E" (at 106.68 182.88 0) (effects (font (size 1.27 1.27)) hide))
-    (property "LCSC" "C17408" (at 106.68 182.88 0) (effects (font (size 1.27 1.27)) hide))
+    (property "MPN" "1206W4F1000T5E" (at 106.68 182.88 0) (effects (font (size 1.27 1.27)) hide))
+    (property "LCSC" "C17901" (at 106.68 182.88 0) (effects (font (size 1.27 1.27)) hide))
     (property "Assembly" "machine" (at 106.68 182.88 0) (effects (font (size 1.27 1.27)) hide))
     (pin "1")
@@
     (property "Reference" "R36" (at 109.22 212.09 0) (effects (font (size 1.27 1.27)) (justify left)))
     (property "Value" "100R 1%" (at 109.22 214.63 0) (effects (font (size 1.27 1.27)) (justify left)))
-    (property "Footprint" "Resistor_SMD:R_0805_2012Metric" (at 105.41 213.36 0) (effects (font (size 1.27 1.27)) hide))
+    (property "Footprint" "Resistor_SMD:R_1206_3216Metric" (at 105.41 213.36 0) (effects (font (size 1.27 1.27)) hide))
     (property "Datasheet" "" (at 106.68 213.36 0) (effects (font (size 1.27 1.27)) hide))
     (property "Row" "R-CHAIN-SER" (at 106.68 213.36 0) (effects (font (size 1.27 1.27)) hide))
     (property "Pins" "1=1 2=2" (at 106.68 213.36 0) (effects (font (size 1.27 1.27)) hide))
     (property "Manufacturer" "UNI-ROYAL" (at 106.68 213.36 0) (effects (font (size 1.27 1.27)) hide))
-    (property "MPN" "0805W8F1000T5E" (at 106.68 213.36 0) (effects (font (size 1.27 1.27)) hide))
-    (property "LCSC" "C17408" (at 106.68 213.36 0) (effects (font (size 1.27 1.27)) hide))
+    (property "MPN" "1206W4F1000T5E" (at 106.68 213.36 0) (effects (font (size 1.27 1.27)) hide))
+    (property "LCSC" "C17901" (at 106.68 213.36 0) (effects (font (size 1.27 1.27)) hide))
     (property "Assembly" "machine" (at 106.68 213.36 0) (effects (font (size 1.27 1.27)) hide))
     (pin "1")
