File: hardware/boards/main-board/main-board.cold.kicad_pcb (KiCad board)
At the start: 4 copper layers, 292.4 x 42 mm, 170 parts, among them J1 2x12 1.27mm shrouded box head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, J2 1x3, J4 12-way, J5 12-way, J6 8-way 2.54mm right-angle pin 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, J7 S3B-PH-SM4-TB, Q1 AO3401A, Q2 DMN3404L, SW1 KS-33, SW2 KS-33, SW3 KS-33, SW4 KS-33, SW5 KS-33, SW6 KS-33, SW7 KS-33, SW8 KS-33, U1 SP0504BAHT or equivalent 4-ch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, U10 MPXV4006DP, U11 SP0504BAHTG 4-channel 5V array, U12 SP0504BAHTG, U13 LM74700-Q1, U2 MCP3202-CI/SN, U3 OPA2197IDR, U4 REF5050IDR, U5 R-78E5.0-1.0, U6 74AHCT125, U7 74HCS165, U8 74HCS165, U9 SP0504BAHTG 4-channel 5V array

Commit message: #46: main-board cold placement checkpoint at 8f7a4121 (placed, not routed)
The placement cold_trial.py --place-only writes at 8f7a4121: no airwire
regressions over the source, check_cad clean, KiCad placement findings none.
The staged routing run (run 3) writes over it when it ends.

Gate-Red: check-staleness 15 cad + 1 sim and kicad.py check 140 (module-main and module sheets) - the same pre-existing failures as 8f7a4121; this commit changes a scratch trial board only; module work is set aside by the owner

Co-Authored-By: Claude Opus 5.5 <noreply@anthropic.com>
Claude-Session: https://claude.ai/code/session_01EojKhSrbGL29aV6hSDYnh2
Parts:
- moved R36 165.1 mm to (297.2, 133.7), turned to 180 degrees
- moved R35 162.3 mm to (297.2, 140.0), turned to 180 degrees
- moved R34 158.9 mm to (297.2, 136.8), turned to 180 degrees
- moved R44 97.5 mm to (139.1, 122.5), turned to 90 degrees
- moved C11 46.5 mm to (293.5, 114.2), turned to 180 degrees
- moved R43 44.5 mm to (333.9, 109.0), turned to -90 degrees
- moved R29 29.1 mm to (236.1, 106.1), turned to 90 degrees
- moved R32 27.3 mm to (139.1, 137.7)
- moved D21 25.6 mm to (340.4, 118.2)
- moved FB1 24.5 mm to (142.9, 102.0), turned to 180 degrees
- moved R42 21.5 mm to (340.4, 125.8), turned to 90 degrees
- moved C13 20.5 mm to (139.2, 130.1)
- moved C40 19.8 mm to (340.4, 122.0)
- moved R33 19.2 mm to (139.2, 133.9)
- moved C206 18.6 mm to (139.1, 126.3)
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Routing:
- net /IO39: track 0.00 -> 167.6 mm, vias 0 -> 4
- net /CHAIN_SHLD: track 167.6 -> 0.00 mm, vias 4 -> 0
- net /IO35: track 150.6 -> 105.3 mm, vias 3 -> 2
- net /power-entry-instrument/USBOR_VCAP: track 0.00 -> 45.3 mm, vias 0 -> 1
Other:
- board text added: "C13"
- board text added: "C40"
- board text added: "C46"
- board text added: "C47"
- board text added: "D2"
- board text added: "D21"
- board text added: "R19"
- board text added: "R40"
- board text added: "R41"
- board text removed: "C35"
- board text removed: "U11"

Commit message: #46: chain family review - a placement on kept copper, and a pin on a moat
Review of the main board's family 3 (chain): CHAIN_SCK and CHAIN_SHLD open.
Traced to three defects, none of them the chain's routing:

1. The cold placement seated U8 on a kept IO39 hand route (a locked route
   between fixed parts): pin 1, CHAIN_SHLD, shorted to it - unreachable. KiCad
   on the placed board: 6 shorts, 5 clearance, 3 hole clearance, 7 mask
   bridges over U8, C24, U6, R37. The packer knew courtyards, not copper.
   pcb_pack: Board.wires (the board's tracks and vias), Part.padgeo, rule
   `wires` - no pad within clearance of another net's copper; in seat_ok and
   RULES. Bench cell `wires` (proved to short without the rule). cold_trial's
   placement gate now refuses any KiCad short, clearance, hole-clearance,
   mask-bridge or crossing finding (it checked courtyards and keep-outs only).
   Re-placed: KiCad placement findings none; airwires 3691 mm vs 3604.
2. Router.open_pad opened a blocked pad's centre cell on every layer, a
   keep-out's layer included. Now not on a layer where a no-tracks keep-out or
   another net's reservation covers the pad.
3. The stub from a pad's centre to the path's first cell crossed a keep-out
   the cell itself was clear of (J5 pin 2, half on the AGND strip's moat on
   B.Cu): the lay refused it, through push and rescue alike. A stub across a
   hard area is dropped - the run starts at the cell, inside the pad's copper.
   Bench cell `moatpin`: fails without the fix exactly as the main board did.
   CHAIN_SCK alone on the old checkpoint: routed, 191 mm, 4 vias (source 255,
   10).

The U13 `connect` edit loses its board-millimetre points: U13 moved 0.25 mm in
the re-placement and the points went stale; at signal width the way under the
body is the shortest anyway. Route2 bench 38/38, pack bench 14/14: PASS.

main-board.cold.kicad_pcb: the new placement (placed, not routed).

Gate-Red: check-staleness 15 cad + 1 sim and kicad.py check 140 (modu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
Parts:
- moved R32 29.9 mm to (169.0, 136.1)
- moved R33 29.9 mm to (169.0, 132.3)
- moved R44 29.9 mm to (169.0, 120.9)
- moved C13 29.9 mm to (169.0, 128.5)
- moved C206 29.9 mm to (169.0, 124.7)
- moved U7 18.2 mm to (151.8, 119.5)
- moved C207 15.0 mm to (309.4, 127.5)
- moved U9 11.4 mm to (132.8, 118.0)
- moved C208 10.6 mm to (288.1, 127.1), turned to 90 degrees
- moved FB1 9.50 mm to (142.9, 111.5)
- moved R29 6.10 mm to (236.1, 112.2)
- moved R31 5.30 mm to (236.1, 104.6)
- moved R30 5.30 mm to (236.1, 108.4)
- moved U6 2.26 mm to (304.3, 131.1)
- moved C15 1.75 mm to (119.5, 130.2)
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Routing:
- net PWR_GND: track 106.1 -> 42.0 mm, vias 40 -> 38
- net /CHAIN_SER_LH: track 0.00 -> 64.1 mm, vias 0 -> 2
- net /IO35: track 105.3 -> 150.6 mm, vias 2 -> 3
- net /power-entry-instrument/USBOR_VCAP: track 45.3 -> 0.00 mm, vias 1 -> 0
Other:
- board text added: "C35"
- board text removed: "R19"
- board text removed: "U1"

Commit message: #46: a part on a net private to its IC is seated at it; reviews can accept
Review of the re-placed power family: BUCK_A_OUT 35 -> 91 mm. C207 (C-USBOR,
U13's VCAP cap - USBOR_VCAP joins only C207 and U13) had been packed in one row
with C208 round U13, and the row fitted 11 mm off. pcb_pack cold(): a passive
whose every signal net (power nets aside) is private to one seated part is
seated alone, round that part, before any group row. Re-placed: C207 6.5 mm
from U13 pin 1 (U6's pin column stands beside U13), and FB1, FB2, R32, R33,
R43 seated alone at theirs; airwires 3691 -> 3651 mm (source 3604); KiCad
placement findings none. Pack bench: PASS.

Router.stage(accept=): review reasons a reviewer already accepted are recorded
in the family's `accepted`, not paused for. cold_trial ACCEPT, each with why:
V3V3_CHAIN_RH's 9.6 mm round J5's end (accepted 2026-10-10).

main-board.cold.kicad_pcb: this placement (placed, not routed).

Gate-Red: check-staleness 15 cad + 1 sim and kicad.py check 140 (module-main and module sheets) - the same pre-existing failures as de765277, none in a file this commit touches; module work is set aside by the owner

Co-Authored-By: Claude Opus 5.5 <noreply@anthropic.com>
Claude-Session: https://claude.ai/code/session_01EojKhSrbGL29aV6hSDYnh2
Parts:
- moved R36 20.3 mm to (315.9, 125.8), turned to 90 degrees
- moved R34 19.0 mm to (312.8, 125.8), turned to 90 degrees
- moved R35 18.8 mm to (309.6, 125.8), turned to 90 degrees
- moved R32 14.4 mm to (157.2, 127.8)
- moved R33 14.3 mm to (157.0, 124.5), turned to 90 degrees
- moved C207 11.8 mm to (297.7, 129.0), turned to 0 degrees
- moved C208 11.3 mm to (297.8, 133.0), turned to 0 degrees
- moved U13 7.58 mm to (291.4, 127.0), turned to 90 degrees
- moved R44 7.11 mm to (163.5, 125.4), turned to 0 degrees
- moved C206 6.55 mm to (163.5, 128.2), turned to 0 degrees
- moved C13 6.08 mm to (163.5, 131.1), turned to 0 degrees
- moved C12 5.58 mm to (309.6, 120.2), turned to 90 degrees
- moved Q2 5.34 mm to (294.7, 131.0), turned to 0 degrees
- moved R51 5.24 mm to (312.2, 120.2), turned to 90 degrees
- moved R50 4.38 mm to (317.6, 120.2), turned to 90 degrees
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Other:
- board text added: "U1"

Commit message: #46: main board cold trial - families 1-3 (power, analog, chain) routed and reviewed
main-board.cold.kicad_pcb: checkpoint 3 of cold_trial.py at e8ccbfc9 - the
placement there, then power, analog and chain, each paused and reviewed, with
the recorded EDITS (2) and ACCEPT (1). 13 min for the three.

Every net of the three families routed; none open, none pushed, no review
reason left. KiCad DRC on the checkpoint: 0 errors (126 unconnected: families
4-7, not routed).

Against the source: chain 969.7 mm / 31 vias (source 1000.6 / 33) - CHAIN_SCK
225.4 / 5 (254.6 / 10), CHAIN_SHLD 226.6 / 9 (272.3 / 9), CHAIN_QH_RT 90.3 / 0
(87.8 / 4); power - DEV_3V3 457.6 / 6 (493.7 / 16), INST_5V_A 69.3 / 0
(81.0 / 5), BUCK_A_OUT 54.4 (28.5) and BUCK_IN 51.4 (28.0), the buck corner's
placement; analog 118.2 mm / 2 vias.

Open, for the finish or a later review: pcb.check_tracks finds 5 acid traps
(four 0-degree overlaps of new copper on kept or pad copper, SENSOR_RAW and
BUCK_IN; one 45-degree join, DEV_3V3) - pcb_route.tidy runs only after the last
family, so they are checked on the finished board, not counted fixed; and
HOP_LT_QH 9.0 mm / 2 vias for the source's 1.0 - R44 (R-HOP-SER) seated
8.4 mm off U7's QH, a placement nit.

Gate-Red: check-staleness 15 cad + 1 sim and kicad.py check 140 (module-main and module sheets) - the same pre-existing failures as e8ccbfc9; this commit changes a scratch trial board only; module work is set aside by the owner

Co-Authored-By: Claude Opus 5.5 <noreply@anthropic.com>
Claude-Session: https://claude.ai/code/session_01EojKhSrbGL29aV6hSDYnh2
Routing:
- net DEV_3V3: track 60.3 -> 457.6 mm, vias 1 -> 6
- net /CHAIN_SHLD: track 0.00 -> 226.6 mm, vias 0 -> 9
- net /CHAIN_SCK: track 13.6 -> 225.4 mm, vias 1 -> 5
- net /CHAIN_SER_LH: track 64.1 -> 225.4 mm, vias 2 -> 4
- net /HOP_LT_RH: track 0.00 -> 130.6 mm, vias 0 -> 7
- net /CHAIN_QH_RT: track 1.70 -> 90.3 mm
- net PWR_GND: track 42.0 -> 100.0 mm, vias 38 -> 84
- net INST_5V_A: track 12.4 -> 69.3 mm
- net /power-entry-instrument/BUCK_A_OUT: track 0.00 -> 54.4 mm
- net BUCK_IN: track 7.85 -> 51.4 mm
- net VS: track 19.5 -> 51.7 mm, vias 2 -> 4
- net /HOP_LH_LT: track 0.00 -> 29.7 mm, vias 0 -> 2
- net UMBILICAL_POS12: track 0.00 -> 29.0 mm
- net /HOP_RH_RT: track 7.43 -> 32.6 mm, vias 0 -> 2
- net REF_VIN: track 0.00 -> 24.1 mm
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
Commit message: #46: the tools read a board in an order of their own - a resumed run was a coin toss
The route2 bench's `resume` cell failed after 92b6af8f - and, bisecting, at
the commit before it too, and passed under some runs and not others: it was
never deterministic. The router and packer read tracks, footprints and zones
in KiCad's order, which follows the items' random ids; every run writes new
ids, so a checkpoint read back by the next run fed the index another order,
and every tie broken by it another answer - one stopped-and-resumed run in
about three laid other copper than one run (the hash seed was a red herring:
fixed seeds passed and failed alike). model_from_board and pcb_pack.board_of
now sort footprints (by reference), zones and tracks (by geometry) first. The
cell then passed four runs of four.

nonplanar cell: "no path" is now either the exhausted search ("none") or the
walled-in proof ("walled: ..."); it accepts both.

main-board.cold.kicad_pcb: the re-placement at 92b6af8f (placed, not routed):
every series termination seated alone at its driver; airwires 3605 mm vs the
source's 3604; KiCad placement findings none.

The full route2 and pack benches are running at this commit; their result
goes in the next.

Gate-Red: check-staleness 15 cad + 1 sim and kicad.py check 140 (module-main and module sheets) - the same pre-existing failures as 92b6af8f, none in a file this commit touches; module work is set aside by the owner

Co-Authored-By: Claude Opus 5.5 <noreply@anthropic.com>
Claude-Session: https://claude.ai/code/session_01EojKhSrbGL29aV6hSDYnh2
Parts:
- moved R30 25.4 mm to (247.1, 131.3)
- moved R31 25.1 mm to (246.6, 127.4)
- moved R36 22.8 mm to (297.4, 139.1), turned to 180 degrees
- moved R42 20.0 mm to (358.6, 134.1)
- moved R29 17.2 mm to (244.1, 127.4)
- moved R34 16.8 mm to (295.9, 127.1), turned to 180 degrees
- moved R35 16.1 mm to (297.4, 136.3), turned to 180 degrees
- moved C13 15.6 mm to (157.0, 116.8), turned to 90 degrees
- moved C24 13.6 mm to (243.3, 131.3)
- moved C40 12.8 mm to (348.7, 131.8), turned to 180 degrees
- moved R28 11.8 mm to (235.1, 127.8), turned to 0 degrees
- moved C207 11.7 mm to (308.1, 123.7), turned to -90 degrees
- moved C208 11.3 mm to (288.1, 127.1), turned to 90 degrees
- moved R1 11.2 mm to (339.1, 123.1)
- moved D21 11.2 mm to (337.4, 129.1)
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Routing:
- net DEV_3V3: track 457.6 -> 60.3 mm, vias 6 -> 1
- net /CHAIN_SHLD: track 226.6 -> 0.00 mm, vias 9 -> 0
- net /CHAIN_SCK: track 225.4 -> 13.6 mm, vias 5 -> 1
- net /CHAIN_SER_LH: track 225.4 -> 64.1 mm, vias 4 -> 2
- net /HOP_LT_RH: track 130.6 -> 0.00 mm, vias 7 -> 0
- net /CHAIN_QH_RT: track 90.3 -> 1.70 mm
- net PWR_GND: track 100.0 -> 42.0 mm, vias 84 -> 38
- net INST_5V_A: track 69.3 -> 12.4 mm
- net /power-entry-instrument/BUCK_A_OUT: track 54.4 -> 0.00 mm
- net BUCK_IN: track 51.4 -> 7.85 mm
- net VS: track 51.7 -> 19.5 mm, vias 4 -> 2
- net /HOP_LH_LT: track 29.7 -> 0.00 mm, vias 2 -> 0
- net UMBILICAL_POS12: track 29.0 -> 0.00 mm
- net /HOP_RH_RT: track 32.6 -> 7.43 mm, vias 2 -> 0
- net REF_VIN: track 24.1 -> 0.00 mm
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Other:
- board text added: "U11"
- board text removed: "C24"
- board text removed: "D2"
- board text removed: "R29"
- board text removed: "R33"
- board text removed: "R44"
- board text removed: "U1"

Commit message: #46: main board cold trial - families 1-4 routed whole; keys reviewed
At baedf9e3, re-placed with the pin rows' room (airwires 3597 mm, the
source's 3604; KiCad placement findings none) and routed in 21 min:
power 624.8 mm / 9 vias, analog 120.5 / 2, chain 854.5 / 31, keys 445.7 /
44 - every net of the four routed, none open, none pushed. The escape bands
and the pin rows' room did what U8 pins 14 and 5 and R33 needed.

Keys paused for two "still long", reviewed and recorded in ACCEPT with why:
KEY_FREE2 9.1 mm (the source's 10.5); LT4/SWITCH_LEG 20.3 mm / 2 vias for an
8.9 mm airwire - H3's bearing keep-out between SW4 and R19, CHAIN_SER_LH
hugging its top 0.5 mm off. A chain-family `clear` would open a lane; left
for the whole board's review with the keys' total, 445.7 mm / 44 vias against
the source's 365.7 / 22 - a placement question (the key networks round their
switches), not this one line.

main-board.cold.kicad_pcb: checkpoint 4. Families 5-7 are routing.

Gate-Red: check-staleness 15 cad + 1 sim and kicad.py check 140 (module-main and module sheets) - the same pre-existing failures as baedf9e3; this commit changes the trial's review record and a scratch trial board only; module work is set aside by the owner

Co-Authored-By: Claude Opus 5.5 <noreply@anthropic.com>
Claude-Session: https://claude.ai/code/session_01EojKhSrbGL29aV6hSDYnh2
Parts:
- moved R36 19.0 mm to (309.2, 124.2)
- moved C207 13.5 mm to (295.2, 127.8), turned to 0 degrees
- moved C208 10.3 mm to (297.8, 123.5)
- moved R34 9.03 mm to (296.7, 136.1)
- moved U13 7.58 mm to (291.4, 127.0), turned to 90 degrees
- moved Q2 5.34 mm to (294.7, 131.0), turned to 0 degrees
- moved R35 2.50 mm to (297.4, 138.8)
- moved U11 2.50 mm to (236.7, 106.7)
- moved FB1 1.27 mm to (144.2, 111.7)
- moved C13 1.25 mm to (158.3, 116.8)
- moved C206 1.25 mm to (158.3, 120.7)
- moved FB2 1.25 mm to (238.8, 111.0)
- moved R33 1.25 mm to (158.2, 124.5)
- moved R44 1.25 mm to (161.3, 125.5)
Routing:
- net DEV_3V3: track 60.3 -> 479.9 mm, vias 1 -> 8
- net /CHAIN_SCK: track 13.6 -> 236.6 mm, vias 1 -> 5
- net /CHAIN_SHLD: track 0.00 -> 221.1 mm, vias 0 -> 10
- net /CHAIN_SER_LH: track 64.1 -> 218.0 mm, vias 2 -> 8
- net /HOP_LT_RH: track 0.00 -> 100.7 mm, vias 0 -> 4
- net /CHAIN_QH_RT: track 1.70 -> 80.3 mm, vias 0 -> 1
- net INST_5V_A: track 12.4 -> 77.5 mm
- net PWR_GND: track 42.0 -> 98.8 mm, vias 38 -> 84
- net /KEY_RT2: track 0.00 -> 48.2 mm, vias 0 -> 6
- net /KEY_LT1: track 0.00 -> 43.8 mm, vias 0 -> 4
- net BUCK_IN: track 7.85 -> 51.4 mm
- net /KEY_LT2: track 0.00 -> 43.1 mm, vias 0 -> 4
- net /KEY_RT1: track 0.00 -> 40.4 mm, vias 0 -> 4
- net /power-entry-instrument/BUCK_A_OUT: track 0.00 -> 37.4 mm, vias 0 -> 2
- net UMBILICAL_POS12: track 0.00 -> 36.0 mm
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Other:
- board text added: "R44"
