File: hardware/carrier/carrier.kicad_sch (KiCad schematic)
At the start: 7 parts

Commit message: Main board: apply the chosen parts to every symbol and row
Every main-board and adapter symbol now carries Footprint, Manufacturer,
MPN, LCSC and Assembly. The values come from the selections whose
datasheets are banked. The BOM rows follow those choices:

- D-USBOR is the SS14 (SMA).
- J-LED is four solder pads, not a connector.
- L-BUCK-IN is 22 uH, C-BUCK-IN is a UCM electrolytic, C-STRIP-BULK is
  470 uF 25 V.
- D-TVS-BREATH is the PESD12VS1UA (SOD-323); the UB is SOD523.
- J-UMB is the hanxia header. Its posts go through the adapter and its
  tails through the tongue; the old wording had them swapped.
- U-BUCK and U-BREATH say where to buy.
- C-ADC-BULK is 1206 if fitted.

The body and geometry follow the chosen parts:

- The J-UMB and J-MCU envelopes in config/body.yaml are now read off the
  parts' drawings.
- J-MCU is longer, so the regulator block moved and the right-hand ribbon
  header followed it by 1.5 mm. The RH key board is re-laid out, with C8
  moving with the header's 3V3 pin. It checks clean.
- A mount candidate is now nudged by up to 3 mm before it is dropped. All
  seven main-board mounts hold.

New footprints and pages:

- New woody.pretty footprints: the MPXV4006DP (case 1351-01) from
  breath-sense-link.md's land pattern, and the NE8FAV from Neutrik's
  layout, mirrored to the top view.
- The input-LC derivation uses the chosen capacitor's banked ESR: Q is at
  most 1.8, and the margin is 120x worst case.
- The main-board README lists what is still open before layout.

Co-Authored-By: Claude Opus 5.5 <noreply@anthropic.com>
Claude-Session: https://claude.ai/code/session_01LmB4muFXnoLprWX4JzuJ5A
Parts:
- J-MCU: footprint (none) -> Connector_PinHeader_1.27mm:PinHeader_2x12_P1.27mm_Horizontal; Assembly (none) -> hand; LCSC (none) -> C5147255; MPN (none) -> X1270WR-2x12A-9TV01; Manufacturer (none) -> XKB Connection
- NT-DIG: footprint (none) -> NetTie:NetTie-2_SMD_Pad2.0mm; Assembly (none) -> none
- R-SPI-SER-CS, R-SPI-SER-MOSI, R-SPI-SER-SCLK: footprint (none) -> Resistor_SMD:R_0805_2012Metric; Assembly (none) -> machine; LCSC (none) -> C17408; MPN (none) -> 0805W8F1000T5E; Manufacturer (none) -> UNI-ROYAL
- U-TVS-SPI: footprint (none) -> Package_TO_SOT_SMD:SOT-23-5; Assembly (none) -> machine; LCSC (none) -> C10675; MPN (none) -> SP0504BAHTG; Manufacturer (none) -> Littelfuse
Changed lines of the file:
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@@
     (property "Reference" "J-MCU" (at 41.91 137.16 0) (effects (font (size 1.27 1.27))))
     (property "Value" "2x12 1.27mm shrouded box header" (at 41.91 170.18 0) (effects (font (size 1.27 1.27))))
-    (property "Footprint" "" (at 40.64 152.4 0) (effects (font (size 1.27 1.27)) hide))
+    (property "Footprint" "Connector_PinHeader_1.27mm:PinHeader_2x12_P1.27mm_Horizontal" (at 40.64 152.4 0) (effects (font (size 1.27 1.27)) hide))
     (property "Datasheet" "" (at 40.64 152.4 0) (effects (font (size 1.27 1.27)) hide))
     (property "Row" "J-MCU" (at 40.64 152.4 0) (effects (font (size 1.27 1.27)) hide))
@@
     (property "Note" "The Matrix's ribbon lands here, conductor n on pin n (ADR 0018). Every fast line has a ground, a supply or a static line on both sides, and pin 9 (GND) separates SCLK (pin 10) from the chain clock (pin 8)" (at 40.64 152.4 0) (effects (font (size 1.27 1.27)) hide))
     (property "Pins_source" "ribbon conductor n on pin n (ADR 0018); odd/even across the two rows as a 2x12 IDC header numbers them" (at 40.64 152.4 0) (effects (font (size 1.27 1.27)) hide))
+    (property "Manufacturer" "XKB Connection" (at 40.64 152.4 0) (effects (font (size 1.27 1.27)) hide))
+    (property "MPN" "X1270WR-2x12A-9TV01" (at 40.64 152.4 0) (effects (font (size 1.27 1.27)) hide))
+    (property "LCSC" "C5147255" (at 40.64 152.4 0) (effects (font (size 1.27 1.27)) hide))
+    (property "Assembly" "hand" (at 40.64 152.4 0) (effects (font (size 1.27 1.27)) hide))
     (pin "1")
     (pin "10")
@@
     (property "Reference" "R-SPI-SER-SCLK" (at 43.18 232.41 0) (effects (font (size 1.27 1.27)) (justify left)))
     (property "Value" "100R 1%" (at 43.18 234.95 0) (effects (font (size 1.27 1.27)) (justify left)))
-    (property "Footprint" "" (at 39.37 233.68 0) (effects (font (size 1.27 1.27)) hide))
+    (property "Footprint" "Resistor_SMD:R_0805_2012Metric" (at 39.37 233.68 0) (effects (font (size 1.27 1.27)) hide))
     (property "Datasheet" "" (at 40.64 233.68 0) (effects (font (size 1.27 1.27)) hide))
     (property "Row" "R-SPI-SER" (at 40.64 233.68 0) (effects (font (size 1.27 1.27)) hide))
@@
     (property "Drawn_as" "R-SPI-SER" (at 40.64 233.68 0) (effects (font (size 1.27 1.27)) hide))
     (property "Note" "At the DRIVING end, which is this board. The far end's threshold is the 74AHCT125's TTL V_IH, not a ratio of its rail" (at 40.64 233.68 0) (effects (font (size 1.27 1.27)) hide))
+    (property "Manufacturer" "UNI-ROYAL" (at 40.64 233.68 0) (effects (font (size 1.27 1.27)) hide))
+    (property "MPN" "0805W8F1000T5E" (at 40.64 233.68 0) (effects (font (size 1.27 1.27)) hide))
+    (property "LCSC" "C17408" (at 40.64 233.68 0) (effects (font (size 1.27 1.27)) hide))
+    (property "Assembly" "machine" (at 40.64 233.68 0) (effects (font (size 1.27 1.27)) hide))
     (pin "1")
     (pin "2")
@@
     (property "Reference" "R-SPI-SER-MOSI" (at 93.98 232.41 0) (effects (font (size 1.27 1.27)) (justify left)))
     (property "Value" "100R 1%" (at 93.98 234.95 0) (effects (font (size 1.27 1.27)) (justify left)))
-    (property "Footprint" "" (at 90.17 233.68 0) (effects (font (size 1.27 1.27)) hide))
+    (property "Footprint" "Resistor_SMD:R_0805_2012Metric" (at 90.17 233.68 0) (effects (font (size 1.27 1.27)) hide))
     (property "Datasheet" "" (at 91.44 233.68 0) (effects (font (size 1.27 1.27)) hide))
     (property "Row" "R-SPI-SER" (at 91.44 233.68 0) (effects (font (size 1.27 1.27)) hide))
     (property "Pins" "1=1 2=2" (at 91.44 233.68 0) (effects (font (size 1.27 1.27)) hide))
+    (property "Manufacturer" "UNI-ROYAL" (at 91.44 233.68 0) (effects (font (size 1.27 1.27)) hide))
+    (property "MPN" "0805W8F1000T5E" (at 91.44 233.68 0) (effects (font (size 1.27 1.27)) hide))
+    (property "LCSC" "C17408" (at 91.44 233.68 0) (effects (font (size 1.27 1.27)) hide))
+    (property "Assembly" "machine" (at 91.44 233.68 0) (effects (font (size 1.27 1.27)) hide))
     (pin "1")
     (pin "2")
@@
     (property "Reference" "R-SPI-SER-CS" (at 144.78 232.41 0) (effects (font (size 1.27 1.27)) (justify left)))
     (property "Value" "100R 1%" (at 144.78 234.95 0) (effects (font (size 1.27 1.27)) (justify left)))
-    (property "Footprint" "" (at 140.97 233.68 0) (effects (font (size 1.27 1.27)) hide))
+    (property "Footprint" "Resistor_SMD:R_0805_2012Metric" (at 140.97 233.68 0) (effects (font (size 1.27 1.27)) hide))
     (property "Datasheet" "" (at 142.24 233.68 0) (effects (font (size 1.27 1.27)) hide))
     (property "Row" "R-SPI-SER" (at 142.24 233.68 0) (effects (font (size 1.27 1.27)) hide))
     (property "Pins" "1=1 2=2" (at 142.24 233.68 0) (effects (font (size 1.27 1.27)) hide))
+    (property "Manufacturer" "UNI-ROYAL" (at 142.24 233.68 0) (effects (font (size 1.27 1.27)) hide))
+    (property "MPN" "0805W8F1000T5E" (at 142.24 233.68 0) (effects (font (size 1.27 1.27)) hide))
+    (property "LCSC" "C17408" (at 142.24 233.68 0) (effects (font (size 1.27 1.27)) hide))
+    (property "Assembly" "machine" (at 142.24 233.68 0) (effects (font (size 1.27 1.27)) hide))
     (pin "1")
     (pin "2")
@@
     (property "Reference" "NT-DIG" (at 193.04 231.14 0) (effects (font (size 1.27 1.27))))
     (property "Value" "net tie" (at 193.04 236.22 0) (effects (font (size 1.27 1.27))))
-    (property "Footprint" "" (at 193.04 233.68 0) (effects (font (size 1.27 1.27)) hide))
+    (property "Footprint" "NetTie:NetTie-2_SMD_Pad2.0mm" (at 193.04 233.68 0) (effects (font (size 1.27 1.27)) hide))
     (property "Datasheet" "" (at 193.04 233.68 0) (effects (font (size 1.27 1.27)) hide))
     (property "Row" "NT-DIG" (at 193.04 233.68 0) (effects (font (size 1.27 1.27)) hide))
@@
     (property "Note" "DIG_GND (J-UMB pin 8) to this board's ground, at the pin: copper only (ADR 0018)" (at 193.04 233.68 0) (effects (font (size 1.27 1.27)) hide))
     (property "Pins_source" "a net tie's two pads: 1 J-UMB pin 8's DIG_GND, 2 PWR_GND" (at 193.04 233.68 0) (effects (font (size 1.27 1.27)) hide))
+    (property "Manufacturer" "" (at 193.04 233.68 0) (effects (font (size 1.27 1.27)) hide))
+    (property "MPN" "" (at 193.04 233.68 0) (effects (font (size 1.27 1.27)) hide))
+    (property "LCSC" "" (at 193.04 233.68 0) (effects (font (size 1.27 1.27)) hide))
+    (property "Assembly" "none" (at 193.04 233.68 0) (effects (font (size 1.27 1.27)) hide))
     (pin "1")
     (pin "2")
@@
     (property "Reference" "U-TVS-SPI" (at 48.26 276.86 0) (effects (font (size 1.27 1.27))))
     (property "Value" "SP0504BAHT or equivalent 4-channel 5V array" (at 48.26 279.4 0) (effects (font (size 1.27 1.27))))
-    (property "Footprint" "" (at 48.26 280.67 0) (effects (font (size 1.27 1.27)) hide))
+    (property "Footprint" "Package_TO_SOT_SMD:SOT-23-5" (at 48.26 280.67 0) (effects (font (size 1.27 1.27)) hide))
     (property "Datasheet" "" (at 43.18 275.59 0) (effects (font (size 1.27 1.27)) hide))
     (property "Row" "U-TVS-SPI" (at 40.64 279.4 0) (effects (font (size 1.27 1.27)) hide))
@@
     (property "Note" "On the umbilical side of the series resistors, where the cable's energy arrives" (at 40.64 279.4 0) (effects (font (size 1.27 1.27)) hide))
     (property "Pins_source" "datasheets/discrete-and-power/SP0504BAHT.pdf p.1 pinout (SOT-23-5): I/O on 1, 3, 4, 5, ground on 2" (at 40.64 279.4 0) (effects (font (size 1.27 1.27)) hide))
+    (property "Manufacturer" "Littelfuse" (at 40.64 279.4 0) (effects (font (size 1.27 1.27)) hide))
+    (property "MPN" "SP0504BAHTG" (at 40.64 279.4 0) (effects (font (size 1.27 1.27)) hide))
+    (property "LCSC" "C10675" (at 40.64 279.4 0) (effects (font (size 1.27 1.27)) hide))
+    (property "Assembly" "machine" (at 40.64 279.4 0) (effects (font (size 1.27 1.27)) hide))
     (pin "2")
     (pin "1")

Commit message: Series resistors on the main board to 1206 1/4 W; fix a render-ledger prefix bug
R-SPI-SER and R-CHAIN-SER (three each) now use UNI-ROYAL 1206W4F1000T5E
(LCSC C17901). A sustained output fault dissipates 109 mW in them. That is
87 % of an 0805's rating and 44 % of this part's. The banked UNI-ROYAL
datasheet covers the 1206 size. The owner approved the change, keeping the
parts surface-mounted.

tools/kicad.py ledger_set matched on a path prefix. Rendering
hardware/carrier therefore dropped the ledger rows of the five circuits
nested under it. It now matches the directory and its fab/ only.

Co-Authored-By: Claude Opus 5.5 <noreply@anthropic.com>
Claude-Session: https://claude.ai/code/session_01LmB4muFXnoLprWX4JzuJ5A
Parts:
- R-SPI-SER-CS, R-SPI-SER-MOSI, R-SPI-SER-SCLK: footprint Resistor_SMD:R_0805_2012Metric -> Resistor_SMD:R_1206_3216Metric; LCSC C17408 -> C17901; MPN 0805W8F1000T5E -> 1206W4F1000T5E
Changed lines of the file:
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@@
     (property "Reference" "R-SPI-SER-SCLK" (at 43.18 232.41 0) (effects (font (size 1.27 1.27)) (justify left)))
     (property "Value" "100R 1%" (at 43.18 234.95 0) (effects (font (size 1.27 1.27)) (justify left)))
-    (property "Footprint" "Resistor_SMD:R_0805_2012Metric" (at 39.37 233.68 0) (effects (font (size 1.27 1.27)) hide))
+    (property "Footprint" "Resistor_SMD:R_1206_3216Metric" (at 39.37 233.68 0) (effects (font (size 1.27 1.27)) hide))
     (property "Datasheet" "" (at 40.64 233.68 0) (effects (font (size 1.27 1.27)) hide))
     (property "Row" "R-SPI-SER" (at 40.64 233.68 0) (effects (font (size 1.27 1.27)) hide))
@@
     (property "Note" "At the DRIVING end, which is this board. The far end's threshold is the 74AHCT125's TTL V_IH, not a ratio of its rail" (at 40.64 233.68 0) (effects (font (size 1.27 1.27)) hide))
     (property "Manufacturer" "UNI-ROYAL" (at 40.64 233.68 0) (effects (font (size 1.27 1.27)) hide))
-    (property "MPN" "0805W8F1000T5E" (at 40.64 233.68 0) (effects (font (size 1.27 1.27)) hide))
-    (property "LCSC" "C17408" (at 40.64 233.68 0) (effects (font (size 1.27 1.27)) hide))
+    (property "MPN" "1206W4F1000T5E" (at 40.64 233.68 0) (effects (font (size 1.27 1.27)) hide))
+    (property "LCSC" "C17901" (at 40.64 233.68 0) (effects (font (size 1.27 1.27)) hide))
     (property "Assembly" "machine" (at 40.64 233.68 0) (effects (font (size 1.27 1.27)) hide))
     (pin "1")
@@
     (property "Reference" "R-SPI-SER-MOSI" (at 93.98 232.41 0) (effects (font (size 1.27 1.27)) (justify left)))
     (property "Value" "100R 1%" (at 93.98 234.95 0) (effects (font (size 1.27 1.27)) (justify left)))
-    (property "Footprint" "Resistor_SMD:R_0805_2012Metric" (at 90.17 233.68 0) (effects (font (size 1.27 1.27)) hide))
+    (property "Footprint" "Resistor_SMD:R_1206_3216Metric" (at 90.17 233.68 0) (effects (font (size 1.27 1.27)) hide))
     (property "Datasheet" "" (at 91.44 233.68 0) (effects (font (size 1.27 1.27)) hide))
     (property "Row" "R-SPI-SER" (at 91.44 233.68 0) (effects (font (size 1.27 1.27)) hide))
     (property "Pins" "1=1 2=2" (at 91.44 233.68 0) (effects (font (size 1.27 1.27)) hide))
     (property "Manufacturer" "UNI-ROYAL" (at 91.44 233.68 0) (effects (font (size 1.27 1.27)) hide))
-    (property "MPN" "0805W8F1000T5E" (at 91.44 233.68 0) (effects (font (size 1.27 1.27)) hide))
-    (property "LCSC" "C17408" (at 91.44 233.68 0) (effects (font (size 1.27 1.27)) hide))
+    (property "MPN" "1206W4F1000T5E" (at 91.44 233.68 0) (effects (font (size 1.27 1.27)) hide))
+    (property "LCSC" "C17901" (at 91.44 233.68 0) (effects (font (size 1.27 1.27)) hide))
     (property "Assembly" "machine" (at 91.44 233.68 0) (effects (font (size 1.27 1.27)) hide))
     (pin "1")
@@
     (property "Reference" "R-SPI-SER-CS" (at 144.78 232.41 0) (effects (font (size 1.27 1.27)) (justify left)))
     (property "Value" "100R 1%" (at 144.78 234.95 0) (effects (font (size 1.27 1.27)) (justify left)))
-    (property "Footprint" "Resistor_SMD:R_0805_2012Metric" (at 140.97 233.68 0) (effects (font (size 1.27 1.27)) hide))
+    (property "Footprint" "Resistor_SMD:R_1206_3216Metric" (at 140.97 233.68 0) (effects (font (size 1.27 1.27)) hide))
     (property "Datasheet" "" (at 142.24 233.68 0) (effects (font (size 1.27 1.27)) hide))
     (property "Row" "R-SPI-SER" (at 142.24 233.68 0) (effects (font (size 1.27 1.27)) hide))
     (property "Pins" "1=1 2=2" (at 142.24 233.68 0) (effects (font (size 1.27 1.27)) hide))
     (property "Manufacturer" "UNI-ROYAL" (at 142.24 233.68 0) (effects (font (size 1.27 1.27)) hide))
-    (property "MPN" "0805W8F1000T5E" (at 142.24 233.68 0) (effects (font (size 1.27 1.27)) hide))
-    (property "LCSC" "C17408" (at 142.24 233.68 0) (effects (font (size 1.27 1.27)) hide))
+    (property "MPN" "1206W4F1000T5E" (at 142.24 233.68 0) (effects (font (size 1.27 1.27)) hide))
+    (property "LCSC" "C17901" (at 142.24 233.68 0) (effects (font (size 1.27 1.27)) hide))
     (property "Assembly" "machine" (at 142.24 233.68 0) (effects (font (size 1.27 1.27)) hide))
     (pin "1")
