File: hardware/module/breath-response-shaper/breath-response-shaper.jack.kicad_sch (KiCad schematic)
At the start: 1 part

Commit message: WIP module schematics: footprints, bought-part fields, and the two board projects (module-main, module-jack)
Recovered from a container restart; not yet exported or checked.

Co-Authored-By: Claude Opus 5.5 <noreply@anthropic.com>
Claude-Session: https://claude.ai/code/session_01LmB4muFXnoLprWX4JzuJ5A
Parts:
- POT-RESP: footprint (none) -> woody:Potentiometer_SongHuei_R0904N_Single_Vertical; Assembly (none) -> hand; MPN (none) -> RV09AF-40-20K-B50K-0C; Manufacturer (none) -> Alpha
Changed lines of the file:
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@@
     (property "Reference" "POT-RESP" (at 40.64 43.18 0) (effects (font (size 1.27 1.27))))
     (property "Value" "50k linear" (at 40.64 45.72 0) (effects (font (size 1.27 1.27))))
-    (property "Footprint" "" (at 40.64 50.8 0) (effects (font (size 1.27 1.27)) hide))
+    (property "Footprint" "woody:Potentiometer_SongHuei_R0904N_Single_Vertical" (at 40.64 50.8 0) (effects (font (size 1.27 1.27)) hide))
     (property "Datasheet" "" (at 40.64 50.8 0) (effects (font (size 1.27 1.27)) hide))
     (property "Row" "POT-RESP" (at 40.64 50.8 0) (effects (font (size 1.27 1.27)) hide))
@@
     (property "Note" "CW end at V_in/2, CCW end at V_shaped. At centre the wiper is at exactly 0 V FOR ANY INPUT, so the diode branch carries no current and the stage is linear by topology rather than by tolerance" (at 40.64 50.8 0) (effects (font (size 1.27 1.27)) hide))
     (property "Pins_source" "datasheets/connectors/R0904N.pdf p.2 (drawing R09N-003): pins 1-2-3, 2 the wiper, shaft drawn full CCW; clockwise toward 3 is the usual convention [from memory]" (at 40.64 50.8 0) (effects (font (size 1.27 1.27)) hide))
+    (property "Manufacturer" "Alpha" (at 40.64 50.8 0) (effects (font (size 1.27 1.27)) hide))
+    (property "MPN" "RV09AF-40-20K-B50K-0C" (at 40.64 50.8 0) (effects (font (size 1.27 1.27)) hide))
+    (property "LCSC" "" (at 40.64 50.8 0) (effects (font (size 1.27 1.27)) hide))
+    (property "Assembly" "hand" (at 40.64 50.8 0) (effects (font (size 1.27 1.27)) hide))
     (pin "1")
     (pin "2")
     (pin "3")
-    (instances (project "breath-response-shaper.jack" (path "/f3cf1183-3ccd-574d-a1a6-4d0a7c605c94" (reference "POT-RESP") (unit 1))) (project "breath-response-shaper" (path "/97139bb3-9c58-5159-a2a9-3813e79c635b/0b5e67e3-5413-52cb-b319-ff120b80b6dc" (reference "POT-RESP") (unit 1))))
+    (instances (project "module-jack" (path "/f69c67ba-c380-5393-90d5-6d2847e300fb/de7f42d8-0ff4-57e8-9765-79c6eff73d2d" (reference "RV3") (unit 1))) (project "breath-response-shaper.jack" (path "/f3cf1183-3ccd-574d-a1a6-4d0a7c605c94" (reference "POT-RESP") (unit 1))) (project "breath-response-shaper" (path "/97139bb3-9c58-5159-a2a9-3813e79c635b/0b5e67e3-5413-52cb-b319-ff120b80b6dc" (reference "POT-RESP") (unit 1))))
   )
   (wire (pts (xy 40.64 54.61) (xy 40.64 57.15)) (stroke (width 0) (type default)))

Commit message: Breath response shaper adopted: restoring half drawn, output feeds POT-GAIN; pots ordered to fit the knob
U-RESP B restores x2 inverting (R-RESTORE-IN 10k, R-RESTORE-FB 20k): unity and
the in-amp's polarity at centre detent. BREATH_SHAPED feeds POT-GAIN on
J-B2B-MOD pin 1; nets.yaml moves the shaper from proposed to fitted.
POT-GAIN linear (the design's working gain sits at noon); POT-OFFSET gets no
detent. POT-GAIN/OFFSET are Song Huei R0904N KC (18-tooth, the T18 knob's
shaft; KQ is 40-tooth); POT-RESP Alpha RV09AF-40-25B-B50K-0C (18-tooth B shaft,
centre click). POT-OFFSET's zero is +18.7 deg on the 280-deg track, not 300.

Co-Authored-By: Claude Opus 5.5 <noreply@anthropic.com>
Claude-Session: https://claude.ai/code/session_01LmB4muFXnoLprWX4JzuJ5A
Parts:
- POT-RESP: MPN RV09AF-40-20K-B50K-0C -> RV09AF-40-25B-B50K-0C; Pins_source datasheets/connectors/R0904N.pdf p.2 (drawing R09N-003): pi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 -> datasheets/connectors/RV09AF-40.pdf p.3 (RV09AF-40 outline)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
Changed lines of the file:
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@@
     (property "Pins" "CW=3(3) W=2(2) CCW=1(1)" (at 40.64 50.8 0) (effects (font (size 1.27 1.27)) hide))
     (property "Note" "CW end at V_in/2, CCW end at V_shaped. At centre the wiper is at exactly 0 V FOR ANY INPUT, so the diode branch carries no current and the stage is linear by topology rather than by tolerance" (at 40.64 50.8 0) (effects (font (size 1.27 1.27)) hide))
-    (property "Pins_source" "datasheets/connectors/R0904N.pdf p.2 (drawing R09N-003): pins 1-2-3, 2 the wiper, shaft drawn full CCW; clockwise toward 3 is the usual convention [from memory]" (at 40.64 50.8 0) (effects (font (size 1.27 1.27)) hide))
+    (property "Pins_source" "datasheets/connectors/RV09AF-40.pdf p.3 (RV09AF-40 outline): pins 1-2-3, 2 the wiper, shaft drawn full CCW. Which end clockwise approaches is not on the drawing: CW toward 3 is the usual convention [from memory] - checked with an ohmmeter at goods-in (module-jack README)" (at 40.64 50.8 0) (effects (font (size 1.27 1.27)) hide))
     (property "Manufacturer" "Alpha" (at 40.64 50.8 0) (effects (font (size 1.27 1.27)) hide))
-    (property "MPN" "RV09AF-40-20K-B50K-0C" (at 40.64 50.8 0) (effects (font (size 1.27 1.27)) hide))
+    (property "MPN" "RV09AF-40-25B-B50K-0C" (at 40.64 50.8 0) (effects (font (size 1.27 1.27)) hide))
     (property "LCSC" "" (at 40.64 50.8 0) (effects (font (size 1.27 1.27)) hide))
     (property "Assembly" "hand" (at 40.64 50.8 0) (effects (font (size 1.27 1.27)) hide))

Commit message: Breath chain fixes (pre-layout review A1): OFFSET clockwise-positive, 1N4448W, chain sim, stale derived statements
POT-OFFSET's ends swapped on the sheet so the panel's + is true (A1-4).
D-RESP bought as Vishay 1N4448W-E3-08, datasheet banked (A1-3, owner).
Shaper-into-output-stage sim added; breath-chain-curve-clip registered (A1-1).
Working point cited as disputed (A1-6, A8-4); REF band, ADR 0006 standing
level, C_cm in the pole, R1b dispute, -12 V row, buffered label, ADC
injection current corrected (A1-8..A1-15). Sims re-run pending.

Co-Authored-By: Claude Opus 5.5 <noreply@anthropic.com>
Claude-Session: https://claude.ai/code/session_01LmB4muFXnoLprWX4JzuJ5A
Other:
- title: Response control (PROPOSED) - the module jack board's page (hardware/module/breath-response-shaper) -> Response control - the module jack board's page (hardware/module/breath-response-shaper)
Changed lines of the file:
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@@
   (paper "A4")
   (title_block
-    (title "Response control (PROPOSED) - the module jack board's page (hardware/module/breath-response-shaper)")
-    (comment 7 "title: Response control (PROPOSED)")
+    (title "Response control - the module jack board's page (hardware/module/breath-response-shaper)")
+    (comment 7 "title: Response control")
     (date "")
     (rev "")
