File: hardware/module/breath-response-shaper/breath-response-shaper.kicad_sch (KiCad schematic)
At the start: 0 parts

Commit message: Breath response shaper adopted: restoring half drawn, output feeds POT-GAIN; pots ordered to fit the knob
U-RESP B restores x2 inverting (R-RESTORE-IN 10k, R-RESTORE-FB 20k): unity and
the in-amp's polarity at centre detent. BREATH_SHAPED feeds POT-GAIN on
J-B2B-MOD pin 1; nets.yaml moves the shaper from proposed to fitted.
POT-GAIN linear (the design's working gain sits at noon); POT-OFFSET gets no
detent. POT-GAIN/OFFSET are Song Huei R0904N KC (18-tooth, the T18 knob's
shaft; KQ is 40-tooth); POT-RESP Alpha RV09AF-40-25B-B50K-0C (18-tooth B shaft,
centre click). POT-OFFSET's zero is +18.7 deg on the 280-deg track, not 300.

Co-Authored-By: Claude Opus 5.5 <noreply@anthropic.com>
Claude-Session: https://claude.ai/code/session_01LmB4muFXnoLprWX4JzuJ5A
Other:
- sheet main ports: added BREATH_SHAPED; removed none
- note added: "AUTHORITATIVE for connectivity. The circuit is ADOPTED (2026-09-30): the in-amp's output comes in on BREATH_INAMP_OUT and the shaped, restored signal leaves on BREATH_SHAPED for POT-GAIN (module/breath-output-stage). [U-RESP] One OPA2197: half A shapes at -1/2, half B restores at -2. [V_IN_HALF] V_in/2, the pot's fixed end. The divider is what makes the null exact. [V_SHAPED] The pot's other end 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"
- note removed: "FROM THE HAND-WRITTEN NETLIST THIS SHEET REPLACES (verbatim; the part notes are on each part's Note field): AUTHORITATIVE for connectivity - of the half of this circuit that is drawn. *** THIS CIRCUIT IS PROPOSED, NOT ADOPTED. *** Every one of its BOM rows is `open`. hardware/nets.yaml carries it under `proposed:` on the three nets it reads, which declares the port without claiming the board has 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"
Changed lines of the file:
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@@
     (pin "MODULE_ANALOG_NEG12" input (at 121.92 66.04 0) (effects (font (size 1.27 1.27)) (justify right)))
     (pin "V_SHAPED" passive (at 121.92 68.58 0) (effects (font (size 1.27 1.27)) (justify right)))
+    (pin "BREATH_SHAPED" output (at 121.92 71.12 0) (effects (font (size 1.27 1.27)) (justify right)))
     (instances (project "breath-response-shaper" (path "/97139bb3-9c58-5159-a2a9-3813e79c635b" (page "2"))))
   )
@@
   (wire (pts (xy 121.92 68.58) (xy 127.0 68.58)) (stroke (width 0) (type default)))
   (label "V_SHAPED" (at 127.0 68.58 0) (fields_autoplaced) (effects (font (size 1.27 1.27)) (justify left bottom)))
+  (wire (pts (xy 121.92 71.12) (xy 127.0 71.12)) (stroke (width 0) (type default)))
+  (hierarchical_label "BREATH_SHAPED" (shape output) (at 127.0 71.12 0) (effects (font (size 1.27 1.27)) (justify left))
+    (property "Dir" "out" (at 127.0 71.12 0) (effects (font (size 1.27 1.27)) hide))
+    (property "To" "module/breath-output-stage" (at 127.0 71.12 0) (effects (font (size 1.27 1.27)) hide)))
   (sheet (at 203.2 50.8) (size 60.96 12.7) (exclude_from_sim no) (in_bom yes) (on_board yes) (dnp no)
     (stroke (width 0.1524) (type solid)) (fill (color 0 0 0 0.0000))
@@
   (wire (pts (xy 264.16 58.42) (xy 269.24 58.42)) (stroke (width 0) (type default)))
   (label "V_SHAPED" (at 269.24 58.42 0) (fields_autoplaced) (effects (font (size 1.27 1.27)) (justify left bottom)))
-  (text "FROM THE HAND-WRITTEN NETLIST THIS SHEET REPLACES (verbatim; the part notes are on each part's Note field):\n\nAUTHORITATIVE for connectivity - of the half of this circuit that is drawn.\n\n*** THIS CIRCUIT IS PROPOSED, NOT ADOPTED. *** Every one of its BOM rows is `open`. hardware/nets.yaml carries\nit under `proposed:` on the three nets it reads, which declares the port without claiming the board has the\nconnection. Nothing here asserts that this stage is fitted.\n\nAND ONLY HALF OF IT IS DRAWN. The page's own cost table spends BOTH remaining OPA2197 halves - \"one shapes at\n/2 inverting, one restores x2 inverting to put scale and polarity back\" - and the drawing shows the shaping\nhalf only. The restoring half has no drawing and no passives in any BOM row, so it is not netlisted: writing\nit would be inventing it. That gap is now a bullet in the page's \"Open before layout\".\n\nTHREE PASSIVES WERE DRAWN AND NEVER LISTED. R1 20k, R2 10k and the 2 x 10k divider are in the page's cost\ntable and were in no bom.csv row until 2026-09-23. They are R-RESP-IN, R-RESP-FB and R-RESP-DIV now.\n\n[U-RESP] ONE OPA2197 PACKAGE. Half A is the shaping half. Half B is the restoring half the page spends and\ndoes not draw: until it is drawn it is tied off as a follower on the star, which is what an unused half is.\n\n[V_IN_HALF] V_in/2, the pot's fixed end. The divider is what makes the null exact.\n\n[VIRTUAL_GND] X, the virtual ground. R-RESP-IN in, R-RESP-FB back, and the diode branch injecting into it\neither way.\n\n[SPARE_B_OUT] The untied half's follower loop.\n\n[V_SHAPED] V_shaped. WHERE THIS INSERTS IS OPEN and the x2 restoring stage that belongs between it and\nanything downstream is not drawn, so this file stops here rather than asserting a path into\nmodule/breath-output-stage." (at 40.64 147.32 0) (effects (font (size 1.27 1.27)) (justify left top)))
+  (text "AUTHORITATIVE for connectivity. The circuit is ADOPTED (2026-09-30): the in-amp's output comes in on\nBREATH_INAMP_OUT and the shaped, restored signal leaves on BREATH_SHAPED for POT-GAIN (module/breath-output-stage).\n\n[U-RESP] One OPA2197: half A shapes at -1/2, half B restores at -2.\n\n[V_IN_HALF] V_in/2, the pot's fixed end. The divider is what makes the null exact.\n\n[V_SHAPED] The pot's other end and the restoring half's input." (at 40.64 147.32 0) (effects (font (size 1.27 1.27)) (justify left top)))
   (text "THIS CIRCUIT IS ON BOTH MODULE BOARDS (ADR 0023). Page main holds its main-board parts, page jack the parts behind the panel; the labels here join the two pages, and on the boards J-B2B-MOD joins them. Each board places its own page." (at 60.96 30.48 0) (effects (font (size 1.27 1.27)) (justify left top)))
   (sheet_instances (path "/" (page "1")))

Commit message: Breath chain fixes (pre-layout review A1): OFFSET clockwise-positive, 1N4448W, chain sim, stale derived statements
POT-OFFSET's ends swapped on the sheet so the panel's + is true (A1-4).
D-RESP bought as Vishay 1N4448W-E3-08, datasheet banked (A1-3, owner).
Shaper-into-output-stage sim added; breath-chain-curve-clip registered (A1-1).
Working point cited as disputed (A1-6, A8-4); REF band, ADR 0006 standing
level, C_cm in the pole, R1b dispute, -12 V row, buffered label, ADC
injection current corrected (A1-8..A1-15). Sims re-run pending.

Co-Authored-By: Claude Opus 5.5 <noreply@anthropic.com>
Claude-Session: https://claude.ai/code/session_01LmB4muFXnoLprWX4JzuJ5A
Other:
- title: Response control (PROPOSED) (hardware/module/breath-response-shaper) -> Response control (hardware/module/breath-response-shaper)
Changed lines of the file:
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@@
   (paper "A3")
   (title_block
-    (title "Response control (PROPOSED) (hardware/module/breath-response-shaper)")
+    (title "Response control (hardware/module/breath-response-shaper)")
     (comment 5 "circuit: module/breath-response-shaper")
     (comment 6 "page: breath-response-shaper.md")
-    (comment 7 "title: Response control (PROPOSED)")
+    (comment 7 "title: Response control")
     (date "")
     (rev "")
