File: hardware/boards/umb-adapter/umb-adapter.kicad_sch (KiCad schematic)
At the start: 2 parts, among them J1 NE8FAV, J2 8-way 2.54mm right-angle pin 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

Commit message: Main board: apply the chosen parts to every symbol and row
Every main-board and adapter symbol now carries Footprint, Manufacturer,
MPN, LCSC and Assembly. The values come from the selections whose
datasheets are banked. The BOM rows follow those choices:

- D-USBOR is the SS14 (SMA).
- J-LED is four solder pads, not a connector.
- L-BUCK-IN is 22 uH, C-BUCK-IN is a UCM electrolytic, C-STRIP-BULK is
  470 uF 25 V.
- D-TVS-BREATH is the PESD12VS1UA (SOD-323); the UB is SOD523.
- J-UMB is the hanxia header. Its posts go through the adapter and its
  tails through the tongue; the old wording had them swapped.
- U-BUCK and U-BREATH say where to buy.
- C-ADC-BULK is 1206 if fitted.

The body and geometry follow the chosen parts:

- The J-UMB and J-MCU envelopes in config/body.yaml are now read off the
  parts' drawings.
- J-MCU is longer, so the regulator block moved and the right-hand ribbon
  header followed it by 1.5 mm. The RH key board is re-laid out, with C8
  moving with the header's 3V3 pin. It checks clean.
- A mount candidate is now nudged by up to 3 mm before it is dropped. All
  seven main-board mounts hold.

New footprints and pages:

- New woody.pretty footprints: the MPXV4006DP (case 1351-01) from
  breath-sense-link.md's land pattern, and the NE8FAV from Neutrik's
  layout, mirrored to the top view.
- The input-LC derivation uses the chosen capacitor's banked ESR: Q is at
  most 1.8, and the margin is 120x worst case.
- The main-board README lists what is still open before layout.

Co-Authored-By: Claude Opus 5.5 <noreply@anthropic.com>
Claude-Session: https://claude.ai/code/session_01LmB4muFXnoLprWX4JzuJ5A
Parts:
- J1: footprint (none) -> woody:Neutrik_NE8FAV_etherCON_Vertical; Assembly (none) -> hand; MPN (none) -> NE8FAV; Manufacturer (none) -> Neutrik
- J2: footprint (none) -> Connector_PinHeader_2.54mm:PinHeader_1x08_P2.54mm_Vertical; Assembly (none) -> none; MPN (none) -> HX PZ2.54-1x8P WZ; Manufacturer (none) -> hanxia
Changed lines of the file:
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@@
     (property "Reference" "J1" (at 76.2 74.93 0) (effects (font (size 1.27 1.27))))
     (property "Value" "NE8FAV" (at 83.82 74.93 0) (effects (font (size 1.27 1.27))))
-    (property "Footprint" "" (at 81.28 88.9 0) (effects (font (size 1.27 1.27)) hide))
+    (property "Footprint" "woody:Neutrik_NE8FAV_etherCON_Vertical" (at 81.28 88.9 0) (effects (font (size 1.27 1.27)) hide))
     (property "Datasheet" "" (at 81.28 88.9 0) (effects (font (size 1.27 1.27)) hide))
     (property "Row" "J-UMBILICAL-INST" (at 81.28 88.9 0) (effects (font (size 1.27 1.27)) hide))
@@
     (property "Note" "The instrument's, behind the tail cap on the umbilical adapter (ADR 0021). Its G tab is not a pin of the umbilical and goes nowhere: the housing is plastic, isolated to panel ground [ds]" (at 81.28 88.9 0) (effects (font (size 1.27 1.27)) hide))
     (property "Pins_source" "datasheets/connectors/NEUTRIK-NE8FAV-DRAWING.pdf, PCB layout: contacts 1-8 as the RJ45's; G, the shield tab, is not a pin of the umbilical" (at 81.28 88.9 0) (effects (font (size 1.27 1.27)) hide))
+    (property "Manufacturer" "Neutrik" (at 81.28 88.9 0) (effects (font (size 1.27 1.27)) hide))
+    (property "MPN" "NE8FAV" (at 81.28 88.9 0) (effects (font (size 1.27 1.27)) hide))
+    (property "LCSC" "" (at 81.28 88.9 0) (effects (font (size 1.27 1.27)) hide))
+    (property "Assembly" "hand" (at 81.28 88.9 0) (effects (font (size 1.27 1.27)) hide))
     (pin "1")
     (pin "2")
@@
     (property "Reference" "J2" (at 177.8 78.74 0) (effects (font (size 1.27 1.27))))
     (property "Value" "8-way 2.54mm right-angle pin header" (at 177.8 101.6 0) (effects (font (size 1.27 1.27))))
-    (property "Footprint" "" (at 177.8 88.9 0) (effects (font (size 1.27 1.27)) hide))
+    (property "Footprint" "Connector_PinHeader_2.54mm:PinHeader_1x08_P2.54mm_Vertical" (at 177.8 88.9 0) (effects (font (size 1.27 1.27)) hide))
     (property "Datasheet" "" (at 177.8 88.9 0) (effects (font (size 1.27 1.27)) hide))
     (property "Row" "J-UMB" (at 177.8 88.9 0) (effects (font (size 1.27 1.27)) hide))
@@
     (property "Note" "On the main board's tongue, soldered into it and into the umbilical adapter, where the carrier's nets reach the umbilical. Pin N is J-UMB-INST pin N through the adapter's tracks; D-REVSHUNT and U-TVS-SPI sit at it" (at 177.8 88.9 0) (effects (font (size 1.27 1.27)) hide))
     (property "Pins_source" "pin N is the etherCON's pin N (ADR 0021); the header is bought and fitted with the main board" (at 177.8 88.9 0) (effects (font (size 1.27 1.27)) hide))
+    (property "Manufacturer" "hanxia" (at 177.8 88.9 0) (effects (font (size 1.27 1.27)) hide))
+    (property "MPN" "HX PZ2.54-1x8P WZ" (at 177.8 88.9 0) (effects (font (size 1.27 1.27)) hide))
+    (property "LCSC" "" (at 177.8 88.9 0) (effects (font (size 1.27 1.27)) hide))
+    (property "Assembly" "none" (at 177.8 88.9 0) (effects (font (size 1.27 1.27)) hide))
     (pin "1")
     (pin "2")

Commit message: NE8FAV: the instrument's and spi-link's etherCONs carry the LCSC code the module's already does (A8-19)
J-UMBILICAL-INST (umb-adapter J1, spi-link J-UMB-INST) and spi-link's
J-UMB-MOD had empty LCSC fields for the part module-main J3 buys as
C368526 (Neutrik NE8FAV, in stock at LCSC 2026-10-01). Fields only;
netlists re-exported unchanged, renders re-ledgered.

Co-Authored-By: Claude Opus 5.5 <noreply@anthropic.com>
Claude-Session: https://claude.ai/code/session_01LmB4muFXnoLprWX4JzuJ5A
Parts:
- J1: LCSC (none) -> C368526
Changed lines of the file:
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@@
     (property "Manufacturer" "Neutrik" (at 81.28 88.9 0) (effects (font (size 1.27 1.27)) hide))
     (property "MPN" "NE8FAV" (at 81.28 88.9 0) (effects (font (size 1.27 1.27)) hide))
-    (property "LCSC" "" (at 81.28 88.9 0) (effects (font (size 1.27 1.27)) hide))
+    (property "LCSC" "C368526" (at 81.28 88.9 0) (effects (font (size 1.27 1.27)) hide))
     (property "Assembly" "hand" (at 81.28 88.9 0) (effects (font (size 1.27 1.27)) hide))
     (pin "1")
