File: hardware/interfaces/spi-link/spi-link.kicad_sch (KiCad schematic)
At the start: 3 parts

Commit message: spi-link: J-UMB-MOD's note named the retired D-series etherCON's 24 mm bore
The module's end is an NE8FAV (ADR 0023), placed by the module CAD
(ADR 0024). Fixed on the sheet; netlist and render re-exported.

Co-Authored-By: Claude Opus 5.5 <noreply@anthropic.com>
Claude-Session: https://claude.ai/code/session_01LmB4muFXnoLprWX4JzuJ5A
Parts:
- J-UMB-MOD: Note The module panel's. BORE IS D24.0 mm MINIMUM, which in a 50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 -> The module panel's: a Neutrik NE8FAV, the same part as the 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
Changed lines of the file:
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@@
     (property "Row" "J-UMBILICAL" (at 238.76 101.6 0) (effects (font (size 1.27 1.27)) hide))
     (property "Pins" "1=1 2=2 3=3 4=4 5=5 6=6 7=7 8=8" (at 238.76 101.6 0) (effects (font (size 1.27 1.27)) hide))
-    (property "Note" "The module panel's. BORE IS D24.0 mm MINIMUM, which in a 50.50 mm 10HP panel leaves 13.25 mm each side - that is a panel constraint before it is a connector choice" (at 238.76 101.6 0) (effects (font (size 1.27 1.27)) hide))
+    (property "Note" "The module panel's: a Neutrik NE8FAV, the same part as the instrument's end (ADR 0023), soldered to the module main board; its bore and screw holes are the module CAD's (mechanical/module/export/panel.dxf, ADR 0024)" (at 238.76 101.6 0) (effects (font (size 1.27 1.27)) hide))
     (property "Pins_source" "datasheets/connectors/NEUTRIK-NE8FAV-DRAWING.pdf, PCB layout: contacts 1-8 as the RJ45's; G, the shield tab, is not a pin of the umbilical" (at 238.76 101.6 0) (effects (font (size 1.27 1.27)) hide))
     (property "Manufacturer" "Neutrik" (at 238.76 101.6 0) (effects (font (size 1.27 1.27)) hide))

Commit message: Main board footprints from the banked drawings: J-MCU, J-UMB drawn; models on J-CHAIN and U-BREATH; LED chamfer mark
J-MCU (XKB X1270WR-2x12A-9TV01): 0.70 holes, 1.50 x 1.07 pads with the
hole off centre (the J-CHAIN pattern, JLC's 0.18 ring), the tail rows
2.60 and 1.33 behind the body per the drawing's rev A1 side view.
J-UMB (HX PZ2.54-1x8P WZ): 1.02 holes, insulator 1.80 in front of the row.
U-BREATH: courtyard takes in the ports. WS2815B-V1: filled silk
triangle at the chamfer (pin 4).

Co-Authored-By: Claude Opus 5.5 <noreply@anthropic.com>
Claude-Session: https://claude.ai/code/session_01LmB4muFXnoLprWX4JzuJ5A
Parts:
- J-UMB: footprint Connector_PinHeader_2.54mm:PinHeader_1x08_P2.54mm_Horizontal -> woody:PinHeader_1x08_P2.54mm_Horizontal_Hanxia_PZ2.54-WZ
Changed lines of the file:
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@@
     (property "Reference" "J-UMB" (at 165.1 91.44 0) (effects (font (size 1.27 1.27))))
     (property "Value" "8-way 2.54mm right-angle pin header" (at 165.1 114.3 0) (effects (font (size 1.27 1.27))))
-    (property "Footprint" "Connector_PinHeader_2.54mm:PinHeader_1x08_P2.54mm_Horizontal" (at 165.1 101.6 0) (effects (font (size 1.27 1.27)) hide))
+    (property "Footprint" "woody:PinHeader_1x08_P2.54mm_Horizontal_Hanxia_PZ2.54-WZ" (at 165.1 101.6 0) (effects (font (size 1.27 1.27)) hide))
     (property "Datasheet" "" (at 165.1 101.6 0) (effects (font (size 1.27 1.27)) hide))
     (property "Row" "J-UMB" (at 165.1 101.6 0) (effects (font (size 1.27 1.27)) hide))

Commit message: NE8FAV: the instrument's and spi-link's etherCONs carry the LCSC code the module's already does (A8-19)
J-UMBILICAL-INST (umb-adapter J1, spi-link J-UMB-INST) and spi-link's
J-UMB-MOD had empty LCSC fields for the part module-main J3 buys as
C368526 (Neutrik NE8FAV, in stock at LCSC 2026-10-01). Fields only;
netlists re-exported unchanged, renders re-ledgered.

Co-Authored-By: Claude Opus 5.5 <noreply@anthropic.com>
Claude-Session: https://claude.ai/code/session_01LmB4muFXnoLprWX4JzuJ5A
Parts:
- J-UMB-INST, J-UMB-MOD: LCSC (none) -> C368526
Changed lines of the file:
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@@
     (property "Manufacturer" "Neutrik" (at 50.8 101.6 0) (effects (font (size 1.27 1.27)) hide))
     (property "MPN" "NE8FAV" (at 50.8 101.6 0) (effects (font (size 1.27 1.27)) hide))
-    (property "LCSC" "" (at 50.8 101.6 0) (effects (font (size 1.27 1.27)) hide))
+    (property "LCSC" "C368526" (at 50.8 101.6 0) (effects (font (size 1.27 1.27)) hide))
     (property "Assembly" "hand" (at 50.8 101.6 0) (effects (font (size 1.27 1.27)) hide))
     (pin "1")
@@
     (property "Manufacturer" "Neutrik" (at 238.76 101.6 0) (effects (font (size 1.27 1.27)) hide))
     (property "MPN" "NE8FAV" (at 238.76 101.6 0) (effects (font (size 1.27 1.27)) hide))
-    (property "LCSC" "" (at 238.76 101.6 0) (effects (font (size 1.27 1.27)) hide))
+    (property "LCSC" "C368526" (at 238.76 101.6 0) (effects (font (size 1.27 1.27)) hide))
     (property "Assembly" "hand" (at 238.76 101.6 0) (effects (font (size 1.27 1.27)) hide))
     (pin "1")
