File: hardware/module/digital-and-supervision/digital-and-supervision.kicad_sch (KiCad schematic)
At the start: 8 parts

Commit message: WIP module schematics: footprints, bought-part fields, and the two board projects (module-main, module-jack)
Recovered from a container restart; not yet exported or checked.

Co-Authored-By: Claude Opus 5.5 <noreply@anthropic.com>
Claude-Session: https://claude.ai/code/session_01LmB4muFXnoLprWX4JzuJ5A
Parts:
- C-DEC-LVL: footprint (none) -> Capacitor_SMD:C_0805_2012Metric; Assembly (none) -> machine; LCSC (none) -> C49678; MPN (none) -> CC0805KRX7R9BB104; Manufacturer (none) -> YAGEO
- R-PULL-CS, R-PULL-DIN, R-PULL-MOSI, R-PULL-SCLK, R-PULL-SCLK-DAC, R-PULL-SYNC: footprint (none) -> Resistor_SMD:R_0805_2012Metric; Assembly (none) -> machine; LCSC (none) -> C17414; MPN (none) -> 0805W8F1002T5E; Manufacturer (none) -> UNI-ROYAL(Uniroyal Elec)
- U-LVL-MOD: footprint (none) -> Package_SO:SOIC-14_3.9x8.7mm_P1.27mm; Assembly (none) -> machine; LCSC (none) -> C155176; MPN (none) -> SN74AHCT125DR; Manufacturer (none) -> Texas Instruments

Commit message: Module: four-layer ground settled, local 5 V, metal standoffs, pitch budget, board-to-board header
Owner decisions of 2026-09-30 applied. dig-gnd-topology settled: one star at
J-PWR-EURO's ground pins, DIG_GND a layer-2 plane tied there by the new
NT-DIG-MOD, AGND_MOD its own region by NT-AGND-MOD, PWR_GND on layer 4; the
proposal's bridge under the DAC dropped per SBAS430E p.49 (DIG_GND was an
island tied only through the cable before). PCB-MODULE four layers, the jack
board two. The bus +5 V is not used: U-REG-LOGIC (ADP7118AUJZ-5.0, banked)
makes LOGIC_5V from the analog +12 V; FB4/C4 gone, the 16-pin header kept
with its +5 V/CV/Gate pins no-connect (ADR 0023 point 3 amended). Metal
standoffs: pads AGND_MOD on the jack board, no net on the main board.
pitch-cents-budget settled at 0.76 cents linear / 0.45 RSS from one table.
J-B2B-MOD is Samtec TSW-110-09-G-D. Module sims are stale and re-run next.

Co-Authored-By: Claude Opus 5.5 <noreply@anthropic.com>
Claude-Session: https://claude.ai/code/session_01LmB4muFXnoLprWX4JzuJ5A
Connections:
- net BUS_5V renamed LOGIC_5V
Changed lines of the file:
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@@
     (property "To" "module/dac8568" (at 142.24 181.61 0) (effects (font (size 1.27 1.27)) hide)))
   (wire (pts (xy 142.24 38.1) (xy 142.24 35.56)) (stroke (width 0) (type default)))
-  (hierarchical_label "BUS_5V" (shape input) (at 142.24 35.56 90) (effects (font (size 1.27 1.27)) (justify left))
+  (hierarchical_label "LOGIC_5V" (shape input) (at 142.24 35.56 90) (effects (font (size 1.27 1.27)) (justify left))
     (property "Dir" "in" (at 142.24 35.56 0) (effects (font (size 1.27 1.27)) hide))
     (property "From" "module/power-entry" (at 142.24 35.56 0) (effects (font (size 1.27 1.27)) hide)))
   (wire (pts (xy 40.64 138.43) (xy 40.64 135.89)) (stroke (width 0) (type default)))
-  (hierarchical_label "BUS_5V" (shape input) (at 40.64 135.89 90) (effects (font (size 1.27 1.27)) (justify left))
+  (hierarchical_label "LOGIC_5V" (shape input) (at 40.64 135.89 90) (effects (font (size 1.27 1.27)) (justify left))
     (property "Dir" "in" (at 40.64 135.89 0) (effects (font (size 1.27 1.27)) hide))
     (property "From" "module/power-entry" (at 40.64 135.89 0) (effects (font (size 1.27 1.27)) hide)))

Commit message: Link supervision not restored; CS_MOD pulled up at both ends of the umbilical
Owner, 2026-09-30: "Assume the module will be operating with an umbilical
attached to a controller" - link supervision stays unfitted, recorded on its
page, its notes and ADR 0004; CLR stays tied inactive, OE enabled.

"Fix the SPI pull up": the module's cable-side CS pull-up had its top end on
no net. It is now R-CS-PULL-INST, 10k to 3V3 on the main board's carrier
sheet (IO34 beside J-MCU 13/14, MCU side of R-SPI-SER-CS), and R-PULL-CS at
the module weakened to 100k and taken to LOGIC_5V (row R-CS-PULL-MOD). The
proposed weak pull-DOWN at the module was not fitted: the 74AHCT125 does not
invert, so it would have held SYNC low (selected) with the umbilical out.
spi-link.md tabulates the four link states; GPIO34 is not a strapping pin.

Co-Authored-By: Claude Opus 5.5 <noreply@anthropic.com>
Claude-Session: https://claude.ai/code/session_01LmB4muFXnoLprWX4JzuJ5A
Parts:
- R-PULL-CS: value 10k 1% -> 100k 1%; LCSC C17414 -> C149504; MPN 0805W8F1002T5E -> 0805W8F1003T5E; Note PULL-UP, and the only one of the six whose top end this fil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 -> PULL-UP TO LOGIC_5V, 100k - the weak half of CS_MOD's two p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; Row R-SPI-PULL -> R-CS-PULL-MOD
Connections:
- net LOGIC_5V: now also R-PULL-CS.2
- no-connect marks 2 -> 1
Other:
- note added: "FROM THE HAND-WRITTEN NETLIST THIS SHEET REPLACES (verbatim; the part notes are on each part's Note field): A LONE NO-CONNECT PIN'S NET IS NAMED AFTER THE PIN (the export names it so, whatever label it carries), so the one-pin net the text below names is, on this sheet: SPARE_GATE_OUT is 4Y. AUTHORITATIVE for connectivity. The ASCII drawing in digital-and-supervision.md is a REPRESENTATION of thi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"
- note removed: "FROM THE HAND-WRITTEN NETLIST THIS SHEET REPLACES (verbatim; the part notes are on each part's Note field): A LONE NO-CONNECT PIN'S NET IS NAMED AFTER THE PIN (the export names it so, whatever label it carries), so the one-pin nets the text below names are, on this sheet: SPARE_GATE_OUT is 4Y; CS_PULLUP_TOP is 2. AUTHORITATIVE for connectivity. The ASCII drawing in digital-and-supervision.md is a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"
Changed lines of the file:
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@@
     (in_bom yes) (on_board yes) (dnp no)
     (property "Reference" "R-PULL-CS" (at 195.58 140.97 0) (effects (font (size 1.27 1.27)) (justify left)))
-    (property "Value" "10k 1%" (at 195.58 143.51 0) (effects (font (size 1.27 1.27)) (justify left)))
+    (property "Value" "100k 1%" (at 195.58 143.51 0) (effects (font (size 1.27 1.27)) (justify left)))
     (property "Footprint" "Resistor_SMD:R_0805_2012Metric" (at 191.77 142.24 0) (effects (font (size 1.27 1.27)) hide))
     (property "Datasheet" "" (at 193.04 142.24 0) (effects (font (size 1.27 1.27)) hide))
-    (property "Row" "R-SPI-PULL" (at 193.04 142.24 0) (effects (font (size 1.27 1.27)) hide))
+    (property "Row" "R-CS-PULL-MOD" (at 193.04 142.24 0) (effects (font (size 1.27 1.27)) hide))
     (property "Pins" "1=1 2=2" (at 193.04 142.24 0) (effects (font (size 1.27 1.27)) hide))
-    (property "Note" "PULL-UP, and the only one of the six whose top end this file cannot assert - see CS_PULLUP_TOP" (at 193.04 142.24 0) (effects (font (size 1.27 1.27)) hide))
+    (property "Note" "PULL-UP TO LOGIC_5V, 100k - the weak half of CS_MOD's two pulls (the strong one is R-CS-PULL-INST, 10k to 3V3 at the instrument). Weak so that with the instrument plugged in and unpowered it drives only ~45 uA into the dead 3V3 rail and the node sits at ~0.45 V, not the 430 uA a 10k here would force through the ESP32's clamp; with nothing plugged in it holds the buffer input, and so SYNC, deselected. interfaces/spi-link/spi-link.md, 'CS_MOD's two pulls'" (at 193.04 142.24 0) (effects (font (size 1.27 1.27)) hide))
     (property "Manufacturer" "UNI-ROYAL(Uniroyal Elec)" (at 193.04 142.24 0) (effects (font (size 1.27 1.27)) hide))
-    (property "MPN" "0805W8F1002T5E" (at 193.04 142.24 0) (effects (font (size 1.27 1.27)) hide))
-    (property "LCSC" "C17414" (at 193.04 142.24 0) (effects (font (size 1.27 1.27)) hide))
+    (property "MPN" "0805W8F1003T5E" (at 193.04 142.24 0) (effects (font (size 1.27 1.27)) hide))
+    (property "LCSC" "C149504" (at 193.04 142.24 0) (effects (font (size 1.27 1.27)) hide))
     (property "Assembly" "machine" (at 193.04 142.24 0) (effects (font (size 1.27 1.27)) hide))
     (pin "1")
@@
     (property "Figure" "dig-gnd-topology" (at 40.64 148.59 0) (effects (font (size 1.27 1.27)) hide)))
   (no_connect (at 99.06 96.52))
-  (no_connect (at 193.04 146.05))
-  (text "FROM THE HAND-WRITTEN NETLIST THIS SHEET REPLACES (verbatim; the part notes are on each part's Note field):\n\nA LONE NO-CONNECT PIN'S NET IS NAMED AFTER THE PIN (the export names it so, whatever label it carries), so the\none-pin nets the text below names are, on this sheet: SPARE_GATE_OUT is 4Y; CS_PULLUP_TOP is 2.\n\nAUTHORITATIVE for connectivity. The ASCII drawing in digital-and-supervision.md is a REPRESENTATION of this\nfile.\n\nALL SIX R-SPI-PULL INSTANCES ARE PLACED HERE. The row lives in interfaces/spi-link's bom.csv because that page\nderives the values, but the resistors are on the module board on both sides of this buffer, and the drawing\nabove shows both triples. Owning a row and placing an instance are different things; `of:` is what says so.\n\nONE OF THE SIX HAS NOWHERE TO GO - see CS_PULLUP_TOP at the bottom.\n\n[pins] WHICH SIGNAL GETS WHICH GATE IS ASSIGNED HERE AND NOWHERE ELSE [derived, not cited]. No page states it;\na netlist has to. Gate 4 is the spare the BOM row mentions. Contradict this in the page and the file follows.\n\n--- cable side: the three pulls that hold the BUFFER's inputs ------\n\n--- DAC side: the three that hold the DAC's inputs ----------------\n\nThese were bought for the state the cable-side three do not reach: module alive, instrument off, which is\nNORMAL and not a fault.\n\n[DIG_GND] THE FOUR ENABLES ARE TIED, NOT DRIVEN. OE_MOD is in hardware/nets.yaml's `retired:` section for\nexactly this reason: the comparator that gated it is not fitted, so there is no net crossing a boundary - just\nfour pins on the local ground.\n\n[4Y] THE SPARE GATE'S INPUT IS TIED, and it is tied because the BOM row says \"TIE EVERY UNUSED INPUT TO VCC OR\nGND\" - a floating CMOS input on an enabled gate is the one wrong answer. GND is chosen over VCC because the\npart has no input clamp to VCC and the ground tie cannot inject current into an unpowered rail. Its output\ndrives nothing, which is fine.\n\n*** THE CABLE-SIDE CS PULL-UP HAS NO RAIL ON THIS BOARD. ***\n\nR-SPI-PULL's own row says \"CABLE-SIDE CS PULLS TO 3V3, NOT +5V\", with the reason: at 5 V it drives 430 uA\ncontinuously through the unpowered ESP32's input clamp in the design's normal resting state, and the node sits\nat ~0.7 V so \"CS idle high\" is not achieved at all. The reasoning is sound and the rail does not exist here -\nthe umbilical carries BREATH/AGND, +12V/PWR_GND, SCLK/MOSI and CS/DIG_GND, and the module makes +12, -12, bus\n+5 and DAC AVDD. There is no 3V3 anywhere on this board.\n\n['2'] So either this resistor belongs at the INSTRUMENT end, where 3V3 exists and where its own argument about\nthe ESP32's clamp is measured, or the row's \"at the module\" description is right and the rail has to come from\nsomewhere. Both cannot be true. Nothing is asserted until it is decided; digital-and-supervision.md's \"Still\nopen\" carries the question." (at 256.54 38.099999999999994 0) (effects (font (size 1.27 1.27)) (justify left top)))
+  (wire (pts (xy 193.04 146.05) (xy 193.04 148.59)) (stroke (width 0) (type default)))
+  (hierarchical_label "LOGIC_5V" (shape input) (at 193.04 148.59 270) (effects (font (size 1.27 1.27)) (justify right))
+    (property "Dir" "in" (at 193.04 148.59 0) (effects (font (size 1.27 1.27)) hide))
+    (property "From" "module/power-entry" (at 193.04 148.59 0) (effects (font (size 1.27 1.27)) hide)))
+  (text "FROM THE HAND-WRITTEN NETLIST THIS SHEET REPLACES (verbatim; the part notes are on each part's Note field):\n\nA LONE NO-CONNECT PIN'S NET IS NAMED AFTER THE PIN (the export names it so, whatever label it carries), so the\none-pin net the text below names is, on this sheet: SPARE_GATE_OUT is 4Y.\n\nAUTHORITATIVE for connectivity. The ASCII drawing in digital-and-supervision.md is a REPRESENTATION of this\nfile.\n\nALL SIX MODULE-END SPI PULLS ARE PLACED HERE (five R-SPI-PULL, and R-PULL-CS of R-CS-PULL-MOD). The row lives in interfaces/spi-link's bom.csv because that page\nderives the values, but the resistors are on the module board on both sides of this buffer, and the drawing\nabove shows both triples. Owning a row and placing an instance are different things; `of:` is what says so.\n\nThe cable-side CS pull is 100k to LOGIC_5V - see the bottom.\n\n[pins] WHICH SIGNAL GETS WHICH GATE IS ASSIGNED HERE AND NOWHERE ELSE [derived, not cited]. No page states it;\na netlist has to. Gate 4 is the spare the BOM row mentions. Contradict this in the page and the file follows.\n\n--- cable side: the three pulls that hold the BUFFER's inputs ------\n\n--- DAC side: the three that hold the DAC's inputs ----------------\n\nThese were bought for the state the cable-side three do not reach: module alive, instrument off, which is\nNORMAL and not a fault.\n\n[DIG_GND] THE FOUR ENABLES ARE TIED, NOT DRIVEN. OE_MOD is in hardware/nets.yaml's `retired:` section for\nexactly this reason: the comparator that gated it is not fitted, so there is no net crossing a boundary - just\nfour pins on the local ground.\n\n[4Y] THE SPARE GATE'S INPUT IS TIED, and it is tied because the BOM row says \"TIE EVERY UNUSED INPUT TO VCC OR\nGND\" - a floating CMOS input on an enabled gate is the one wrong answer. GND is chosen over VCC because the\npart has no input clamp to VCC and the ground tie cannot inject current into an unpowered rail. Its output\ndrives nothing, which is fine.\n\nTHE CABLE-SIDE CS PULL-UP, SETTLED 2026-09-30 (owner: 'Fix the SPI pull up'). CS_MOD has two pulls now, one at each end: R-CS-PULL-INST, 10k to 3V3 on the main board, where 3V3 exists, and R-PULL-CS here, 100k to LOGIC_5V. The strong one holds CS high while the ESP32 boots; the weak one holds it high with nothing plugged in, and is weak enough that a plugged-in, unpowered instrument sees ~45 uA into its dead 3V3 rail instead of 430 uA through its clamp. A pull-DOWN here was proposed and not fitted: the 74AHCT125 does not invert, so it would hold SYNC LOW - selected - whenever the umbilical is out. interfaces/spi-link/spi-link.md carries the three states." (at 256.54 38.099999999999994 0) (effects (font (size 1.27 1.27)) (justify left top)))
   (sheet_instances (path "/" (page "1")))
 )
