File: hardware/boards/module-main/module-main.kicad_sch (KiCad schematic)
At the start: 2 parts, among them J2 2x10 2.54mm pin header, J3 Neutrik NE8FAV

Commit message: LED-PANEL moves to the main board (LTST-C171GKT under a Bivar PLP2-750 light pipe); J-B2B-MOD pin 19 freed; jack board keeps H1-H2; panel standoffs and studs in the BOM
Co-Authored-By: Claude Opus 5.5 <noreply@anthropic.com>
Claude-Session: https://claude.ai/code/session_01LmB4muFXnoLprWX4JzuJ5A
Connections:
- net UMBILICAL_POS12: no longer J2.19 (Pin_19)
- no-connect marks 0 -> 1
Other:
- added sheet panel-led (../../module/panel-led/panel-led.kicad_sch)
Changed lines of the file:
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@@
   (wire (pts (xy 457.2 165.1) (xy 454.66 165.1)) (stroke (width 0) (type default)))
   (label "MOD3_JACK" (at 454.66 165.1 180) (fields_autoplaced) (effects (font (size 1.27 1.27)) (justify right bottom)))
-  (wire (pts (xy 101.6 76.2) (xy 99.06 76.2)) (stroke (width 0) (type default)))
-  (label "UMBILICAL_POS12" (at 99.06 76.2 180) (fields_autoplaced) (effects (font (size 1.27 1.27)) (justify right bottom)))
   (wire (pts (xy 254.0 55.88) (xy 256.54 55.88)) (stroke (width 0) (type default)))
   (symbol (lib_id "power:+12V") (at 256.54 55.88 270) (unit 1)
@@
     (instances (project "module-main" (path "/fc77e9f9-9171-5c83-92ae-8cafe880764e" (page "10"))))
   )
+  (no_connect (at 101.6 76.2))
+  (wire (pts (xy 457.2 193.04) (xy 454.66 193.04)) (stroke (width 0) (type default)))
+  (label "UMBILICAL_POS12" (at 454.66 193.04 180) (fields_autoplaced) (effects (font (size 1.27 1.27)) (justify right bottom)))
+  (wire (pts (xy 457.2 195.58) (xy 454.66 195.58)) (stroke (width 0) (type default)))
+  (label "AGND_MOD" (at 454.66 195.58 180) (fields_autoplaced) (effects (font (size 1.27 1.27)) (justify right bottom)))
+  (sheet (at 457.2 190.5) (size 50.8 10.16) (exclude_from_sim no) (in_bom yes) (on_board yes) (dnp no)
+    (stroke (width 0.1524) (type solid)) (fill (color 0 0 0 0.0000))
+    (property "Sheetname" "panel-led" (at 457.2 189.23 0) (effects (font (size 1.27 1.27)) (justify left bottom)))
+    (property "Sheetfile" "../../module/panel-led/panel-led.kicad_sch" (at 457.2 200.66 0) (effects (font (size 1.27 1.27)) (justify left top)))
+    (pin "UMBILICAL_POS12" input (at 457.2 193.04 180) (effects (font (size 1.27 1.27)) (justify left)))
+    (pin "AGND_MOD" passive (at 457.2 195.58 180) (effects (font (size 1.27 1.27)) (justify left)))
+    (instances (project "module-main" (path "/fc77e9f9-9171-5c83-92ae-8cafe880764e" (page "11"))))
+  )
   (sheet_instances (path "/" (page "1")))
