File: hardware/boards/module-main/module-main.kicad_pcb (KiCad board)
At the start: 4 copper layers, 48.5 x 108.5 mm, 177 parts, among them J1 2x8 2.54mm shrouded box heade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, J2 2x10 2.54mm pin header, J3 Neutrik NE8FAV, J4 JST B2B-XH-A, Q1 PSMN2R0-30YLE, SW1 NKK M2011SD4G01, U1 LT3042EMSE, U10 OPA2197, U11 OPA2197, U12 OPA2197, U13 ADP7118AUJZ-5.0, U14 RPA20-2412SAW, U15 74AHCT14, U2 LT1641-1IS8, U3 DAC8568ICPW, U4 74AHCT125, U5 OPA2197, U6 INA828IDR, U7 OPA2197, U8 OPA2197IDR, U9 OPA2197

Commit message: module-main: routing state (window fix pass)
Co-Authored-By: Claude Opus 5.5 <noreply@anthropic.com>
Claude-Session: https://claude.ai/code/session_01LmB4muFXnoLprWX4JzuJ5A
Routing:
- net /power-entry/BUS_GND: track 16.9 -> 27.0 mm, vias 1 -> 4
- net /breath-output-stage/BREATH_OUT: track 9.49 -> 17.7 mm, vias 2 -> 4
- net AGND_MOD: track 86.1 -> 87.5 mm
- net /SYNC: track 1.92 -> 3.26 mm
- net /DIN: track 9.58 -> 10.9 mm
- net /DAC_CH4: track 0.00 -> 1.34 mm
- net /DAC_CH2: track 2.92 -> 4.25 mm
- net /DAC_AVDD: track 146.0 -> 147.3 mm
- net /pitch-stage/GAIN_TRIM_MID: track 4.56 -> 5.89 mm
Changed lines of the file:
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@@
 	)
 	(segment
+		(start 71.9625 93.175)
+		(end 73.3 93.175)
+		(width 0.2)
+		(locked yes)
+		(layer "F.Cu")
+		(net 7)
+	)
+	(segment
 		(start 88.8 44.8)
 		(end 88.775 44.775)
@@
 	)
 	(segment
+		(start 66.2375 92.525)
+		(end 64.9 92.525)
+		(width 0.2)
+		(locked yes)
+		(layer "F.Cu")
+		(net 9)
+	)
+	(segment
 		(start 77.0625 82.9)
 		(end 76.8 83.1625)
@@
 	)
 	(segment
+		(start 66.2375 91.875)
+		(end 64.9 91.875)
+		(width 0.2)
+		(locked yes)
+		(layer "F.Cu")
+		(net 11)
+	)
+	(segment
 		(start 80.2 89.8546)
 		(end 80.2 87.3)
@@
 	)
 	(segment
+		(start 66.2375 93.825)
+		(end 64.9 93.825)
+		(width 0.2)
+		(locked yes)
+		(layer "F.Cu")
+		(net 14)
+	)
+	(segment
 		(start 73.2 102.7)
 		(end 72.6 102.1)
@@
 	)
 	(segment
+		(start 71.9625 93.825)
+		(end 73.3 93.825)
+		(width 0.2)
+		(locked yes)
+		(layer "F.Cu")
+		(net 29)
+	)
+	(segment
 		(start 79 104.035)
 		(end 79 104.1)
@@
 	(segment
 		(start 74.8 59.6875)
-		(end 74.8 59.0875)
+		(end 74.8 58.5)
 		(width 0.25)
 		(layer "F.Cu")
@@
 	)
 	(via
+		(at 74.8 58.5)
+		(size 0.7)
+		(drill 0.3)
+		(layers "F.Cu" "B.Cu")
+		(net 32)
+	)
+	(via
 		(at 75.6 64.9)
 		(size 0.7)
@@
 	)
 	(via
+		(at 72.8 58.5)
+		(size 0.7)
+		(drill 0.3)
+		(layers "F.Cu" "B.Cu")
+		(net 32)
+	)
+	(via
 		(at 78.4 65.099999)
 		(size 0.7)
@@
 	)
 	(segment
+		(start 72.8 58.5)
+		(end 72.8 62.1)
+		(width 0.25)
+		(layer "B.Cu")
+		(net 32)
+	)
+	(segment
 		(start 75.4 64.7)
 		(end 75.6 64.9)
@@
 	)
 	(segment
+		(start 72.8 62.1)
+		(end 74.2 63.5)
+		(width 0.25)
+		(layer "B.Cu")
+		(net 32)
+	)
+	(segment
 		(start 75.3414 64.4539)
 		(end 74.8 63.9125)
@@
 	)
 	(segment
+		(start 74.8 58.5)
+		(end 72.8 58.5)
+		(width 0.25)
+		(layer "In2.Cu")
+		(net 32)
+	)
+	(segment
 		(start 72 64.12)
 		(end 72 64.3)
@@
 	)
 	(segment
+		(start 96.15 69.675)
+		(end 97.475 69.675)
+		(width 0.2)
+		(locked yes)
+		(layer "F.Cu")
+		(net 75)
+	)
+	(segment
 		(start 93.96 55)
 		(end 91.42 55)
@@
 	)
 	(segment
+		(start 99.4 118.7)
+		(end 99.8 119.1)
+		(width 0.25)
+		(layer "F.Cu")
+		(net 83)
+	)
+	(segment
+		(start 99 118.7)
+		(end 98.1 119.6)
+		(width 0.25)
+		(layer "F.Cu")
+		(net 83)
+	)
+	(segment
 		(start 99.4 116.9)
 		(end 99.2 116.9)
@@
 	)
 	(segment
+		(start 98.1 119.6)
+		(end 98.6 120.1)
+		(width 0.25)
+		(layer "F.Cu")
+		(net 83)
+	)
+	(segment
 		(start 99.1 116.9)
 		(end 99 116.8)
@@
 		(net 83)
 	)
+	(segment
+		(start 99 118.7)
+		(end 99.4 118.7)
+		(width 0.25)
+		(layer "F.Cu")
+		(net 83)
+	)
+	(segment
+		(start 99 120.1)
+		(end 98.6 120.1)
+		(width 0.25)
+		(layer "F.Cu")
+		(net 83)
+	)
+	(segment
+		(start 98.1 119.6)
+		(end 97.4 118.9)
+		(width 0.25)
+		(layer "F.Cu")
+		(net 83)
+	)
+	(via
+		(at 99.8 120.9)
+		(size 0.7)
+		(drill 0.3)
+		(layers "F.Cu" "B.Cu")
+		(net 83)
+	)
+	(via
+		(at 99.8 119.1)
+		(size 0.7)
+		(drill 0.3)
+		(layers "F.Cu" "B.Cu")
+		(net 83)
+	)
 	(via
 		(at 99.6 116.5)
@@
 		(net 83)
 	)
+	(via
+		(at 97.4 118.9)
+		(size 0.7)
+		(drill 0.3)
+		(layers "F.Cu" "B.Cu")
+		(net 83)
+	)
 	(segment
 		(start 101 117.27)
@@
 	)
 	(segment
+		(start 99.8 119.1)
+		(end 99.8 120.9)
+		(width 0.25)
+		(layer "B.Cu")
+		(net 83)
+	)
+	(segment
 		(start 103.77 120.07)
 		(end 103.77 118.81)
@@
 	)
 	(segment
+		(start 97.4 118.9)
+		(end 100.6 118.9)
+		(width 0.25)
+		(layer "In2.Cu")
+		(net 83)
+	)
+	(segment
 		(start 100.6 116.5)
 		(end 101 116.5)
@@
 	)
 	(segment
+		(start 99.8 120.9)
+		(end 100.6 120.9)
+		(width 0.25)
+		(layer "In2.Cu")
+		(net 83)
+	)
+	(segment
 		(start 104.4 123.7)
 		(end 104.6 123.9)
@@
 		(locked yes)
 		(layer "F.Cu")
+		(net 107)
+	)
+	(segment
+		(start 66.2375 93.175)
+		(end 64.9 93.175)
+		(width 0.2)
+		(locked yes)
+		(layer "F.Cu")

Commit message: module-main: best routing state (20 unrouted; pcb.py check fails - README says so); pcb.py silk title tries listed places, then searches both faces
Co-Authored-By: Claude Opus 5.5 <noreply@anthropic.com>
Claude-Session: https://claude.ai/code/session_01LmB4muFXnoLprWX4JzuJ5A
Other:
- board text added: "C1"
- board text added: "C12"
- board text added: "C18"
- board text added: "C19"
- board text added: "C2"
- board text added: "C21"
- board text added: "C22"
- board text added: "C24"
- board text added: "C3"
- board text added: "C38"
- board text added: "C44"
- board text added: "C46"
- board text added: "C51"
- board text added: "C6"
- board text added: "C7"
- board text added: "D1"
- board text added: "D14"
- board text added: "D15"
- board text added: "D2"
- board text added: "F1"
- board text added: "F2"
- board text added: "F3"
- board text added: "FB2"
- board text added: "FB3"
- board text added: "FB4"
- board text added: "J1"
- board text added: "J2"
- board text added: "J3"
- board text added: "JP1"
- board text added: "L1"
- board text added: "L2"
- board text added: "R11"
- board text added: "R14"
- board text added: "R25"
- board text added: "R26"
- board text added: "R27"
- board text added: "R31"
- board text added: "R34"
- board text added: "R52"
- board text added: "R56"
- board text added: "R57"
- board text added: "R58"
- board text added: "R59"
- board text added: "R6"
- board text added: "R60"
- board text added: "R62"
- board text added: "R63"
- board text added: "R8"
- board text added: "R9"
- board text added: "RV1"
- board text added: "RV3"
- board text added: "RV4"
- board text added: "U12"
- board text added: "U15"
- board text added: "U2"
- board text added: "U3"
- board text added: "U4"
- board text added: "U5"
- board text added: "U7"
- board text added: "WOODY mod-main"
- board text added: "rev A 2026-10-02"

Commit message: module-main placed for the iso board: U-ISO and its filter gone, J-B2B-ISO (J5) and three iso standoffs in; parts the new holes displaced re-placed (#22)
Co-Authored-By: Claude Opus 5.5 <noreply@anthropic.com>
Claude-Session: https://claude.ai/code/session_01LmB4muFXnoLprWX4JzuJ5A
Parts:
- removed C2: 100uF 50V, Capacitor_SMD:CP_Elec_6.3x7.7
- removed C44: 4.7uF 50V, Capacitor_SMD:C_1206_3216Metric
- removed C45: 100uF 25V, Capacitor_SMD:CP_Elec_6.3x5.8
- removed C46: 22nF, Capacitor_SMD:C_0805_2012Metric
- removed L1: 22uH, Inductor_SMD:L_Sunlord_SWPA6028S
- removed L2: 1mH, woody:L_CommonModeChoke_Bourns_PM3700
- removed U14: RPA20-2412SAW, woody:Converter_DCDC_RECOM_RPA20-RP20-xxxxSAW_THT
- added H5: MECH-STANDOFF-ISO 1, MountingHole:MountingHole_3.2mm_M3_Pad, F.Cu at (71.5, 108.2)
- added H6: MECH-STANDOFF-ISO 2, MountingHole:MountingHole_3.2mm_M3_Pad, F.Cu at (64.8, 69.9)
- added H7: MECH-STANDOFF-ISO 3, MountingHole:MountingHole_3.2mm_M3_Pad, F.Cu at (105.7, 69.9)
- added J5: 2x5 2.54mm pin header, Connector_PinHeader_2.54mm:PinHeader_2x05_P2.54mm_Vertical, F.Cu at (84.9, 109.3)
- C25: moved to F.Cu
- C28, D11, D9, U9: moved to B.Cu
- moved D1 26.3 mm to (97.2, 88.0), turned to 0 degrees
- moved D15 14.1 mm to (84.9, 99.6), turned to 0 degrees
- moved C25 13.1 mm to (90.2, 67.2), turned to 0 degrees
- moved C28 11.4 mm to (98.0, 77.0)
- moved JP1 10.5 mm to (66.2, 82.2)
- moved D2 8.99 mm to (84.9, 103.1), turned to 0 degrees
- moved D9 8.64 mm to (96.8, 60.0), turned to 0 degrees
- moved U9 6.33 mm to (103.0, 76.2), turned to 180 degrees
- moved D11 4.25 mm to (63.2, 78.8), turned to 90 degrees
- moved R43 4.18 mm to (64.7, 75.5), turned to 180 degrees
- moved C27 0.67 mm to (104.8, 75.2), turned to 0 degrees
Connections:
- FB2 pad 2: /power-entry/ISO_FB2 -> /ISO_FB2
- FB4 pad 2: /power-entry/ISO_FILT_NEG -> /ISO_FILT_NEG
Routing:
- net MODULE_ANALOG_POS12: track 343.8 -> 0.00 mm, vias 41 -> 0
- net MODULE_ANALOG_NEG12: track 302.3 -> 0.00 mm, vias 48 -> 0
- net /dac8568/CLR: track 166.5 -> 0.00 mm, vias 12 -> 0
- net /mod-channels/MINUS_3: track 149.1 -> 0.00 mm, vias 8 -> 0
- net /DAC_AVDD: track 147.3 -> 0.00 mm, vias 15 -> 0
- net PWR_GND: track 105.9 -> 0.00 mm, vias 12 -> 0
- net /BREATH_SENSE: track 103.2 -> 0.00 mm, vias 2 -> 0
- net /AGND_SENSE: track 98.0 -> 0.00 mm, vias 3 -> 0
- net AGND_MOD: track 87.5 -> 0.00 mm, vias 61 -> 0
- net /mod-channels/VREF_MOD: track 76.7 -> 0.00 mm, vias 6 -> 0
- net /power-entry/ISO_VIN_POS: track 61.6 -> 0.00 mm, vias 2 -> 0
- net /power-entry/NEG12_PTC3: track 59.0 -> 0.00 mm, vias 3 -> 0
- net /VREFOUT: track 56.6 -> 0.00 mm, vias 2 -> 0
- net ISO_POS12: track 55.5 -> 0.00 mm, vias 2 -> 0
- net /UMBILICAL_POS12: track 54.9 -> 0.00 mm, vias 8 -> 0
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Other:
- board text removed: "C1"
- board text removed: "C12"
- board text removed: "C18"
- board text removed: "C19"
- board text removed: "C2"
- board text removed: "C21"
- board text removed: "C22"
- board text removed: "C24"
- board text removed: "C3"
- board text removed: "C38"
- board text removed: "C44"
- board text removed: "C46"
- board text removed: "C51"
- board text removed: "C6"
- board text removed: "C7"
- board text removed: "D1"
- board text removed: "D14"
- board text removed: "D15"
- board text removed: "D2"
- board text removed: "F1"
- board text removed: "F2"
- board text removed: "F3"
- board text removed: "FB2"
- board text removed: "FB3"
- board text removed: "FB4"
- board text removed: "J1"
- board text removed: "J2"
- board text removed: "J3"
- board text removed: "JP1"
- board text removed: "L1"
- board text removed: "L2"
- board text removed: "R11"
- board text removed: "R14"
- board text removed: "R25"
- board text removed: "R26"
- board text removed: "R27"
- board text removed: "R31"
- board text removed: "R34"
- board text removed: "R52"
- board text removed: "R56"
- board text removed: "R57"
- board text removed: "R58"
- board text removed: "R59"
- board text removed: "R6"
- board text removed: "R60"
- board text removed: "R62"
- board text removed: "R63"
- board text removed: "R8"
- board text removed: "R9"
- board text removed: "RV1"
- board text removed: "RV3"
- board text removed: "RV4"
- board text removed: "U12"
- board text removed: "U15"
- board text removed: "U2"
- board text removed: "U3"
- board text removed: "U4"
- board text removed: "U5"
- board text removed: "U7"
- board text removed: "WOODY mod-main"
- board text removed: "rev A 2026-10-02"

Commit message: module-main: placed for the iso board and free-routed under the owner's policy - 31 connections left (#22)
Free routing (no direction per layer) on layers 1, 3 and 4 after the iso split:
31 unrouted (11 the DAC's), three shorts and two crossings the router left in
the load switch, five connect_first runs not laid. README status says so.

Gate-Red: module-main routing incomplete (31 unrouted, shorts in the load switch) - the open item of #22; the body branch's stale CAD outputs are not this change's
Co-Authored-By: Claude Opus 5.5 <noreply@anthropic.com>
Claude-Session: https://claude.ai/code/session_01LmB4muFXnoLprWX4JzuJ5A
Parts:
- removed H7: MECH-STANDOFF-ISO 3, MountingHole:MountingHole_3.2mm_M3_Pad
- D11: moved to F.Cu
- moved H6 40.9 mm to (105.7, 69.9)
- moved D11 13.8 mm to (69.0, 66.2), turned to -90 degrees
Routing:
- net MODULE_ANALOG_POS12: track 0.00 -> 273.9 mm, vias 0 -> 29
- net MODULE_ANALOG_NEG12: track 0.00 -> 196.9 mm, vias 0 -> 22
- net /pitch-stage/AMP_OUT: track 0.00 -> 169.7 mm, vias 0 -> 8
- net /pitch-stage/VREF_BUFFERED: track 0.00 -> 126.4 mm, vias 0 -> 3
- net /DAC_AVDD: track 0.00 -> 108.1 mm, vias 0 -> 4
- net AGND_MOD: track 0.00 -> 105.1 mm, vias 0 -> 58
- net /BREATH_SENSE: track 0.00 -> 96.3 mm, vias 0 -> 3
- net /AGND_SENSE: track 0.00 -> 90.2 mm, vias 0 -> 1
- net /VREFOUT: track 0.00 -> 75.3 mm, vias 0 -> 5
- net /power-entry/NEG12_PTC3: track 0.00 -> 56.6 mm, vias 0 -> 1
- net /MOD3_JACK: track 0.00 -> 52.8 mm, vias 0 -> 4
- net /digital-and-supervision/SCLK_BUF: track 0.00 -> 43.9 mm, vias 0 -> 3
- net /RESP_V_SHAPED: track 0.00 -> 43.8 mm, vias 0 -> 6
- net /digital-and-supervision/CS_BUF: track 0.00 -> 42.3 mm, vias 0 -> 3
- net /mod-channels/VREF_MOD: track 0.00 -> 38.5 mm, vias 0 -> 4
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Other:
- board text added: "C12"
- board text added: "C18"
- board text added: "C19"
- board text added: "C20"
- board text added: "C24"
- board text added: "C27"
- board text added: "C29"
- board text added: "C3"
- board text added: "C38"
- board text added: "C43"
- board text added: "C49"
- board text added: "C51"
- board text added: "C6"
- board text added: "C7"
- board text added: "C9"
- board text added: "D1"
- board text added: "D10"
- board text added: "D14"
- board text added: "D15"
- board text added: "D2"
- board text added: "D4"
- board text added: "D6"
- board text added: "D8"
- board text added: "F1"
- board text added: "F2"
- board text added: "F3"
- board text added: "FB1"
- board text added: "FB2"
- board text added: "FB4"
- board text added: "J1"
- board text added: "J2"
- board text added: "J3"
- board text added: "J4"
- board text added: "J5"
- board text added: "JP1"
- board text added: "Q1"
- board text added: "R10"
- board text added: "R11"
- board text added: "R12"
- board text added: "R14"
- board text added: "R15"
- board text added: "R21"
- board text added: "R24"
- board text added: "R26"
- board text added: "R27"
- board text added: "R28"
- board text added: "R29"
- board text added: "R31"
- board text added: "R33"
- board text added: "R34"
- board text added: "R35"
- board text added: "R4"
- board text added: "R42"
- board text added: "R52"
- board text added: "R56"
- board text added: "R57"
- board text added: "R58"
- board text added: "R59"
- board text added: "R6"
- board text added: "R60"
- board text added: "R62"
- board text added: "R63"
- board text added: "R66"
- board text added: "R69"
- board text added: "R8"
- board text added: "R9"
- board text added: "RN1"
- board text added: "RV1"
- board text added: "RV2"
- board text added: "RV3"
- board text added: "SW1"
- board text added: "U1"
- board text added: "U12"
- board text added: "U15"
- board text added: "U2"
- board text added: "U5"
- board text added: "U9"
- board text added: "rev A 2026-10-02"
