File: hardware/boards/module-jack/module-jack.kicad_sch (KiCad schematic)
At the start: 3 parts, among them J7 2x10 2.54mm pin header

Commit message: module-jack: renders and fab; 3D models for the 2x10 header and the PJ398SM
setup-env fetches KiCad's 2x10 header model and installs the banked community
PJ398SM model under the name KiCad's footprint gives it (KiCad ships none).
layout.yaml models: moves that model onto the footprint's sleeve pad and turns
J7's header over so its insulator is on the board's rear. J7 on the jack sheet
is excluded from the BOM (one header is bought; the sheet already marked it
Assembly none). pcb.py render writes the ledger.

Co-Authored-By: Claude Opus 5.5 <noreply@anthropic.com>
Claude-Session: https://claude.ai/code/session_01LmB4muFXnoLprWX4JzuJ5A
Parts:
- J7: now left out of the parts list
Changed lines of the file:
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@@
   (label "AGND_MOD" (at 53.34 106.68 270) (fields_autoplaced) (effects (font (size 1.27 1.27)) (justify right bottom)))
   (symbol (lib_id "Connector_Generic:Conn_02x10_Odd_Even") (at 106.68 63.5 0) (unit 1)
-    (in_bom yes) (on_board yes) (dnp no)
+    (in_bom no) (on_board yes) (dnp no)
     (property "Reference" "J7" (at 107.95 50.8 0) (effects (font (size 1.27 1.27))))
     (property "Value" "2x10 2.54mm pin header" (at 107.95 78.74 0) (effects (font (size 1.27 1.27))))
