File: hardware/boards/main-board/.rescue-w1xcu14g/main-board.kicad_pcb (KiCad board)
At the start: 4 copper layers, 292.4 x 42 mm, 154 parts, among them J1 2x12 1.27mm shrouded box head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, J2 1x5, J4 12-way, J5 12-way, J6 8-way 2.54mm right-angle pin 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, Q1 AO3401A, SW1 KS-33, SW2 KS-33, SW3 KS-33, SW4 KS-33, SW5 KS-33, SW6 KS-33, SW7 KS-33, SW8 KS-33, U1 SP0504BAHT or equivalent 4-ch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, U10 MPXV4006DP, U11 SP0504BAHTG 4-channel 5V array, U2 MCP3202-CI/SN, U3 OPA2197IDR, U4 REF5050IDR, U5 R-78E5.0-1.0, U6 74AHCT125, U7 74HCS165, U8 74HCS165, U9 SP0504BAHTG 4-channel 5V array

Commit message: #8: main board routed on the far-edge breath corridor with arcs (14 connections left for finish)
Gate-Red: main-board routing in progress (pair ends, VS at the mouth, U7 3V3, J-MCU 5V left); photo/clash/CAD renders stale; module-iso coverage row is another branch's

Co-Authored-By: Claude Opus 5.5 <noreply@anthropic.com>
Claude-Session: https://claude.ai/code/session_01LmB4muFXnoLprWX4JzuJ5A
Routing:
- net DEV_3V3: track 483.4 -> 467.4 mm
- net /IO33: track 44.6 -> 32.0 mm
- net INST_5V_A: track 40.9 -> 50.6 mm
Changed lines of the file:
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@@
 	)
 	(segment
-		(start 314.3 140.1)
-		(end 326.1 140.1)
-		(width 0.25)
-		(layer "B.Cu")
-		(net 17)
-	)
-	(segment
 		(start 296.9 122.7)
 		(end 314.3 140.1)
@@
 	)
 	(segment
-		(start 326.1 140.1)
-		(end 326.7 139.5)
-		(width 0.25)
-		(layer "B.Cu")
-		(net 17)
-	)
-	(segment
 		(start 296.9 117.3)
 		(end 296.9 122.7)
@@
 	)
 	(segment
-		(start 323.1 139.5)
-		(end 323.1 139.7)
-		(width 0.3)
-		(layer "F.Cu")
-		(net 82)
-	)
-	(segment
 		(start 91.1 127.1)
 		(end 90.7 126.7)
@@
 	)
 	(segment
-		(start 322.3 140.1)
-		(end 322.9 139.5)
-		(width 0.3)
-		(layer "F.Cu")
-		(net 82)
-	)
-	(segment
 		(start 124.5 110.9)
 		(end 123.3 109.7)
@@
 	)
 	(segment
-		(start 314.3 140.1)
-		(end 322.3 140.1)
-		(width 0.3)
-		(layer "F.Cu")
-		(net 82)
-	)
-	(segment
 		(start 115.3 103.5)
 		(end 115.3 103.3)
@@
 	)
 	(segment
-		(start 323.1 139.7)
-		(end 323.5 140.1)
-		(width 0.3)
-		(layer "F.Cu")
-		(net 82)
-	)
-	(segment
 		(start 222.5 141.3)
 		(end 215.5 141.3)
@@
 	)
 	(segment
-		(start 323.5 140.1)
-		(end 329.9 140.1)
-		(width 0.3)
-		(layer "F.Cu")
-		(net 82)
-	)
-	(segment
 		(start 247.84 130.44)
 		(end 248.38 129.9)
@@
 	)
 	(segment
+		(start 325.3 139.9)
+		(end 325.3 139.5)
+		(width 0.5)
+		(layer "F.Cu")
+		(net 83)
+	)
+	(segment
+		(start 324.9 140.3)
+		(end 325.3 139.9)
+		(width 0.5)
+		(layer "F.Cu")
+		(net 83)
+	)
+	(segment
 		(start 314.9 138.5)
 		(end 314.3 138.5)
@@
 	)
 	(segment
+		(start 316.7 139.9)
+		(end 317.1 140.3)
+		(width 0.5)
+		(layer "F.Cu")
+		(net 83)
+	)
+	(segment
 		(start 292.9 129.5)
 		(end 293.9 129.5)
@@
 	)
 	(segment
+		(start 317.1 140.3)
+		(end 324.9 140.3)
+		(width 0.5)
+		(layer "F.Cu")
+		(net 83)
+	)
+	(segment
 		(start 315.7 138.7)
 		(end 316.1 138.7)
@@
 		(width 0.5)
 		(layer "F.Cu")
+		(net 83)
+	)
+	(segment
+		(start 316.7 139.5)
+		(end 316.7 139.9)
+		(width 0.5)
+		(layer "F.Cu")
