File: hardware/module/breath-output-stage/breath-output-stage.kicad_sch (KiCad schematic)
At the start: 0 parts

Commit message: Breath response shaper adopted: restoring half drawn, output feeds POT-GAIN; pots ordered to fit the knob
U-RESP B restores x2 inverting (R-RESTORE-IN 10k, R-RESTORE-FB 20k): unity and
the in-amp's polarity at centre detent. BREATH_SHAPED feeds POT-GAIN on
J-B2B-MOD pin 1; nets.yaml moves the shaper from proposed to fitted.
POT-GAIN linear (the design's working gain sits at noon); POT-OFFSET gets no
detent. POT-GAIN/OFFSET are Song Huei R0904N KC (18-tooth, the T18 knob's
shaft; KQ is 40-tooth); POT-RESP Alpha RV09AF-40-25B-B50K-0C (18-tooth B shaft,
centre click). POT-OFFSET's zero is +18.7 deg on the 280-deg track, not 300.

Co-Authored-By: Claude Opus 5.5 <noreply@anthropic.com>
Claude-Session: https://claude.ai/code/session_01LmB4muFXnoLprWX4JzuJ5A
Other:
- sheet jack ports: added BREATH_SHAPED; removed BREATH_INAMP_OUT
Changed lines of the file:
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@@
     (property "Sheetname" "jack" (at 203.2 49.53 0) (effects (font (size 1.27 1.27)) (justify left bottom)))
     (property "Sheetfile" "breath-output-stage.jack.kicad_sch" (at 203.2 73.66 0) (effects (font (size 1.27 1.27)) (justify left top)))
-    (pin "BREATH_INAMP_OUT" input (at 264.16 53.34 0) (effects (font (size 1.27 1.27)) (justify right)))
+    (pin "BREATH_SHAPED" input (at 264.16 53.34 0) (effects (font (size 1.27 1.27)) (justify right)))
     (pin "GAIN_FLOOR" passive (at 264.16 55.88 0) (effects (font (size 1.27 1.27)) (justify right)))
     (pin "GAIN_WIPER" passive (at 264.16 58.42 0) (effects (font (size 1.27 1.27)) (justify right)))
@@
   )
   (wire (pts (xy 264.16 53.34) (xy 269.24 53.34)) (stroke (width 0) (type default)))
-  (hierarchical_label "BREATH_INAMP_OUT" (shape input) (at 269.24 53.34 0) (effects (font (size 1.27 1.27)) (justify left))
+  (hierarchical_label "BREATH_SHAPED" (shape input) (at 269.24 53.34 0) (effects (font (size 1.27 1.27)) (justify left))
     (property "Dir" "in" (at 269.24 53.34 0) (effects (font (size 1.27 1.27)) hide))
-    (property "From" "module/breath-receive-stage" (at 269.24 53.34 0) (effects (font (size 1.27 1.27)) hide))
-    (property "Note" "0 to inamp-full-scale, rest at 0" (at 269.24 53.34 0) (effects (font (size 1.27 1.27)) hide)))
+    (property "From" "module/breath-response-shaper" (at 269.24 53.34 0) (effects (font (size 1.27 1.27)) hide))
+    (property "Note" "The in-amp's output after the response shaper: equal to it at centre detent" (at 269.24 53.34 0) (effects (font (size 1.27 1.27)) hide)))
   (wire (pts (xy 264.16 55.88) (xy 269.24 55.88)) (stroke (width 0) (type default)))
   (label "GAIN_FLOOR" (at 269.24 55.88 0) (fields_autoplaced) (effects (font (size 1.27 1.27)) (justify left bottom)))

Commit message: #32: checkpoint — switchable breath band-limit, 1.5 kHz ADC filter, breath LED
Receive stage: C_diff switched by U-BW-SW (TMUX6112) from SW-BREATH-BW
(NKK M2024, left 500 Hz / centre 1.5 kHz / right WIDE): 680 pF fixed,
3.9 nF and 10 nF switched; C_cm 68 pF matched pair. C-OUT-BREATH 10 nF C0G.
C-AA-ADC 18 nF (1.47 kHz), sample rate kept at 4 kHz. Breath LED driver on
U-REF-BUF B. Sheets, BOM fragments, datasheets (TMUX6112, MMBT3904), sims,
ADR 0003/0004 amendments, pages. Sims still being re-run.

Gate-Red: sims stale while re-running (breath-receive-stage, breath-output-stage, interfaces/system, pitch-stage); breath-sense-link/sim pg_gain_max < 1e-3 fails in every mode and power-entry/sim led-pwm breath_mv fails at 2 kHz - both consequences of #32 left for the owner, not loosened; breath-receive-stage cmrr-wide fails 58.5 dB above ~7.4 kHz (owner); kicad: module-main and main-board .kicad_pcb parity broken by the new/changed parts (re-placement is the module re-layout's; pcb not touched), plus module-main's pre-existing routing failures

Co-Authored-By: Claude Opus 5.5 <noreply@anthropic.com>
Claude-Session: https://claude.ai/code/session_01LmB4muFXnoLprWX4JzuJ5A
Other:
- sheet jack ports: added BREATH_OUT; removed none
Changed lines of the file:
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@@
     (pin "GAIN_WIPER" passive (at 264.16 58.42 0) (effects (font (size 1.27 1.27)) (justify right)))
     (pin "DAC_AVDD" input (at 264.16 60.96 0) (effects (font (size 1.27 1.27)) (justify right)))
+    (pin "BREATH_OUT" output (at 264.16 71.12 0) (effects (font (size 1.27 1.27)) (justify right)))
     (pin "OFFSET_WIPER" passive (at 264.16 63.5 0) (effects (font (size 1.27 1.27)) (justify right)))
     (pin "JACK_TIP" passive (at 264.16 66.04 0) (effects (font (size 1.27 1.27)) (justify right)))
@@
     (property "From" "module/power-entry" (at 269.24 68.58 0) (effects (font (size 1.27 1.27)) hide)))
   (text "FROM THE HAND-WRITTEN NETLIST THIS SHEET REPLACES (verbatim; the part notes are on each part's Note field):\n\nAUTHORITATIVE for connectivity. The ASCII drawing in breath-output-stage.md is a REPRESENTATION of this file,\nnot the other way round.\n\nHand-authored YAML is the first step and KiCad is generated from it later, so this is the file to edit. If\nthis and the drawing disagree, THIS WINS and the drawing is the defect - see hardware/README.md.\n\ntools/check-netlist.py proves: every refdes here exists in bom.csv with a matching value; every net has at\nleast two endpoints; every declared pin is used exactly once; and every `[REFDES value]` label in the page's\ndrawing agrees with this file.\n\nNets that cross this circuit's boundary. These must match the page's ## Interfaces table - that table is how a\nreader matches the two.\n\n[pins] CW = signal end, CCW = floor end\n\n[U-BREATH-OPA] ONE OPA2197 PACKAGE, BOTH HALVES: A buffers the gain pot's wiper, B is the summer. Its supply\npins are netted, with one C-DECOUPLE at each.\n\n[pins] dual series diode: anode, cathode, common\n\nTHE CLAMP'S RAILS ARE THE MODULE'S SUPPLY: \"D-JACK-CLAMP returns to both rails\" (the page's Interfaces table),\nnetted as pitch-stage and mod-channels net theirs." (at 40.64 147.32 0) (effects (font (size 1.27 1.27)) (justify left top)))
+  (wire (pts (xy 264.16 71.12) (xy 269.24 71.12)) (stroke (width 0) (type default)))
+  (hierarchical_label "BREATH_OUT" (shape output) (at 269.24 71.12 0) (effects (font (size 1.27 1.27)) (justify left))
+    (property "Dir" "out" (at 269.24 71.12 0) (effects (font (size 1.27 1.27)) hide))
+    (property "To" "module/breath-receive-stage" (at 269.24 71.12 0) (effects (font (size 1.27 1.27)) hide))
+    (property "Note" "The summer's output inside its loop, ahead of R-OUT-PROT: the breath LED's driver reads it (#32)" (at 269.24 71.12 0) (effects (font (size 1.27 1.27)) hide)))
   (text "THIS CIRCUIT IS ON BOTH MODULE BOARDS (ADR 0023). Page main holds its main-board parts, page jack the parts behind the panel; the labels here join the two pages, and on the boards J-B2B-MOD joins them. Each board places its own page." (at 60.96 30.48 0) (effects (font (size 1.27 1.27)) (justify left top)))
   (sheet_instances (path "/" (page "1")))
