File: hardware/module/breath-receive-stage/breath-receive-stage.kicad_sch (KiCad schematic)
At the start: 18 parts

Commit message: #32: checkpoint — switchable breath band-limit, 1.5 kHz ADC filter, breath LED
Receive stage: C_diff switched by U-BW-SW (TMUX6112) from SW-BREATH-BW
(NKK M2024, left 500 Hz / centre 1.5 kHz / right WIDE): 680 pF fixed,
3.9 nF and 10 nF switched; C_cm 68 pF matched pair. C-OUT-BREATH 10 nF C0G.
C-AA-ADC 18 nF (1.47 kHz), sample rate kept at 4 kHz. Breath LED driver on
U-REF-BUF B. Sheets, BOM fragments, datasheets (TMUX6112, MMBT3904), sims,
ADR 0003/0004 amendments, pages. Sims still being re-run.

Gate-Red: sims stale while re-running (breath-receive-stage, breath-output-stage, interfaces/system, pitch-stage); breath-sense-link/sim pg_gain_max < 1e-3 fails in every mode and power-entry/sim led-pwm breath_mv fails at 2 kHz - both consequences of #32 left for the owner, not loosened; breath-receive-stage cmrr-wide fails 58.5 dB above ~7.4 kHz (owner); kicad: module-main and main-board .kicad_pcb parity broken by the new/changed parts (re-placement is the module re-layout's; pcb not touched), plus module-main's pre-existing routing failures

Co-Authored-By: Claude Opus 5.5 <noreply@anthropic.com>
Claude-Session: https://claude.ai/code/session_01LmB4muFXnoLprWX4JzuJ5A
Parts:
- added C-BW-FILT0, C-BW-FILT1, C-DEC-BWSW-NEG, C-DEC-BWSW-POS: 100nF, Capacitor_SMD:C_0805_2012Metric, symbol Device:C
- added C-DIFF-BW-1K5: 3.9nF, Capacitor_SMD:C_0805_2012Metric, symbol Device:C
- added C-DIFF-BW-500: 10nF, Capacitor_SMD:C_0805_2012Metric, symbol Device:C
- added D-LEDB: 1N4448W, Diode_SMD:D_SOD-123, symbol Diode:1N4148W
- added J-LED-BREATH: JST B2B-XH-A, Connector_JST:JST_XH_B2B-XH-A_1x02_P2.50mm_Vertical, symbol Connector_Generic:Conn_01x02
- added LED-BREATH: 605-2211-110F, symbol Device:LED
- added Q-LEDB: MMBT3904, Package_TO_SOT_SMD:SOT-23, symbol Transistor_BJT:MMBT3904
- added R-BW-COM: 4.7k 1%, Resistor_SMD:R_0805_2012Metric, symbol Device:R
- added R-BW-FILT0, R-BW-FILT1, R-LEDB-TOP: 100k 1%, Resistor_SMD:R_0805_2012Metric, symbol Device:R
- added R-BW-PD0, R-BW-PD1, R-LEDB-BOT: 10k 1%, Resistor_SMD:R_0805_2012Metric, symbol Device:R
- added R-LEDB-A: 1k 1% 1206, Resistor_SMD:R_1206_3216Metric, symbol Device:R
- added R-LEDB-BASE: 1k 1%, Resistor_SMD:R_0805_2012Metric, symbol Device:R
- added R-LEDB-SENSE: 180R 1%, Resistor_SMD:R_0805_2012Metric, symbol Device:R
- added SW-BREATH-BW: NKK M2024SD4G01, Connector_Wire:SolderWire-0.25sqmm_1x03_P4.2mm_D0.65mm_OD1.7mm, symbol woody:SW_NKK_M2024_wired
- added U-BW-SW: TMUX6112PWR, Package_SO:TSSOP-16_4.4x5mm_P0.65mm, symbol woody:TMUX6112xPW
- C-CM-IN+, C-CM-IN-: value 1.5nF -> 68pF; LCSC C541572 -> C541517; MPN CC0805FRNPO9BN152 -> CC0805FRNPO9BN680; Note A MATCHED PAIR with its twin (owner, 2026-10-03: 'Tighten cap matching'): C-CM-IN+ and C-CM-IN- from one reel of the 1 % C0G part, measured on one LCR meter at 1 kHz and fitted together only when each is within 0.5 % of the pair's mean. Their mismatch converts the umbilical's common mode in proportion to frequency, and at 1 % each the link misses its CMRR at the breath band's top (module/breath-receive-stage/sim cmrr-as-netlisted). No catalogue C0G at 1.5 nF is sold tighter than 1 %, so the match is made by hand: fitted by hand, after measuring -> A MATCHED PAIR with its twin (owner, 2026-10-03: 'Tighten cap matching'; 68 pF since #32): C-CM-IN+ and C-CM-IN- from one reel of the 1 % C0G part, measured on one LCR meter (open-circuit compensated, at 100 kHz if it has it) and fitted together only when each is within 0.5 % of the pair's mean. Their mismatch converts the umbilical's common mode in proportion to frequency, so it sets each bandwidth mode's CMRR at its top (module/breath-receive-stage/sim cmrr-*). The 1 % C0G is the tightest catalogued, so the match is made by hand: fitted by hand, after measuring. Fixed in every mode of the bandwidth toggle
- C-DIFF-BREATH: value 15nF -> 680pF; LCSC C445728 -> C107121; MPN C2012C0G1H153JT000N -> CC0805JRNPO9BN681; Manufacturer TDK -> YAGEO
- U-REF-BUF: Note Half A buffers the trimmer wiper into the in-amp REF pin: a bare divider there degrades CMRR one-for-one. Half B is spare, a follower with its input on the star -> Half A buffers the trimmer wiper into the in-amp REF pin: a bare divider there degrades CMRR one-for-one. Half B drives the breath LED (since 2026-10-04, #32): its (+) input takes BREATH_OUT/11 from R-LEDB-TOP/R-LEDB-BOT and its loop holds Q-LEDB's emitter there, so the LED current follows the jack
Connections:
- net AGND_MOD: now also C-BW-FILT0.2, C-BW-FILT1.2, C-DEC-BWSW-NEG.2, C-DEC-BWSW-POS.2, R-BW-PD0.2, R-BW-PD1.2, R-LEDB-BOT.2, R-LEDB-SENSE.2, U-BW-SW.5 (GND); no longer U-REF-BUF.5 (+)
- net IN_NEG: now also U-BW-SW.15 (D2), U-BW-SW.7 (D4)
- net IN_POS: now also U-BW-SW.10 (D3), U-BW-SW.2 (D1)
- net MODULE_ANALOG_NEG12: now also C-DEC-BWSW-NEG.1, U-BW-SW.4 (VSS)
- net MODULE_ANALOG_POS12: now also C-DEC-BWSW-POS.1, R-BW-COM.1, R-LEDB-A.1, U-BW-SW.13 (VDD)
- net SPARE_B_OUT renamed LEDB_DRV
- net LEDB_DRV: now also R-LEDB-BASE.1; no longer U-REF-BUF.6 (-)
- new net BREATH_OUT: R-LEDB-TOP.1
- new net BW0: C-BW-FILT0.1, R-BW-FILT0.2, U-BW-SW.8 (SEL4), U-BW-SW.9 (SEL3)
- new net BW0_SW: R-BW-FILT0.1, R-BW-PD0.1, SW-BREATH-BW.3 (L1)
- new net BW1: C-BW-FILT1.1, R-BW-FILT1.2, U-BW-SW.1 (SEL1), U-BW-SW.16 (SEL2)
- new net BW1_SW: R-BW-FILT1.1, R-BW-PD1.1, SW-BREATH-BW.2 (L4)
- new net BW_COM: R-BW-COM.2, SW-BREATH-BW.1 (COM)
- new net CBW1K5_N: C-DIFF-BW-1K5.2, U-BW-SW.14 (S2)
- new net CBW1K5_P: C-DIFF-BW-1K5.1, U-BW-SW.3 (S1)
- new net CBW500_N: C-DIFF-BW-500.2, U-BW-SW.6 (S4)
- new net CBW500_P: C-DIFF-BW-500.1, U-BW-SW.11 (S3)
- new net LEDB_A: J-LED-BREATH.1 (Pin_1), LED-BREATH.2 (A), R-LEDB-A.2
- new net LEDB_B: D-LEDB.1 (K), Q-LEDB.1 (B)
- new net LEDB_D: D-LEDB.2 (A), R-LEDB-BASE.2
- new net LEDB_IN: R-LEDB-BOT.1, R-LEDB-TOP.2, U-REF-BUF.5 (+)
- new net LEDB_K: J-LED-BREATH.2 (Pin_2), LED-BREATH.1 (K), Q-LEDB.3 (C)
- new net LEDB_SENSE: Q-LEDB.2 (E), R-LEDB-SENSE.1, U-REF-BUF.6 (-)
- no-connect marks 0 -> 1

Commit message: #32: checkpoint - the owner's three answers and side-adjust trimmers
Owner decisions of 2026-10-04, recorded in ADR 0003/0004/0023/0024:
- WIDE's CMRR requirement band is DC to 7 kHz ("Keep 10 kHz, accept");
  cmrr-wide holds 58.5 dB there and records 10 kHz.
- D-TVS-BREATH is the PESD12VL1BA (19 pF), datasheet banked; PWR_GND
  held under -60 dB in each mode's band, WIDE at the accepted figure.
- The -12 V offset leg is filtered: R-BREATH-OFFNEG-A/-B 47.5k with
  C-BREATH-OFFNEG 1 uF at the split (6.7 Hz). Rest level +16 mV.
- The four trimmers are Bourns 3296X side-adjust, set with the module
  out of the rack; no rear-access windows. Current 3296 datasheet banked.

Sims are mid-run; their results land in the next commit.

Gate-Red: sim results stale or pre-change for receive-stage, power-entry, pitch-stage, mod-channels, shaper, system, breath-excitation-reference, digital-and-supervision and panel-led while they re-run on these inputs (checkpoint, as asked every 45 min); module-main and main-board .kicad_pcb parity with the new/changed parts (layout's, not touched here); main-board fab stale against the breath-adc sheet; module-main's existing routing/silk/acid-trap failures.

Co-Authored-By: Claude Opus 5.5 <noreply@anthropic.com>
Claude-Session: https://claude.ai/code/session_01LmB4muFXnoLprWX4JzuJ5A
Parts:
- TRIM-BREATH-ZERO: footprint Potentiometer_THT:Potentiometer_Bourns_3296W_Vertical -> Potentiometer_THT:Potentiometer_Bourns_3296X_Horizontal; LCSC C34846 -> C111776; MPN 3296W-1-103LF -> 3296X-1-103LF
Changed lines of the file:
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@@
     (property "Reference" "TRIM-BREATH-ZERO" (at 91.44 317.5 0) (effects (font (size 1.27 1.27))))
     (property "Value" "10k multiturn cermet" (at 91.44 320.04 0) (effects (font (size 1.27 1.27))))
-    (property "Footprint" "Potentiometer_THT:Potentiometer_Bourns_3296W_Vertical" (at 91.44 325.12 0) (effects (font (size 1.27 1.27)) hide))
+    (property "Footprint" "Potentiometer_THT:Potentiometer_Bourns_3296X_Horizontal" (at 91.44 325.12 0) (effects (font (size 1.27 1.27)) hide))
     (property "Datasheet" "" (at 91.44 325.12 0) (effects (font (size 1.27 1.27)) hide))
     (property "Row" "TRIM-BREATH-ZERO" (at 91.44 325.12 0) (effects (font (size 1.27 1.27)) hide))
@@
     (property "Pins_source" "datasheets/discrete-and-power/BOURNS-3296-TRIMPOT.pdf p.1 circuit: 1 CCW, 2 wiper, 3 CW" (at 91.44 325.12 0) (effects (font (size 1.27 1.27)) hide))
     (property "Manufacturer" "Bourns" (at 91.44 325.12 0) (effects (font (size 1.27 1.27)) hide))
-    (property "MPN" "3296W-1-103LF" (at 91.44 325.12 0) (effects (font (size 1.27 1.27)) hide))
-    (property "LCSC" "C34846" (at 91.44 325.12 0) (effects (font (size 1.27 1.27)) hide))
+    (property "MPN" "3296X-1-103LF" (at 91.44 325.12 0) (effects (font (size 1.27 1.27)) hide))
+    (property "LCSC" "C111776" (at 91.44 325.12 0) (effects (font (size 1.27 1.27)) hide))
     (property "Assembly" "hand" (at 91.44 325.12 0) (effects (font (size 1.27 1.27)) hide))
     (pin "1")
