File: hardware/interfaces/breath-sense-link/breath-sense-link.kicad_sch (KiCad schematic)
At the start: 8 parts

Commit message: BOM review (issue #7): ST owns the breath sensor, order routes, status held to the sheets, two gaps banked
#7-1  U-BREATH: manufacturer STMicroelectronics (ex-NXP) on the row and the
      sheet; the row's supply note replaced with the 2026-10-03 stock and
      route [web], the 2028 promise retired as NXP's (ADR 0003 amended).
      AN3150 banked from the Wayback raw capture: 245 degC max on an MPXV DP,
      no-clean flux, no washing - the row and breath-sense-link.md now carry
      the soldering conditions instead of "open". ST's datasheet (DS15256)
      recorded BLOCKED with every URL tried.
#7-2  FB-IN: Global Sourcing verified possible (DigiKey 378k) and cited;
      status selected. Sheet already said so; unchanged.
#7-3  U-BUCK: buy route DigiKey 945-2201-ND; LCSC named only as the place
      not to buy; sheet LCSC field cleared (hand-fitted, no tool reads it).
#7-4  U-LOADSW: ADI lists PRODUCTION (archived product page); stock and
      route refreshed. Part unchanged.
#7-6  merge-bom.py --check fails a candidate/open row whose part a sheet
      names (ADR 0019); 58 rows promoted to selected; PCB-CLUSTER selected
      (fab packs pass), PCB-CARRIER/PCB-UMB-ADAPTER say what closes them.
#7-8  J-UMB and J-B2B-MOD: buy once, on two boards' hand lists.
#7-12 merge-manifests.py: RETIRES THE BLOCKED ROW '<part>' counts as a
      declaration, and a LIVE line counts open gaps; TE 36149 product sheet
      banked (OK-SUBSTITUTE).

Co-Authored-By: Claude Opus 5.5 <noreply@anthropic.com>
Claude-Session: https://claude.ai/code/session_01LmB4muFXnoLprWX4JzuJ5A
Parts:
- U-BREATH: Manufacturer NXP -> STMicroelectronics
Changed lines of the file:
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@@
     (property "Note" "SOLDERED TO THE MAIN BOARD, no socket (case 1351-01 is surface mount). Pin 2 VS, pin 3 GND, pin 4 VOUT; pins 1 and 5-8 are N/C and carry no net (Style 2 - breath-sense-link.md, Mounting). P1 takes the breath tube with its PTFE plug and its <=1 mL trap; P2 IS OPEN TO THE CAVITY AND MUST NEVER BE BLOCKED. Neither is a net, so neither is here - which is exactly the kind of fact a netlist cannot carry and the page must" (at 76.2 101.6 0) (effects (font (size 1.27 1.27)) hide))
     (property "Pins_source" "datasheets/analog/MPXV4006DP.pdf, case 1351-01 Style 2: pin 2 VS, 3 GND, 4 VOUT, 1 and 5-8 N/C - the same 8-lead pinout as KiCad's MPXA6115A" (at 76.2 101.6 0) (effects (font (size 1.27 1.27)) hide))
-    (property "Manufacturer" "NXP" (at 76.2 101.6 0) (effects (font (size 1.27 1.27)) hide))
+    (property "Manufacturer" "STMicroelectronics" (at 76.2 101.6 0) (effects (font (size 1.27 1.27)) hide))
     (property "MPN" "MPXV4006DP" (at 76.2 101.6 0) (effects (font (size 1.27 1.27)) hide))
     (property "LCSC" "C5190605" (at 76.2 101.6 0) (effects (font (size 1.27 1.27)) hide))

Commit message: Owner decisions D1, D2, D3, D5, CMRR: the parts on the sheets (#11, #14, #15, #16, #5, #12)
The owner's choices of 2026-10-03 (working chat), applied to the KiCad sheets,
exported, rendered, and carried into the BOM fragments:

- D1 (#11 F2, #14 A1, #12-3), "10 ohm + 22 uF + 10 uF": breath-adc gains
  R-ADC-VDD (10R 1% 0805, UNI-ROYAL 0805W8F100JT5E, C17415, JLC basic) from
  DEV_3V3 to a new local net ADC_VDD = U-ADC pin 8, with C-ADC-VDD (22 uF
  X5R 25 V 1206, Samsung CL31A226KAHNNNE, C12891, JLC basic) beside the
  existing C-ADC-BULK and C-DEC-ADC (C3 kept); a PWR_FLAG on ADC_VDD for
  ERC. power-entry-instrument gains C-BUCK-OUT (10 uF X5R 50 V 1206,
  Samsung CL31A106KBHNNNE, C13585, JLC basic) at U-BUCK-A's OUT (main-board
  U5, the R-78E5.0 - RECOM's standard application, #14 A1 item 3).
  Main board: R47, C42, C43.
- D5: U-ADC CH1 tied to AGND_INST.
- D2 (#15 C2, #16 B2), "Yes, all 4 channels": a second SP0504BAHTG at J5
  on CHAIN_SCK, CHAIN_SHLD, HOP_LT_RH, HOP_RH_RT - main-board U11 on the
  root sheet, U-TVS-CHAIN-RH on the key-chain-loom sheet; row qty 2.
- D3 (#15 C3): R-SPI-SER (R1-R3) Panasonic ERJ-P08F82R0V (C4065013, 0 at
  JLC and LCSC; in-stock equivalent Vishay CRCW120682R0FKEAHP, C1854869,
  named in the row); R-SER-BREATH-INST (R38/R39) ERJ-P08F1001V (C4261071,
  JLC 4,299).
- CMRR (#5-5), "Tighten cap matching": C-CM-BREATH a matched pair, each
  within 0.5 % of the pair's mean, from one reel of the 1 % C0G, measured
  and hand-fitted (no 1.5 nF C0G is catalogued tighter than 1 %).

Banked: Samsung CL31A226KAHNNNE and CL31A106KBHNNNE spec sheets, Vishay
CRCW-HP e3 (fragment .manifest-R51-owner-decisions.csv). Also two module
sims the deff676 merge staled and these changes do not touch (panel-led,
digital-and-supervision) re-run: 0 failed.

Gate-Red: sims staled by these netlists are re-running in the next commits; main-board .kicad_pcb awaits wave-3 placement of R47, C42, C43, U11 (and fab/ renders); known stale photos/clash

Co-Authored-By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
Parts:
- R1, R1b: LCSC C4410 -> C4261071; MPN 1206W4F1001T5E -> ERJ-P08F1001V; Manufacturer UNI-ROYAL -> Panasonic
Changed lines of the file:
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@@
     (property "Drawn_as" "R-SER-BREATH-INST" (at 139.7 88.9 0) (effects (font (size 1.27 1.27)) hide))
     (property "Note" "Instrument-side series protection on the BREATH leg. 1206 and >=250mW because a jack fault has to land somewhere" (at 139.7 88.9 0) (effects (font (size 1.27 1.27)) hide))
-    (property "Manufacturer" "UNI-ROYAL" (at 139.7 88.9 0) (effects (font (size 1.27 1.27)) hide))
-    (property "MPN" "1206W4F1001T5E" (at 139.7 88.9 0) (effects (font (size 1.27 1.27)) hide))
-    (property "LCSC" "C4410" (at 139.7 88.9 0) (effects (font (size 1.27 1.27)) hide))
+    (property "Manufacturer" "Panasonic" (at 139.7 88.9 0) (effects (font (size 1.27 1.27)) hide))
+    (property "MPN" "ERJ-P08F1001V" (at 139.7 88.9 0) (effects (font (size 1.27 1.27)) hide))
+    (property "LCSC" "C4261071" (at 139.7 88.9 0) (effects (font (size 1.27 1.27)) hide))
     (property "Assembly" "machine" (at 139.7 88.9 0) (effects (font (size 1.27 1.27)) hide))
     (pin "1")
@@
     (property "Pins" "1=1 2=2" (at 139.7 139.7 0) (effects (font (size 1.27 1.27)) hide))
     (property "Note" "THE TWIN IN THE AGND_SENSE LEG. Without it the return is not matched to the signal leg and the link's CMRR is set by that asymmetry rather than by the in-amp. Its AGND_INST end is a trace of its own from U-BREATH pin 3 (breath-sense-link.md, Where it sits)" (at 139.7 139.7 0) (effects (font (size 1.27 1.27)) hide))
-    (property "Manufacturer" "UNI-ROYAL" (at 139.7 139.7 0) (effects (font (size 1.27 1.27)) hide))
-    (property "MPN" "1206W4F1001T5E" (at 139.7 139.7 0) (effects (font (size 1.27 1.27)) hide))
-    (property "LCSC" "C4410" (at 139.7 139.7 0) (effects (font (size 1.27 1.27)) hide))
+    (property "Manufacturer" "Panasonic" (at 139.7 139.7 0) (effects (font (size 1.27 1.27)) hide))
+    (property "MPN" "ERJ-P08F1001V" (at 139.7 139.7 0) (effects (font (size 1.27 1.27)) hide))
+    (property "LCSC" "C4261071" (at 139.7 139.7 0) (effects (font (size 1.27 1.27)) hide))
     (property "Assembly" "machine" (at 139.7 139.7 0) (effects (font (size 1.27 1.27)) hide))
     (pin "1")

Commit message: #34: owner's decisions on iron room recorded - networks stay moved; U10 accepted, hand-soldered first with a fine tip (Fit column); SW2/SW6/SW8 accepted for rev A
Owner, 2026-10-04 (working chat): "Keep moved" for the key networks;
"Accept, solder sensor first" for U10 against R7/U3. Measured pad to pad on
the board: U10 pin 5 to R7 pad 2 0.80 mm; U10 pins 5-8 to U3's pin-1 row
1.59 mm (courtyards 0.28 / 0.86 mm). The near pins are U10's own no-connect
row 5-8 (its mechanical joints), and they DO face R7 and U3 - the option
text's "its pins face away" is not right; pins 1-4 (NC, VS, GND, Vout) are
the far-edge row with open room. R7 and U3 are machine-fitted, so they are on
the board before U10. A 0.4 mm tip line from each of pins 5-8's outer ends
clears other pads by 0.3 mm only in narrow directions (pin 8 straight down
the board; 6 and 7 within ~15 deg of it; 5 from the mouth end).

- iron_room: except: U10/R7 and U10/U3 with "owner 2026-10-04: accepted;
  hand-solder U10 first with a fine tip" and the measured gaps; SW2/H2,
  SW6/H6 and SW8/J5 "accepted for rev A, check on the boards in hand".
- U-BREATH's sheet symbol has a Fit field (order, 0.8-1.0 mm conical tip,
  polyimide tape on R7/U3, pin by pin, check for bridges); pcb.py writes a
  Fit column on the hand-assembly sheet when any hand part has one (boards
  with none keep their four columns).
- README and tooling.md say so. pcb.py check 0 errors; renders and fab/
  written; check-netlist --strict 0 problems.

Gate-Red: 8 CAD photo renders stale against the board (about 25 min each, not rebuilt here); module-main's pre-existing kicad.py failures and its missing silk title (check_title); module-iso's sim coverage row (another branch).

Co-Authored-By: Claude Opus 5.5 <noreply@anthropic.com>
Claude-Session: https://claude.ai/code/session_01LmB4muFXnoLprWX4JzuJ5A
Parts:
- U-BREATH: Fit (none) -> First of the hand-fitted parts. Fine conical tip, 0.8-1.0 m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
Changed lines of the file:
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@@
     (property "LCSC" "C5190605" (at 76.2 101.6 0) (effects (font (size 1.27 1.27)) hide))
     (property "Assembly" "hand" (at 76.2 101.6 0) (effects (font (size 1.27 1.27)) hide))
+    (property "Fit" "First of the hand-fitted parts. Fine conical tip, 0.8-1.0 mm. Pins 1-4 (NC, VS, GND, Vout: the far-edge row) have open room. Pins 5-8 (no-connect, the mechanical joints) face the machine-fitted R7 (0.80 mm pad to pad, from pin 5) and U3 (1.59 mm, from pins 5-8): mask R7 and U3 with polyimide tape, land the tip on each pin's outer end coming from down the board (pin 5 from the mouth end), one pin at a time - no drag soldering - and check R7 and U3 for bridges after" (at 76.2 101.6 0) (effects (font (size 1.27 1.27)) hide))
     (pin "1")
     (pin "2")
