File: hardware/interfaces/breath-sense-link/breath-sense-link.kicad_sch (KiCad schematic)
At the start: 8 parts

Commit message: #36: no breath trap - one clear tube from the inlet to U-BREATH (owner, 2026-10-05)
Owner (chat, 2026-10-05): "I think we should remove it from the inside and
it's okay to kind of have a longer tube that loops around I think. Also it's
not a diffusion risk because it'll be clear". ADR 0003 amendment of
2026-10-05 records it and the reason (pressure, no flow: the dead-ended run
gathers little).

- config/body.yaml: routing.trap_d/trap_l deleted; routing.tube_id/od (3/32 x
  7/32 clear silicone) and tube_bend_r (tbd) added; inlet.tube_* replaced by
  inlet.inner_barb_* (the inside barb is a Clippard 12843 so one tube grips it
  and P1).
- woody_body.scad: trap solids, trap claim on the mouth length and the
  trap-over-LED note gone (overall length unchanged, 325.8 - the mouth band
  was set by layout.gap); one 'breath tube' along the inlet's axis, an S and
  one U onto P1 at tube_bend_r; drc 'breath tube bends no tighter than
  routing.tube_bend_r', 'breath tube clear of the columns', LED crossing
  re-derived. drc: 0 FAIL.
- BOM (unplaced.csv -> bom.csv): TUBE is the clear tube, no trap; TUBE-INLET
  deleted; INLET-BARB-IN is a 12843; MECH-PTFE no trap.
- Pages brought in line: ADR 0009/0017 inline amendments, carrier.md,
  breath-sense-link.md and its sheet's U-BREATH Note (netlist re-exported,
  sheet re-rendered), latency-budget.md, mechanical README/DESIGN, ROADMAP,
  figures.yaml breath-working-point decided_by; clash-allow, render groups
  and the breakdown-breath title.
- Sims made stale by the Note's re-export, rerun: breath-sense-link,
  breath-excitation-reference, fallback-mpxv7007, breath-output-stage
  (0 failed).

Gate-Red: hardware/module/breath-receive-stage/sim stale from this commit's U-BREATH Note text in the breath-sense-link netlist (no electrical change) - its rerun outlasts a session step, follow-up commit; clash, renders, DXFs, pcb-geometry and photos deferred to the coordinator's one rebuild; system sim and module-iso coverage pre-existing on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
Parts:
- U-BREATH: Note SOLDERED TO THE MAIN BOARD, no socket (case 1351-01 is surface mount). Pin 2 VS, pin 3 GND, pin 4 VOUT; pins 1 and 5-8 are N/C and carry no net (Style 2 - breath-sense-link.md, Mounting). P1 takes the breath tube with its PTFE plug and its <=1 mL trap; P2 IS OPEN TO THE CAVITY AND MUST NEVER BE BLOCKED. Neither is a net, so neither is here - which is exactly the kind of fact a netlist cannot carry and the page must -> SOLDERED TO THE MAIN BOARD, no socket (case 1351-01 is surface mount). Pin 2 VS, pin 3 GND, pin 4 VOUT; pins 1 and 5-8 are N/C and carry no net (Style 2 - breath-sense-link.md, Mounting). P1 takes the clear breath tube with its PTFE plug (no trap, ADR 0003 2026-10-05); P2 IS OPEN TO THE CAVITY AND MUST NEVER BE BLOCKED. Neither is a net, so neither is here - which is exactly the kind of fact a netlist cannot carry and the page must
Changed lines of the file:
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@@
     (property "Row" "U-BREATH" (at 76.2 101.6 0) (effects (font (size 1.27 1.27)) hide))
     (property "Pins" "VS=2(Vcc) VOUT=4(Vout) GND=3(GND)" (at 76.2 101.6 0) (effects (font (size 1.27 1.27)) hide))
-    (property "Note" "SOLDERED TO THE MAIN BOARD, no socket (case 1351-01 is surface mount). Pin 2 VS, pin 3 GND, pin 4 VOUT; pins 1 and 5-8 are N/C and carry no net (Style 2 - breath-sense-link.md, Mounting). P1 takes the breath tube with its PTFE plug and its <=1 mL trap; P2 IS OPEN TO THE CAVITY AND MUST NEVER BE BLOCKED. Neither is a net, so neither is here - which is exactly the kind of fact a netlist cannot carry and the page must" (at 76.2 101.6 0) (effects (font (size 1.27 1.27)) hide))
+    (property "Note" "SOLDERED TO THE MAIN BOARD, no socket (case 1351-01 is surface mount). Pin 2 VS, pin 3 GND, pin 4 VOUT; pins 1 and 5-8 are N/C and carry no net (Style 2 - breath-sense-link.md, Mounting). P1 takes the clear breath tube with its PTFE plug (no trap, ADR 0003 2026-10-05); P2 IS OPEN TO THE CAVITY AND MUST NEVER BE BLOCKED. Neither is a net, so neither is here - which is exactly the kind of fact a netlist cannot carry and the page must" (at 76.2 101.6 0) (effects (font (size 1.27 1.27)) hide))
     (property "Pins_source" "datasheets/analog/MPXV4006DP.pdf, case 1351-01 Style 2: pin 2 VS, 3 GND, 4 VOUT, 1 and 5-8 N/C - the same 8-lead pinout as KiCad's MPXA6115A" (at 76.2 101.6 0) (effects (font (size 1.27 1.27)) hide))
     (property "Manufacturer" "STMicroelectronics" (at 76.2 101.6 0) (effects (font (size 1.27 1.27)) hide))
