File: hardware/boards/matrix-carrier/matrix-carrier.kicad_sch (KiCad schematic)
At the start: 3 parts, among them J1 2x12 1.27mm shrouded box head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, J2 1x10 2.54mm pin header, SMD, J3 1x10 2.54mm pin header, SMD

Commit message: #37: MIDI out circuit, the ribbon's MIDI pair, carrier re-route, ADR 0015 amendment
- hardware/carrier/midi-out/: new circuit (sheet, netlist, BOM, page): CA-033's 5 V row
  from U-LVLSHIFT gates B/C, R-MIDI 220R, FB-MIDI, U-TVS-MIDI, J-MIDI (JST PH SMD),
  J-MIDI-OUT (SJ5-43502PM, panel-mount, no footprint), CBL-MIDI. TRS Type A/B in firmware.
- led-strip-drive: gates B/C drive tip/ring; R-MIDI-PU-T/R 10k to DEV_3V3 (power-on default).
- carrier: IO6 on J-MCU 23 (tip) and IO2 on J-MCU 5 (ring) become ports. J-MCU 24 stays
  unconnected: on the Matrix carrier J-MCU-C pin 1 is boxed in by the hand-routed bus.
- matrix-carrier: IO6 routed J-MCU-C pin 2 -> J2.5 (carrier_routes.py); pcb.py check 0 errors.
- main-board root sheet places midi-out; nets.yaml; BOM fragments; CBL-USB-EXT leaves unplaced.csv.
- tools/merge-bom.py: the new fragment added to ORDER (the tool refuses to write when a
  fragment is not listed); no check changed.
- ADR 0015 amendment, ADR 0012 note, firmware/README.md (config mode/OTA deferred; MIDI out),
  draft design in docs/research/.

Gate-Red: pre-existing at 18d0b5f - 37 stale CAD outputs and kicad 131 problems (main-board/module-main PCB parity and clearance). Also red from this checkpoint: the main board's .kicad_pcb is #35's and is not touched, so J-MIDI, R-MIDI-T/R, FB-MIDI-T/R, U-TVS-MIDI, R-MIDI-PU-T/R are unplaced on it and its parity, renders and fab are stale; the CAD and body.yaml changes and the four other stale sims follow in the next commit.

Co-Authored-By: Claude Opus 5.5 <noreply@anthropic.com>
Claude-Session: https://claude.ai/code/session_01LmB4muFXnoLprWX4JzuJ5A
Parts:
- J1: Note The Matrix ribbon's carrier end (CBL-MCU-RIBBON): the same header as J-MCU, upside down on the carrier's underside straight above it, its mouth the same way (toward the far side). Hanging upside down it numbers the ribbon from the other edge: pin k carries J-MCU pin 25-k (the carrier socket is crimped turned over, pin 1 on conductor 24), held by tools/kicad.py check against hardware/carrier/netlist.yaml. Pins 1 and 2 (J-MCU 24 and 23, EN and IO0 until the owner chose to program the Matrix over its own USB-C only, 2026-10-03) are on no net -> The Matrix ribbon's carrier end (CBL-MCU-RIBBON): the same header as J-MCU, upside down on the carrier's underside straight above it, its mouth the same way (toward the far side). Hanging upside down it numbers the ribbon from the other edge: pin k carries J-MCU pin 25-k (the carrier socket is crimped turned over, pin 1 on conductor 24), held by tools/kicad.py check against hardware/carrier/netlist.yaml. Pin 2 (J-MCU 23) carries IO6, the MIDI out's tip line, since issue #37 (carrier/midi-out); pin 1 (J-MCU 24) is on no net - it is boxed in by the bus (carrier_routes.py). Both were EN and IO0 until the owner chose to program the Matrix over its own USB-C only, 2026-10-03
- J2: Note The Matrix's 5V..IO1 pad row: a 1x10 surface-mount header standing on the carrier's top face, its staggered feet soldered there (nothing comes through: J-MCU-C's insulator is under it) and its posts through the Matrix's pads, the Matrix sitting on its 2.5 mm plastic (config/body.yaml boards.matrix_hdr_h); the posts cut flush on the Matrix's top face. IO4, IO5 and IO6 reach nothing (spare, carrier.md) and are soldered for strength. -> The Matrix's 5V..IO1 pad row: a 1x10 surface-mount header standing on the carrier's top face, its staggered feet soldered there (nothing comes through: J-MCU-C's insulator is under it) and its posts through the Matrix's pads, the Matrix sitting on its 2.5 mm plastic (config/body.yaml boards.matrix_hdr_h); the posts cut flush on the Matrix's top face. IO6 is the MIDI out's tip line (issue #37), to J-MCU-C pin 2 (J-MCU 23); IO2, its ring line, was already routed. IO4 and IO5 reach nothing (spare, carrier.md) and are soldered for strength.
Connections:
- net IO6: now reaches J1.2 (Pin_2)
- net IO6: now also J2.5 (Pin_5)
- no-connect marks 5 -> 3
Changed lines of the file:
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@@
     (property "Pins" "1=1 2=2 3=3 4=4 5=5 6=6 7=7 8=8 9=9 10=10 11=11 12=12 13=13 14=14 15=15 16=16 17=17 18=18 19=19 20=20 21=21 22=22 23=23 24=24" (at 330.20 60.96 0) (effects (font (size 1.27 1.27)) hide))
     (property "Pins_source" "J-MCU pin 25-k on pin k: J-MCU's pin map (hardware/carrier/netlist.yaml, ADR 0018) through a straight IDC ribbon into the same header hung upside down straight above it (ADR 0021 amendment 2026-10-03)" (at 330.20 60.96 0) (effects (font (size 1.27 1.27)) hide))
-    (property "Note" "The Matrix ribbon's carrier end (CBL-MCU-RIBBON): the same header as J-MCU, upside down on the carrier's underside straight above it, its mouth the same way (toward the far side). Hanging upside down it numbers the ribbon from the other edge: pin k carries J-MCU pin 25-k (the carrier socket is crimped turned over, pin 1 on conductor 24), held by tools/kicad.py check against hardware/carrier/netlist.yaml. Pins 1 and 2 (J-MCU 24 and 23, EN and IO0 until the owner chose to program the Matrix over its own USB-C only, 2026-10-03) are on no net" (at 330.20 60.96 0) (effects (font (size 1.27 1.27)) hide))
+    (property "Note" "The Matrix ribbon's carrier end (CBL-MCU-RIBBON): the same header as J-MCU, upside down on the carrier's underside straight above it, its mouth the same way (toward the far side). Hanging upside down it numbers the ribbon from the other edge: pin k carries J-MCU pin 25-k (the carrier socket is crimped turned over, pin 1 on conductor 24), held by tools/kicad.py check against hardware/carrier/netlist.yaml. Pin 2 (J-MCU 23) carries IO6, the MIDI out's tip line, since issue #37 (carrier/midi-out); pin 1 (J-MCU 24) is on no net - it is boxed in by the bus (carrier_routes.py). Both were EN and IO0 until the owner chose to program the Matrix over its own USB-C only, 2026-10-03" (at 330.20 60.96 0) (effects (font (size 1.27 1.27)) hide))
     (property "Manufacturer" "XKB Connection" (at 330.20 60.96 0) (effects (font (size 1.27 1.27)) hide))
     (property "MPN" "X1270WR-2x12A-9TV01" (at 330.20 60.96 0) (effects (font (size 1.27 1.27)) hide))
@@
   )
   (no_connect (at 325.12 48.26))
-  (no_connect (at 337.82 48.26))
   (wire (pts (xy 325.12 50.80) (xy 322.58 50.80)) (stroke (width 0) (type default)))
   (label "U0TXD" (at 322.58 50.80 180) (fields_autoplaced) (effects (font (size 1.27 1.27)) (justify right bottom)))
@@
     (property "Pins" "P5V=1 GND=2 P3V3=3 IO7=4 IO6=5 IO5=6 IO4=7 IO3=8 IO2=9 IO1=10" (at 330.20 121.92 0) (effects (font (size 1.27 1.27)) hide))
     (property "Pins_source" "datasheets/mechanical/WAVESHARE-ESP32-S3-MATRIX-pinout.png (top view): 5V, GND, 3V3(OUT), 7, 6, 5, 4, 3, 2, 1 from the USB-C edge" (at 330.20 121.92 0) (effects (font (size 1.27 1.27)) hide))
-    (property "Note" "The Matrix's 5V..IO1 pad row: a 1x10 surface-mount header standing on the carrier's top face, its staggered feet soldered there (nothing comes through: J-MCU-C's insulator is under it) and its posts through the Matrix's pads, the Matrix sitting on its 2.5 mm plastic (config/body.yaml boards.matrix_hdr_h); the posts cut flush on the Matrix's top face. IO4, IO5 and IO6 reach nothing (spare, carrier.md) and are soldered for strength." (at 330.20 121.92 0) (effects (font (size 1.27 1.27)) hide))
+    (property "Note" "The Matrix's 5V..IO1 pad row: a 1x10 surface-mount header standing on the carrier's top face, its staggered feet soldered there (nothing comes through: J-MCU-C's insulator is under it) and its posts through the Matrix's pads, the Matrix sitting on its 2.5 mm plastic (config/body.yaml boards.matrix_hdr_h); the posts cut flush on the Matrix's top face. IO6 is the MIDI out's tip line (issue #37), to J-MCU-C pin 2 (J-MCU 23); IO2, its ring line, was already routed. IO4 and IO5 reach nothing (spare, carrier.md) and are soldered for strength." (at 330.20 121.92 0) (effects (font (size 1.27 1.27)) hide))
     (property "Manufacturer" "hanxia" (at 330.20 121.92 0) (effects (font (size 1.27 1.27)) hide))
     (property "MPN" "HX PZ2.54-1x10P TP-YQ" (at 330.20 121.92 0) (effects (font (size 1.27 1.27)) hide))
@@
   (wire (pts (xy 325.12 119.38) (xy 322.58 119.38)) (stroke (width 0) (type default)))
   (label "IO7" (at 322.58 119.38 180) (fields_autoplaced) (effects (font (size 1.27 1.27)) (justify right bottom)))
-  (no_connect (at 325.12 121.92))
   (no_connect (at 325.12 124.46))
   (no_connect (at 325.12 127.00))
@@
     (instances (project "matrix-carrier" (path "/3094b460-1210-5398-95c5-036d1afe7fc5" (reference "#FLG41") (unit 1))))
   )
+  (wire (pts (xy 337.82 48.26) (xy 340.36 48.26)) (stroke (width 0) (type default)))
+  (label "IO6" (at 340.36 48.26 0) (fields_autoplaced) (effects (font (size 1.27 1.27)) (justify left bottom)))
+  (wire (pts (xy 325.12 121.92) (xy 322.58 121.92)) (stroke (width 0) (type default)))
+  (label "IO6" (at 322.58 121.92 180) (fields_autoplaced) (effects (font (size 1.27 1.27)) (justify right bottom)))
   (sheet_instances (path "/" (page "1")))
 )
