File: hardware/carrier/led-strip-drive/led-strip-drive.kicad_sch (KiCad schematic)
At the start: 32 parts

Commit message: #8 #17 #19: the LED row even over the main board (owner), J-MCU off the row as one config figure, cone NOTE; ADR 0028 amendment, firmware, LED drive sim
- ADR 0028 amendment 2026-10-03, the owner quoted: fourteen LEDs in ONE row at one pitch with
  equal margins to the main board's ends; the corner LED is gone. The body CAD derives the
  pitch (19.869 mm, margins 17.05 mm): the even tiling's half-pitch margin is overridden at
  the mouth only, by the breath sensor's courtyard + board_clear. The tail end mount steps
  clear of LED1 by the CAD's own rule (278.313 -> 275.313). lighting.tail_led and
  led_pitch removed from config; drc.echo 'LED row on the main board', 'LED row clear of its
  neighbours'; the U-bolt rule now tests what it is for (no LED under the strap: 5.30 mm
  clear) and prints the station's 0.83 mm off the midpoint instead of shifting the row.
- J-MCU's place is ONE config figure, boards.mcu_conn_at [x, y, facing] (owner: "moved to
  the side so that it doesn't cause coverage of the led"): turned along the body at the near
  edge, mouth toward the row, the Matrix branch's value [261.27, 12.29, 90]. drc 'J-MCU, its
  plug and the Matrix ribbon off the LED row' (the row band, every height); NOTE 'tall parts
  in the LEDs' cone' (lighting.led_view_angle 120 [from memory], the diffusion test decides).
  The regulator block decoupled (boards.tall_at_x); HDR-SERVICE to the tail corner
  (boards.service_hdr_at). pcb_main places and checks a connector turned across the body.
- Main board re-placed round the row (layout.yaml), not routed: routing waits for the Matrix
  branch's J-MCU / J-MCU-KB pair.
- firmware/README.md: fourteen pixels in one row, no per-LED gain. led-strip-drive: page,
  sheet note (netlist re-exported), BOM, notes.md history; sim re-run: the edge 33 ns nominal,
  29-42 ns over the corners (was 37 / 30-50 with the corner LED's feed), bar 55 -> 45 ns.
- Corner-LED wording on ADR 0005/0014/0016/0021 (superseded on the line), DESIGN.md,
  ne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
Parts:
- D-LED-1, D-LED-10, D-LED-11, D-LED-12, D-LED-13, D-LED-14, D-LED-2, D-LED-3, D-LED-4, D-LED-5, D-LED-6, D-LED-7, D-LED-8, D-LED-9: Note On the main board's top face (ADR 0028): D-LED-1 in the tai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 -> On the main board's top face (ADR 0028): the LEDs in one ro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

Commit message: #19 #8: thirteen LEDs (tail-end LED removed, owner); C-STRIP-BULK two 6.3x7.7 polymer cans; J-MCU at 262.27
The owner, 2026-10-03: "remove that bottom led again" / "Keep current
layout, remove bottom one". ADR 0028 second amendment of 2026-10-03.

- lighting.led_count 14 -> 13; new lighting.led_slots 14 keeps LED2-14
  where they stood (pitch 19.869, x 24.55 ... 262.98), now LED1-13;
  drc.echo 'LED row on the main board' prints count and places.
- led-strip-drive sheet: D-LED-1 / C-LED-1 (D7 / C25) removed, the chain
  renumbered from the tail with every part's UUID kept; new D-LED-1's DIN2
  grounded; BOM qty 13.
- Figures by the three-step rule (the 14-LED spellings grepped first, moved
  into forbidden; the 13-LED spellings that are correct again taken out):
  led-row-current 170-195 mA, umbilical-current 359 mA, hotplug-iso-ocp
  0.49-0.54 A / 3.4x, instrument-input-z-margin 55x / 159x, led-pwm-rail-ripple
  5.6 mV / 0.00088 cents, led-pwm-pitch 0.0034 / 0.011 cents,
  diode-split-rationale back at 0.22 A.
- C10 replacement (coordinator-approved, all four criteria hold):
  C-STRIP-BULK is two MA25V220M6X8 (JIERR, LCSC C46550464), 220 uF 25 V
  polymer, 6.3 x 7.7 mm, in parallel (C10, C44): 14 mohm at 100 kHz
  (<= 0.16), ripple 2.9 A x 0.3 at 1-10 kHz per can vs a 0.367 A swing,
  440 uF; every sim that takes the bulk now takes the pair (c_strip,
  r_strip) and passes. Datasheet and EasyEDA footprint banked (fragment
  R52), JLC rotation row by pin function (0).
- Sims re-run, not scaled, 0 failed: led-strip-drive, power-entry-instrument,
  umbilical-load-switch, panel-led, digital-and-supervision, power-entry,
  interfaces/system, breath-adc, breath-output-stage.
- ADR 0005, 0014, 0016, 0021, 0027, 0028 (amendment), firmware README
  (13 pixels), led-strip-drive, power-entry-instrument, power-entry,
  umbilical-load-switch pages and sim READMEs follow.
- boards.mcu_conn_at [262.27, 12.29, 90] (the owner's option 1; the
  Matrix branch carries the same line); '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
Parts:
- removed C-LED-1: 100nF, Capacitor_SMD:C_0805_2012Metric, symbol Device:C
- removed D-LED-1: WS2815B-V1, woody:LED_WS2815B-V1_PLCC6_5.4x5.0mm_P1.6mm, symbol woody:WS2815B-V1
- renumbered C-LED-2 to C-LED-1, C-LED-11 to C-LED-10, C-LED-12 to C-LED-11, C-LED-13 to C-LED-12, C-LED-14 to C-LED-13, C-LED-3 to C-LED-2, C-LED-4 to C-LED-3, C-LED-5 to C-LED-4, C-LED-6 to C-LED-5, C-LED-7 to C-LED-6, C-LED-8 to C-LED-7, C-LED-9 to C-LED-8, C-LED-10 to C-LED-9, D-LED-2 to D-LED-1, D-LED-11 to D-LED-10, D-LED-12 to D-LED-11, D-LED-13 to D-LED-12, D-LED-14 to D-LED-13, D-LED-3 to D-LED-2, D-LED-4 to D-LED-3, D-LED-5 to D-LED-4, D-LED-6 to D-LED-5, D-LED-7 to D-LED-6, D-LED-8 to D-LED-7, D-LED-9 to D-LED-8, D-LED-10 to D-LED-9
Connections:
- net LED_D13 is gone; now on net LED_D12: D-LED-12.3 (DO), D-LED-13.4 (DIN1)
- net LED_D1: now also D-LED-1.3 (DO), D-LED-2.4 (DIN1), D-LED-3.6 (DIN2); no longer D-LED-1.4 (DIN1), D-LED-2.6 (DIN2)
- net LED_D10: now also D-LED-10.3 (DO), D-LED-11.4 (DIN1), D-LED-12.6 (DIN2); no longer D-LED-10.4 (DIN1), D-LED-11.6 (DIN2), D-LED-9.3 (DO)
- net LED_D11: now also D-LED-11.3 (DO), D-LED-12.4 (DIN1), D-LED-13.6 (DIN2); no longer D-LED-10.3 (DO), D-LED-11.4 (DIN1), D-LED-12.6 (DIN2)
- net LED_D12: no longer D-LED-11.3 (DO), D-LED-12.4 (DIN1), D-LED-13.6 (DIN2)
- net LED_D2: now also D-LED-2.3 (DO), D-LED-3.4 (DIN1), D-LED-4.6 (DIN2); no longer D-LED-1.3 (DO), D-LED-2.4 (DIN1), D-LED-3.6 (DIN2)
- net LED_D3: now also D-LED-3.3 (DO), D-LED-4.4 (DIN1), D-LED-5.6 (DIN2); no longer D-LED-2.3 (DO), D-LED-3.4 (DIN1), D-LED-4.6 (DIN2)
- net LED_D4: now also D-LED-4.3 (DO), D-LED-5.4 (DIN1), D-LED-6.6 (DIN2); no longer D-LED-3.3 (DO), D-LED-4.4 (DIN1), D-LED-5.6 (DIN2)
- net LED_D5: now also D-LED-5.3 (DO), D-LED-6.4 (DIN1), D-LED-7.6 (DIN2); no longer D-LED-4.3 (DO), D-LED-5.4 (DIN1), D-LED-6.6 (DIN2)
- net LED_D6: now also D-LED-6.3 (DO), D-LED-7.4 (DIN1), D-LED-8.6 (DIN2); no longer D-LED-5.3 (DO), D-LED-6.4 (DIN1), D-LED-7.6 (DIN2)
- net LED_D7: now also D-LED-7.3 (DO), D-LED-8.4 (DIN1), D-LED-9.6 (DIN2); no longer D-LED-6.3 (DO), D-LED-7.4 (DIN1), D-LED-8.6 (DIN2)
- net LED_D8: now also D-LED-10.6 (DIN2), D-LED-8.3 (DO), D-LED-9.4 (DIN1); no longer D-LED-7.3 (DO), D-LED-8.4 (DIN1), D-LED-9.6 (DIN2)
- net LED_D9: now also D-LED-10.4 (DIN1), D-LED-11.6 (DIN2), D-LED-9.3 (DO); no longer D-LED-10.6 (DIN2), D-LED-8.3 (DO), D-LED-9.4 (DIN1)
- net LED_DI: now also D-LED-1.4 (DIN1), D-LED-2.6 (DIN2); no longer D-LED-1.6 (DIN2)
- net PWR_GND: now also D-LED-1.6 (DIN2)
- no-connect marks 18 -> 17
Other:
- note added: "R-LED-PD holds the input low through the bootloader window: GPIO1 floats, OE is tied low, and a floating AHCT input would put clean 5 V edges into the LED row before firmware runs. Gates B-D are spare: inputs and enables tied low (an enabled CMOS gate never floats). THE LEDS (ADR 0028): WS2815B-V1 on the main board (count: config/body.yaml lighting.led_count), 12 V, one data line. D-LED-1 is at t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"
- note removed: "R-LED-PD holds the input low through the bootloader window: GPIO1 floats, OE is tied low, and a floating AHCT input would put clean 5 V edges into the LED row before firmware runs. Gates B-D are spare: inputs and enables tied low (an enabled CMOS gate never floats). THE LEDS (ADR 0028): WS2815B-V1 on the main board (count: config/body.yaml lighting.led_count), 12 V, one data line. D-LED-1 is in t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"

Commit message: #37: MIDI out circuit, the ribbon's MIDI pair, carrier re-route, ADR 0015 amendment
- hardware/carrier/midi-out/: new circuit (sheet, netlist, BOM, page): CA-033's 5 V row
  from U-LVLSHIFT gates B/C, R-MIDI 220R, FB-MIDI, U-TVS-MIDI, J-MIDI (JST PH SMD),
  J-MIDI-OUT (SJ5-43502PM, panel-mount, no footprint), CBL-MIDI. TRS Type A/B in firmware.
- led-strip-drive: gates B/C drive tip/ring; R-MIDI-PU-T/R 10k to DEV_3V3 (power-on default).
- carrier: IO6 on J-MCU 23 (tip) and IO2 on J-MCU 5 (ring) become ports. J-MCU 24 stays
  unconnected: on the Matrix carrier J-MCU-C pin 1 is boxed in by the hand-routed bus.
- matrix-carrier: IO6 routed J-MCU-C pin 2 -> J2.5 (carrier_routes.py); pcb.py check 0 errors.
- main-board root sheet places midi-out; nets.yaml; BOM fragments; CBL-USB-EXT leaves unplaced.csv.
- tools/merge-bom.py: the new fragment added to ORDER (the tool refuses to write when a
  fragment is not listed); no check changed.
- ADR 0015 amendment, ADR 0012 note, firmware/README.md (config mode/OTA deferred; MIDI out),
  draft design in docs/research/.

Gate-Red: pre-existing at 18d0b5f - 37 stale CAD outputs and kicad 131 problems (main-board/module-main PCB parity and clearance). Also red from this checkpoint: the main board's .kicad_pcb is #35's and is not touched, so J-MIDI, R-MIDI-T/R, FB-MIDI-T/R, U-TVS-MIDI, R-MIDI-PU-T/R are unplaced on it and its parity, renders and fab are stale; the CAD and body.yaml changes and the four other stale sims follow in the next commit.

Co-Authored-By: Claude Opus 5.5 <noreply@anthropic.com>
Claude-Session: https://claude.ai/code/session_01LmB4muFXnoLprWX4JzuJ5A
Parts:
- added R-MIDI-PU-R, R-MIDI-PU-T: 10k 1%, Resistor_SMD:R_0805_2012Metric, symbol Device:R
- U-LVLSHIFT: Note ON THE 5 V RAIL, and that is the point: TTL thresholds mean a 3.3 V input reads high, and the output (~4.4 V minimum) clears the WS2815B-V1 V_IH (2.7 V min) and stays under its 5.7 V logic-input maximum. Gates B, C and D are spare: the row has one data line, and LED 1 grounds its DIN2 rather than having it driven -> ON THE 5 V RAIL, and that is the point: TTL thresholds mean a 3.3 V input reads high, and the output (~4.4 V minimum) clears the WS2815B-V1 V_IH (2.7 V min) and stays under its 5.7 V logic-input maximum. Gate A drives the row (one data line; LED 1 grounds its DIN2). Gates B and C are the MIDI out's tip and ring drivers since issue #37 (carrier/midi-out): IO6 into B, IO2 into C, each output through 220R to the jack - push-pull at 5 V, so either line can be the current source or the sink and TRS Type A/B is a firmware choice. Gate D is spare, input and enable tied low
Connections:
- net PWR_GND: no longer U-LVLSHIFT.5, U-LVLSHIFT.9
- net MIDI_TIP_DRV: now reaches U-LVLSHIFT.6
- net MIDI_RING_DRV: now reaches U-LVLSHIFT.8
- new net DEV_3V3: R-MIDI-PU-R.1, R-MIDI-PU-T.1
- new net IO2: R-MIDI-PU-R.2, U-LVLSHIFT.9
- new net IO6: R-MIDI-PU-T.2, U-LVLSHIFT.5
- no-connect marks 17 -> 15
Other:
- note added: "R-LED-PD holds the input low through the bootloader window: GPIO1 floats, OE is tied low, and a floating AHCT input would put clean 5 V edges into the LED row before firmware runs. Gates B and C drive the MIDI out's tip and ring (issue #37, carrier/midi-out), their inputs IO6 and IO2 pulled up to DEV_3V3 by R-MIDI-PU-T and R-MIDI-PU-R: high through boot, so tip and ring sit at one voltage and no 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"
- note removed: "R-LED-PD holds the input low through the bootloader window: GPIO1 floats, OE is tied low, and a floating AHCT input would put clean 5 V edges into the LED row before firmware runs. Gates B-D are spare: inputs and enables tied low (an enabled CMOS gate never floats). THE LEDS (ADR 0028): WS2815B-V1 on the main board (count: config/body.yaml lighting.led_count), 12 V, one data line. D-LED-1 is at t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"
