File: hardware/carrier/power-entry-instrument/power-entry-instrument.kicad_sch (KiCad schematic)
At the start: 17 parts

Commit message: #8: plane stitching - three C-STITCH-12V (INST_POS12 to PWR_GND) at J-MCU, J-UMB and the analog end (#8-8)
Owner, 2026-10-04 (working chat): "add 2-3 now". Three 100 nF 50 V X7R 0805
(C-LED's part, YAGEO CC0805KRX7R9BB104 / C49678), new BOM row C-STITCH-12V in
the power-entry-instrument fragment, on that sheet as C-STITCH-12V-1..3 and
on the board as C45 (beside J-MCU's LED-row side, 8.7 mm from the target at
its top edge - the nearest clear place), C46 (inboard of J-UMB) and C47 (at
the analog end, its PWR_GND pad on the plane beside the AGND_INST island).
Each pad meets its plane through its own via at the pad (pcb.py finish's
fanout, 1.0-1.2 mm stubs). kicad.py export, merge-bom, check-netlist
--strict (0 problems), pcb.py check 0 errors, renders and fab/ written; the
power-entry-instrument page (Plane stitching) and the board README (Open
row removed, references, Revisions H) say so. Sims re-run against the new
netlist: carrier power-entry-instrument, interfaces/system,
umbilical-load-switch - 0 failed.

Gate-Red: hardware/module/power-entry/sim results stale against this netlist (its re-run is in progress on a loaded machine; lands in the next commit on this branch); 8 CAD photo renders stale against the board (about 25 min each, to be rebuilt once the board settles); module-main's pre-existing kicad.py failures and its missing silk title (check_title); module-iso's sim coverage row (another branch).

Co-Authored-By: Claude Opus 5.5 <noreply@anthropic.com>
Claude-Session: https://claude.ai/code/session_01LmB4muFXnoLprWX4JzuJ5A
Parts:
- added C-STITCH-12V-1, C-STITCH-12V-2, C-STITCH-12V-3: 100nF 50V X7R, Capacitor_SMD:C_0805_2012Metric, symbol Device:C
Connections:
- net INST_POS12: now also C-STITCH-12V-1.1, C-STITCH-12V-2.1, C-STITCH-12V-3.1
- net PWR_GND: now also C-STITCH-12V-1.2, C-STITCH-12V-2.2, C-STITCH-12V-3.2
Other:
- note added: "PLANE STITCHING (#8-8; owner, 2026-10-04: "add 2-3 now"): three 100 nF from INST_POS12 (layer 3) to PWR_GND (layer 2), one each at J-MCU, J-UMB and the analog end, where signals change layers between the two planes' references more than 20 mm from the nearest C-LED. Each pad meets its plane by its own via at the pad (power-entry-instrument.md, Plane stitching)."
Changed lines of the file:
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@@
     (property "From" "module/power-entry" (at 101.6 186.69 0) (effects (font (size 1.27 1.27)) hide))
     (property "Figure" "umbilical-pinmap" (at 101.6 186.69 0) (effects (font (size 1.27 1.27)) hide)))
+  (symbol (lib_id "Device:C") (at 63.5 224.79 0) (unit 1)
+    (in_bom yes) (on_board yes) (dnp no)
+    (property "Reference" "C-STITCH-12V-1" (at 67.31 223.51999999999998 0) (effects (font (size 1.27 1.27)) (justify left)))
+    (property "Value" "100nF 50V X7R" (at 67.31 226.06 0) (effects (font (size 1.27 1.27)) (justify left)))
+    (property "Footprint" "Capacitor_SMD:C_0805_2012Metric" (at 63.5 224.79 0) (effects (font (size 1.27 1.27)) hide))
+    (property "Datasheet" "" (at 63.5 224.79 0) (effects (font (size 1.27 1.27)) hide))
+    (property "Row" "C-STITCH-12V" (at 63.5 224.79 0) (effects (font (size 1.27 1.27)) hide))
+    (property "Pins" "1=1 2=2" (at 63.5 224.79 0) (effects (font (size 1.27 1.27)) hide))
+    (property "Note" "Stitching INST_POS12 to PWR_GND at J-MCU, where the SPI and IO lines change layers between the two planes' references: their return current crosses here, not 20 mm away at a C-LED (#8-8)" (at 63.5 224.79 0) (effects (font (size 1.27 1.27)) hide))
+    (property "Pins_source" "a ceramic capacitor: either way round" (at 63.5 224.79 0) (effects (font (size 1.27 1.27)) hide))
+    (property "Manufacturer" "YAGEO" (at 63.5 224.79 0) (effects (font (size 1.27 1.27)) hide))
+    (property "MPN" "CC0805KRX7R9BB104" (at 63.5 224.79 0) (effects (font (size 1.27 1.27)) hide))
+    (property "LCSC" "C49678" (at 63.5 224.79 0) (effects (font (size 1.27 1.27)) hide))
+    (property "Assembly" "machine" (at 63.5 224.79 0) (effects (font (size 1.27 1.27)) hide))
+    (pin "1")
+    (pin "2")
+    (instances (project "main-board" (path "/b12a49ac-ffa0-5078-b2ba-e15d161f1936/4727eca5-0a6b-5761-98ac-51ca9f544ea2" (reference "C45") (unit 1))) (project "power-entry-instrument" (path "/ba12e546-d582-5654-bb26-6a94a8f78514" (reference "C-STITCH-12V-1") (unit 1))))
+  )
+  (wire (pts (xy 63.5 220.98) (xy 63.5 218.44)) (stroke (width 0) (type default)))
+  (hierarchical_label "INST_POS12" (shape output) (at 63.5 218.44 90) (effects (font (size 1.27 1.27)) (justify left))
+    (property "Dir" "out" (at 63.5 218.44 0) (effects (font (size 1.27 1.27)) hide))
+    (property "To" "carrier/led-strip-drive" (at 63.5 218.44 0) (effects (font (size 1.27 1.27)) hide))
+    (property "Figure" "umbilical-current" (at 63.5 218.44 0) (effects (font (size 1.27 1.27)) hide)))
+  (wire (pts (xy 63.5 228.6) (xy 63.5 231.14)) (stroke (width 0) (type default)))
+  (hierarchical_label "PWR_GND" (shape passive) (at 63.5 231.14 270) (effects (font (size 1.27 1.27)) (justify right))
+    (property "Dir" "ref" (at 63.5 231.14 0) (effects (font (size 1.27 1.27)) hide))
+    (property "From" "module/power-entry" (at 63.5 231.14 0) (effects (font (size 1.27 1.27)) hide))
+    (property "Figure" "umbilical-pinmap" (at 63.5 231.14 0) (effects (font (size 1.27 1.27)) hide)))
+  (symbol (lib_id "Device:C") (at 88.9 224.79 0) (unit 1)
+    (in_bom yes) (on_board yes) (dnp no)
+    (property "Reference" "C-STITCH-12V-2" (at 92.71000000000001 223.51999999999998 0) (effects (font (size 1.27 1.27)) (justify left)))
+    (property "Value" "100nF 50V X7R" (at 92.71000000000001 226.06 0) (effects (font (size 1.27 1.27)) (justify left)))
+    (property "Footprint" "Capacitor_SMD:C_0805_2012Metric" (at 88.9 224.79 0) (effects (font (size 1.27 1.27)) hide))
+    (property "Datasheet" "" (at 88.9 224.79 0) (effects (font (size 1.27 1.27)) hide))
+    (property "Row" "C-STITCH-12V" (at 88.9 224.79 0) (effects (font (size 1.27 1.27)) hide))
+    (property "Pins" "1=1 2=2" (at 88.9 224.79 0) (effects (font (size 1.27 1.27)) hide))
+    (property "Note" "Stitching INST_POS12 to PWR_GND at J-UMB, where the umbilical's lines change layers between the two planes' references (#8-8)" (at 88.9 224.79 0) (effects (font (size 1.27 1.27)) hide))
+    (property "Pins_source" "a ceramic capacitor: either way round" (at 88.9 224.79 0) (effects (font (size 1.27 1.27)) hide))
+    (property "Manufacturer" "YAGEO" (at 88.9 224.79 0) (effects (font (size 1.27 1.27)) hide))
+    (property "MPN" "CC0805KRX7R9BB104" (at 88.9 224.79 0) (effects (font (size 1.27 1.27)) hide))
+    (property "LCSC" "C49678" (at 88.9 224.79 0) (effects (font (size 1.27 1.27)) hide))
+    (property "Assembly" "machine" (at 88.9 224.79 0) (effects (font (size 1.27 1.27)) hide))
+    (pin "1")
+    (pin "2")
+    (instances (project "main-board" (path "/b12a49ac-ffa0-5078-b2ba-e15d161f1936/4727eca5-0a6b-5761-98ac-51ca9f544ea2" (reference "C46") (unit 1))) (project "power-entry-instrument" (path "/ba12e546-d582-5654-bb26-6a94a8f78514" (reference "C-STITCH-12V-2") (unit 1))))
+  )
+  (wire (pts (xy 88.9 220.98) (xy 88.9 218.44)) (stroke (width 0) (type default)))
+  (hierarchical_label "INST_POS12" (shape output) (at 88.9 218.44 90) (effects (font (size 1.27 1.27)) (justify left))
+    (property "Dir" "out" (at 88.9 218.44 0) (effects (font (size 1.27 1.27)) hide))
+    (property "To" "carrier/led-strip-drive" (at 88.9 218.44 0) (effects (font (size 1.27 1.27)) hide))
+    (property "Figure" "umbilical-current" (at 88.9 218.44 0) (effects (font (size 1.27 1.27)) hide)))
+  (wire (pts (xy 88.9 228.6) (xy 88.9 231.14)) (stroke (width 0) (type default)))
+  (hierarchical_label "PWR_GND" (shape passive) (at 88.9 231.14 270) (effects (font (size 1.27 1.27)) (justify right))
+    (property "Dir" "ref" (at 88.9 231.14 0) (effects (font (size 1.27 1.27)) hide))
+    (property "From" "module/power-entry" (at 88.9 231.14 0) (effects (font (size 1.27 1.27)) hide))
+    (property "Figure" "umbilical-pinmap" (at 88.9 231.14 0) (effects (font (size 1.27 1.27)) hide)))
+  (symbol (lib_id "Device:C") (at 114.3 224.79 0) (unit 1)
+    (in_bom yes) (on_board yes) (dnp no)
+    (property "Reference" "C-STITCH-12V-3" (at 118.11 223.51999999999998 0) (effects (font (size 1.27 1.27)) (justify left)))
+    (property "Value" "100nF 50V X7R" (at 118.11 226.06 0) (effects (font (size 1.27 1.27)) (justify left)))
+    (property "Footprint" "Capacitor_SMD:C_0805_2012Metric" (at 114.3 224.79 0) (effects (font (size 1.27 1.27)) hide))
+    (property "Datasheet" "" (at 114.3 224.79 0) (effects (font (size 1.27 1.27)) hide))
+    (property "Row" "C-STITCH-12V" (at 114.3 224.79 0) (effects (font (size 1.27 1.27)) hide))
+    (property "Pins" "1=1 2=2" (at 114.3 224.79 0) (effects (font (size 1.27 1.27)) hide))
+    (property "Note" "Stitching INST_POS12 to PWR_GND at the analog end, where the ADC's digital lines and the chain change layers between the two planes' references (#8-8)" (at 114.3 224.79 0) (effects (font (size 1.27 1.27)) hide))
+    (property "Pins_source" "a ceramic capacitor: either way round" (at 114.3 224.79 0) (effects (font (size 1.27 1.27)) hide))
+    (property "Manufacturer" "YAGEO" (at 114.3 224.79 0) (effects (font (size 1.27 1.27)) hide))
+    (property "MPN" "CC0805KRX7R9BB104" (at 114.3 224.79 0) (effects (font (size 1.27 1.27)) hide))
+    (property "LCSC" "C49678" (at 114.3 224.79 0) (effects (font (size 1.27 1.27)) hide))
+    (property "Assembly" "machine" (at 114.3 224.79 0) (effects (font (size 1.27 1.27)) hide))
+    (pin "1")
+    (pin "2")
+    (instances (project "main-board" (path "/b12a49ac-ffa0-5078-b2ba-e15d161f1936/4727eca5-0a6b-5761-98ac-51ca9f544ea2" (reference "C47") (unit 1))) (project "power-entry-instrument" (path "/ba12e546-d582-5654-bb26-6a94a8f78514" (reference "C-STITCH-12V-3") (unit 1))))
+  )
+  (wire (pts (xy 114.3 220.98) (xy 114.3 218.44)) (stroke (width 0) (type default)))
+  (hierarchical_label "INST_POS12" (shape output) (at 114.3 218.44 90) (effects (font (size 1.27 1.27)) (justify left))
+    (property "Dir" "out" (at 114.3 218.44 0) (effects (font (size 1.27 1.27)) hide))
+    (property "To" "carrier/led-strip-drive" (at 114.3 218.44 0) (effects (font (size 1.27 1.27)) hide))
+    (property "Figure" "umbilical-current" (at 114.3 218.44 0) (effects (font (size 1.27 1.27)) hide)))
+  (wire (pts (xy 114.3 228.6) (xy 114.3 231.14)) (stroke (width 0) (type default)))
+  (hierarchical_label "PWR_GND" (shape passive) (at 114.3 231.14 270) (effects (font (size 1.27 1.27)) (justify right))
+    (property "Dir" "ref" (at 114.3 231.14 0) (effects (font (size 1.27 1.27)) hide))
+    (property "From" "module/power-entry" (at 114.3 231.14 0) (effects (font (size 1.27 1.27)) hide))
+    (property "Figure" "umbilical-pinmap" (at 114.3 231.14 0) (effects (font (size 1.27 1.27)) hide)))
+  (text "PLANE STITCHING (#8-8; owner, 2026-10-04: \"add 2-3 now\"): three 100 nF from INST_POS12 (layer 3) to PWR_GND\n(layer 2), one each at J-MCU, J-UMB and the analog end, where signals change layers between the two planes'\nreferences more than 20 mm from the nearest C-LED. Each pad meets its plane by its own via at the pad\n(power-entry-instrument.md, Plane stitching)." (at 40.64 205.74 0) (effects (font (size 1.27 1.27)) (justify left top)))
   (sheet_instances (path "/" (page "1")))
 )

Commit message: #39: ideal-diode 5 V OR (U-USBOR LM74700-Q1 + Q-USBOR DMN3404L) replaces D-USBOR; R-MIDI 182R 1%
Checkpoint. D-USBOR's SS14 is replaced on power-entry-instrument by an
LM74700-Q1 ideal-diode controller and a DMN3404L N-FET (C-USBOR x2 for its
VCAP and CATHODE), datasheets banked (.manifest-R56). INST_5V_A with the
rack up is 4.625-5.325 V (sim or-rack); no back-feed either way (or-both),
switch-over and rack-loss simulated. R-MIDI-T/R are 182R 1% (UNI-ROYAL
1206W4F1820T5E, C247358), sized to the gate's 25 mA at the rail's ceiling.
MIDI worst corner 3.69 mA: still under CA-033's 3.75 mA, kept recorded.

Gate-Red: main-board parity (main-board.kicad_pcb deliberately not touched: D4 gone, U13/Q2/C207/C208 unplaced, fab/ stale - another agent places them); midi-out and main-board renders not yet regenerated for R-MIDI's value (next commit); interfaces/system sim stale (pre-existing, re-run in progress); 38 stale CAD renders and module-iso coverage (pre-existing; no bulk CAD renders allowed)

Co-Authored-By: Claude Opus 5.5 <noreply@anthropic.com>
Claude-Session: https://claude.ai/code/session_01LmB4muFXnoLprWX4JzuJ5A
Parts:
- removed D-USBOR-A: SS14, Diode_SMD:D_SMA, symbol Device:D_Schottky
- added C-USBOR-CAP, C-USBOR-OUT: 100nF 50V X7R, Capacitor_SMD:C_0805_2012Metric, symbol Device:C
- added Q-USBOR: DMN3404L, Package_TO_SOT_SMD:SOT-23, symbol Transistor_FET:DMN3404L
- added U-USBOR: LM74700-Q1, Package_TO_SOT_SMD:SOT-23-6, symbol Power_Management:LM74700
- C-BUCK-OUT: Note D1 (owner, 2026-10-03: '10 ohm + 22 uF + 10 uF'): RECOM's standard-application output capacitor, a 10 uF MLCC at U-BUCK-A's OUT pin (R-78E5.0-1.0 datasheet p.I-4), returned to its GND pin. It lowers the converter's ripple at its source, ahead of D-USBOR-A. Well inside the part's 220 uF capacitive-load limit -> D1 (owner, 2026-10-03: '10 ohm + 22 uF + 10 uF'): RECOM's standard-application output capacitor, a 10 uF MLCC at U-BUCK-A's OUT pin (R-78E5.0-1.0 datasheet p.I-4), returned to its GND pin. It lowers the converter's ripple at its source, ahead of U-USBOR and Q-USBOR. Well inside the part's 220 uF capacitive-load limit
Connections:
- net BUCK_A_OUT: now also C-USBOR-CAP.2, Q-USBOR.2 (S), U-USBOR.3 (EN), U-USBOR.6 (ANODE)
- net INST_5V_A: now also C-USBOR-OUT.1, Q-USBOR.3 (D), U-USBOR.4 (CATHODE)
- net PWR_GND: now also C-USBOR-OUT.2, U-USBOR.2 (GND)
- new net USBOR_GATE: Q-USBOR.1 (G), U-USBOR.5 (GATE)
- new net USBOR_VCAP: C-USBOR-CAP.1, U-USBOR.1 (VCAP)
Other:
- note added: "IDEAL-DIODE OR (issue #39; owner, 2026-10-05: "Let's go both"): U-USBOR (LM74700-Q1) and Q-USBOR replace D-USBOR-A (SS14). BUCK_A_OUT reaches INST_5V_A through the FET, 20 mV regulated; the Matrix's USB-C 5 V (through its own D1) cannot back-feed the buck, nor the buck the USB host (power-entry-instrument.md)."
