File: hardware/carrier/service-uart/service-uart.kicad_sch (KiCad schematic)
At the start: 1 part

Commit message: Main board: apply the chosen parts to every symbol and row
Every main-board and adapter symbol now carries Footprint, Manufacturer,
MPN, LCSC and Assembly. The values come from the selections whose
datasheets are banked. The BOM rows follow those choices:

- D-USBOR is the SS14 (SMA).
- J-LED is four solder pads, not a connector.
- L-BUCK-IN is 22 uH, C-BUCK-IN is a UCM electrolytic, C-STRIP-BULK is
  470 uF 25 V.
- D-TVS-BREATH is the PESD12VS1UA (SOD-323); the UB is SOD523.
- J-UMB is the hanxia header. Its posts go through the adapter and its
  tails through the tongue; the old wording had them swapped.
- U-BUCK and U-BREATH say where to buy.
- C-ADC-BULK is 1206 if fitted.

The body and geometry follow the chosen parts:

- The J-UMB and J-MCU envelopes in config/body.yaml are now read off the
  parts' drawings.
- J-MCU is longer, so the regulator block moved and the right-hand ribbon
  header followed it by 1.5 mm. The RH key board is re-laid out, with C8
  moving with the header's 3V3 pin. It checks clean.
- A mount candidate is now nudged by up to 3 mm before it is dropped. All
  seven main-board mounts hold.

New footprints and pages:

- New woody.pretty footprints: the MPXV4006DP (case 1351-01) from
  breath-sense-link.md's land pattern, and the NE8FAV from Neutrik's
  layout, mirrored to the top view.
- The input-LC derivation uses the chosen capacitor's banked ESR: Q is at
  most 1.8, and the margin is 120x worst case.
- The main-board README lists what is still open before layout.

Co-Authored-By: Claude Opus 5.5 <noreply@anthropic.com>
Claude-Session: https://claude.ai/code/session_01LmB4muFXnoLprWX4JzuJ5A
Parts:
- HDR-SERVICE: footprint (none) -> Connector_PinHeader_2.54mm:PinHeader_1x05_P2.54mm_Vertical; Assembly (none) -> hand; LCSC (none) -> C32713271; MPN (none) -> HX PZ2.54-1x5P ZZ; Manufacturer (none) -> hanxia
Changed lines of the file:
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@@
     (property "Reference" "HDR-SERVICE" (at 40.64 43.18 0) (effects (font (size 1.27 1.27))))
     (property "Value" "1x5" (at 40.64 58.42 0) (effects (font (size 1.27 1.27))))
-    (property "Footprint" "" (at 40.64 50.8 0) (effects (font (size 1.27 1.27)) hide))
+    (property "Footprint" "Connector_PinHeader_2.54mm:PinHeader_1x05_P2.54mm_Vertical" (at 40.64 50.8 0) (effects (font (size 1.27 1.27)) hide))
     (property "Datasheet" "" (at 40.64 50.8 0) (effects (font (size 1.27 1.27)) hide))
     (property "Row" "HDR-SERVICE" (at 40.64 50.8 0) (effects (font (size 1.27 1.27)) hide))
@@
     (property "Note" "FIVE PINS (ADR 0018): 1 TXD, 2 RXD, 3 GND, 4 EN, 5 IO0 - the ground between the UART pair and the control pair. EN and IO0 are pulled up on the Matrix; drive them to ground only" (at 40.64 50.8 0) (effects (font (size 1.27 1.27)) hide))
     (property "Pins_source" "pin n is header position n (service-uart.md)" (at 40.64 50.8 0) (effects (font (size 1.27 1.27)) hide))
+    (property "Manufacturer" "hanxia" (at 40.64 50.8 0) (effects (font (size 1.27 1.27)) hide))
+    (property "MPN" "HX PZ2.54-1x5P ZZ" (at 40.64 50.8 0) (effects (font (size 1.27 1.27)) hide))
+    (property "LCSC" "C32713271" (at 40.64 50.8 0) (effects (font (size 1.27 1.27)) hide))
+    (property "Assembly" "hand" (at 40.64 50.8 0) (effects (font (size 1.27 1.27)) hide))
     (pin "1")
     (pin "2")

Commit message: #11 F7, #14 A2, #14 A3: C-EN on EN, R-TXD-SER in U0TXD; Espressif's guidelines banked
#14 A2 (verified): Espressif's ESP32-S3 Hardware Design Guidelines p.11 ask
for an RC on CHIP_PU, "usually R = 10 kOhm and C = 1 uF", and a short trace;
the Matrix fits R8 (10k) and no C, and EN runs down the ribbon and across
the main board to HDR-SERVICE. C-EN, 1 uF X7R (CL21B105KBFNNNE, C28323,
the C-SENSOR-VS-BULK part), EN to PWR_GND at J-MCU pin 24, main-board C41:
tau 10 ms against t_STBL 50 us (ESP32-S3 datasheet Table 2-13 p.30).
#11 F7's "EN keeps the dev board's RC" was wrong: there is no RC.

#14 A3 (verified): the same document p.16 asks for 499 ohm in series with
U0TXD. R-TXD-SER, 499R 1% 0805 (0805W8F4990T5E, C17722, JLC extended),
main-board R46, at J-MCU pin 22; HDR-SERVICE pin 1 is now net TXD_HDR.

Both on the service-uart sheet (new BOM rows in its fragment); page,
nets.yaml notes, the sheet's text and the tooling.md coverage row follow.
The guidelines PDF is banked (logic/ESP-HARDWARE-DESIGN-GUIDELINES-ESP32S3.pdf,
fragment .manifest-R50-wave2-controller.csv). #11 F7's IO0 series R / TVS
on the header is left to the owner (no manufacturer asks for it).

Gate-Red: tree known-red - main-board .kicad_pcb awaits re-layout (R45, R46, C41 not on it yet), photos/clash stale, breath-adc vdd-ripple fails pending the owner's filter decision

Co-Authored-By: Claude Opus 5.5 <noreply@anthropic.com>
Claude-Session: https://claude.ai/code/session_01LmB4muFXnoLprWX4JzuJ5A
Parts:
- added C-EN: 1uF, Capacitor_SMD:C_0805_2012Metric, symbol Device:C
- added R-TXD-SER: 499R 1%, Resistor_SMD:R_0805_2012Metric, symbol Device:R
Connections:
- net EN: now also C-EN.1
- net PWR_GND: now also C-EN.2
- net U0TXD: now also R-TXD-SER.1; no longer HDR-SERVICE.1 (Pin_1)
- new net TXD_HDR: HDR-SERVICE.1 (Pin_1), R-TXD-SER.2
Other:
- note added: "FROM THE HAND-WRITTEN NETLIST THIS SHEET REPLACES (verbatim; the part notes are on each part's Note field): AUTHORITATIVE for connectivity. This circuit is one header, the conductors to it, R-TXD-SER in TXD and C-EN on EN (Espressif's guidelines, #14 A2/A3), and the drawing in the page is a REPRESENTATION of this file. Whatever is plugged into the service header is not part of the instrument, so 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"
- note removed: "FROM THE HAND-WRITTEN NETLIST THIS SHEET REPLACES (verbatim; the part notes are on each part's Note field): AUTHORITATIVE for connectivity. This circuit is one header and the conductors to it, and the drawing in the page is a REPRESENTATION of this file. Whatever is plugged into the service header is not part of the instrument, so hardware/nets.yaml marks that end with `external_driver:` rather t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"
Changed lines of the file:
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@@
   )
   (wire (pts (xy 35.56 45.72) (xy 33.02 45.72)) (stroke (width 0) (type default)))
-  (hierarchical_label "U0TXD" (shape input) (at 33.02 45.72 180) (effects (font (size 1.27 1.27)) (justify right))
-    (property "Dir" "in" (at 33.02 45.72 0) (effects (font (size 1.27 1.27)) hide))
-    (property "From" "carrier/carrier" (at 33.02 45.72 0) (effects (font (size 1.27 1.27)) hide)))
+  (label "TXD_HDR" (at 33.02 45.72 180) (fields_autoplaced) (effects (font (size 1.27 1.27)) (justify right bottom)))
   (wire (pts (xy 35.56 48.26) (xy 33.02 48.26)) (stroke (width 0) (type default)))
   (hierarchical_label "U0RXD" (shape input) (at 33.02 48.26 180) (effects (font (size 1.27 1.27)) (justify right))
@@
     (property "Dir" "in" (at 33.02 55.88 0) (effects (font (size 1.27 1.27)) hide))
     (property "From" "carrier/carrier" (at 33.02 55.88 0) (effects (font (size 1.27 1.27)) hide)))
-  (text "FROM THE HAND-WRITTEN NETLIST THIS SHEET REPLACES (verbatim; the part notes are on each part's Note field):\n\nAUTHORITATIVE for connectivity. This circuit is one header and the conductors to it, and the drawing in the\npage is a REPRESENTATION of this file. Whatever is plugged into the service header is not part of the\ninstrument, so hardware/nets.yaml marks that end with `external_driver:` rather than inventing a driver or\ncalling the net undriven." (at 205.74 38.099999999999994 0) (effects (font (size 1.27 1.27)) (justify left top)))
+  (text "FROM THE HAND-WRITTEN NETLIST THIS SHEET REPLACES (verbatim; the part notes are on each part's Note field):\n\nAUTHORITATIVE for connectivity. This circuit is one header, the conductors to it, R-TXD-SER in TXD and C-EN on\nEN (Espressif's guidelines, #14 A2/A3), and the drawing in the page is a REPRESENTATION of this file. Whatever is plugged into the service header is not part of the\ninstrument, so hardware/nets.yaml marks that end with `external_driver:` rather than inventing a driver or\ncalling the net undriven." (at 205.74 38.099999999999994 0) (effects (font (size 1.27 1.27)) (justify left top)))
+  (symbol (lib_id "Device:R") (at 101.60 50.80 0) (unit 1)
+    (in_bom yes) (on_board yes) (dnp no)
+    (property "Reference" "R-TXD-SER" (at 104.14 49.53 0) (effects (font (size 1.27 1.27)) (justify left)))
+    (property "Value" "499R 1%" (at 104.14 52.07 0) (effects (font (size 1.27 1.27)) (justify left)))
+    (property "Footprint" "Resistor_SMD:R_0805_2012Metric" (at 101.60 50.80 0) (effects (font (size 1.27 1.27)) hide))
+    (property "Datasheet" "" (at 101.60 50.80 0) (effects (font (size 1.27 1.27)) hide))
+    (property "Row" "R-TXD-SER" (at 101.60 50.80 0) (effects (font (size 1.27 1.27)) hide))
+    (property "Pins" "1=1 2=2" (at 101.60 50.80 0) (effects (font (size 1.27 1.27)) hide))
+    (property "Note" "U0TXD's series resistor (#14 A3, #11 F7): Espressif asks for 499 ohm in series with U0TXD 'to suppress harmonics' [ds logic/ESP-HARDWARE-DESIGN-GUIDELINES-ESP32S3.pdf p.16, 1.3.7 UART]. Here it is the first part on IO43 after the ribbon, at J-MCU pin 22, and it also limits what a strike on HDR-SERVICE pin 1 can push into the pin. 499 ohm against a UART receiver's input is nothing at 115200 baud" (at 101.60 50.80 0) (effects (font (size 1.27 1.27)) hide))
+    (property "Pins_source" "a two-terminal resistor" (at 101.60 50.80 0) (effects (font (size 1.27 1.27)) hide))
+    (property "Manufacturer" "UNI-ROYAL(Uniroyal Elec)" (at 101.60 50.80 0) (effects (font (size 1.27 1.27)) hide))
+    (property "MPN" "0805W8F4990T5E" (at 101.60 50.80 0) (effects (font (size 1.27 1.27)) hide))
+    (property "LCSC" "C17722" (at 101.60 50.80 0) (effects (font (size 1.27 1.27)) hide))
+    (property "Assembly" "machine" (at 101.60 50.80 0) (effects (font (size 1.27 1.27)) hide))
+    (pin "1")
+    (pin "2")
+    (instances (project "main-board" (path "/b12a49ac-ffa0-5078-b2ba-e15d161f1936/993f4837-2260-5646-9a14-8beddecedd97" (reference "R46") (unit 1))) (project "service-uart" (path "/cef56e05-f716-52bd-88f7-88ccc70bb739" (reference "R-TXD-SER") (unit 1))))
+  )
+  (wire (pts (xy 101.60 46.99) (xy 101.60 44.45)) (stroke (width 0) (type default)))
+  (hierarchical_label "U0TXD" (shape input) (at 101.60 44.45 90) (effects (font (size 1.27 1.27)) (justify left))
+    (property "Dir" "in" (at 101.60 44.45 0) (effects (font (size 1.27 1.27)) hide))
+    (property "From" "carrier/carrier" (at 101.60 44.45 0) (effects (font (size 1.27 1.27)) hide)))
+  (wire (pts (xy 101.60 54.61) (xy 101.60 57.15)) (stroke (width 0) (type default)))
+  (label "TXD_HDR" (at 101.60 57.15 270) (fields_autoplaced) (effects (font (size 1.27 1.27)) (justify right bottom)))
+  (symbol (lib_id "Device:C") (at 127.00 50.80 0) (unit 1)
+    (in_bom yes) (on_board yes) (dnp no)
+    (property "Reference" "C-EN" (at 129.54 49.53 0) (effects (font (size 1.27 1.27)) (justify left)))
+    (property "Value" "1uF" (at 129.54 52.07 0) (effects (font (size 1.27 1.27)) (justify left)))
+    (property "Footprint" "Capacitor_SMD:C_0805_2012Metric" (at 127.00 50.80 0) (effects (font (size 1.27 1.27)) hide))
+    (property "Datasheet" "" (at 127.00 50.80 0) (effects (font (size 1.27 1.27)) hide))
+    (property "Row" "C-EN" (at 127.00 50.80 0) (effects (font (size 1.27 1.27)) hide))
+    (property "Pins" "1=1 2=2" (at 127.00 50.80 0) (effects (font (size 1.27 1.27)) hide))
+    (property "Note" "EN's (CHIP_PU's) delay capacitor (#14 A2, #11 F7): Espressif advises 'an RC delay circuit at the CHIP_PU pin ... usually R = 10 kohm and C = 1 uF' [ds logic/ESP-HARDWARE-DESIGN-GUIDELINES-ESP32S3.pdf p.11]. The Matrix fits the R (R8, 10k to its 3V3) and no C, and EN runs down the ribbon and across this board to HDR-SERVICE. 1 uF against R8 is 10 ms, past the 50 us t_STBL [ds ESP32-S3-datasheet-v2.2.pdf Table 2-13]. At J-MCU pin 24, returned to J-MCU's grounds. Key1, a jumper or an adapter's open-collector reset still pulls it low at once" (at 127.00 50.80 0) (effects (font (size 1.27 1.27)) hide))
+    (property "Pins_source" "a two-terminal capacitor" (at 127.00 50.80 0) (effects (font (size 1.27 1.27)) hide))
+    (property "Manufacturer" "Samsung Electro-Mechanics" (at 127.00 50.80 0) (effects (font (size 1.27 1.27)) hide))
+    (property "MPN" "CL21B105KBFNNNE" (at 127.00 50.80 0) (effects (font (size 1.27 1.27)) hide))
+    (property "LCSC" "C28323" (at 127.00 50.80 0) (effects (font (size 1.27 1.27)) hide))
+    (property "Assembly" "machine" (at 127.00 50.80 0) (effects (font (size 1.27 1.27)) hide))
+    (pin "1")
+    (pin "2")
+    (instances (project "main-board" (path "/b12a49ac-ffa0-5078-b2ba-e15d161f1936/993f4837-2260-5646-9a14-8beddecedd97" (reference "C41") (unit 1))) (project "service-uart" (path "/cef56e05-f716-52bd-88f7-88ccc70bb739" (reference "C-EN") (unit 1))))
+  )
+  (wire (pts (xy 127.00 46.99) (xy 127.00 44.45)) (stroke (width 0) (type default)))
+  (hierarchical_label "EN" (shape input) (at 127.00 44.45 90) (effects (font (size 1.27 1.27)) (justify left))
+    (property "Dir" "in" (at 127.00 44.45 0) (effects (font (size 1.27 1.27)) hide))
+    (property "From" "carrier/carrier" (at 127.00 44.45 0) (effects (font (size 1.27 1.27)) hide)))
+  (wire (pts (xy 127.00 54.61) (xy 127.00 57.15)) (stroke (width 0) (type default)))
+  (hierarchical_label "PWR_GND" (shape passive) (at 127.00 57.15 270) (effects (font (size 1.27 1.27)) (justify right))
+    (property "Dir" "ref" (at 127.00 57.15 0) (effects (font (size 1.27 1.27)) hide))
+    (property "From" "module/power-entry" (at 127.00 57.15 0) (effects (font (size 1.27 1.27)) hide))
+    (property "Figure" "dig-gnd-topology" (at 127.00 57.15 0) (effects (font (size 1.27 1.27)) hide)))
   (sheet_instances (path "/" (page "1")))
 )
