File: hardware/carrier/service-uart/service-uart.kicad_sch (KiCad schematic)
At the start: 3 parts

Commit message: WIP #23: Matrix carrier (option c) in progress - RH key board back to its original outline, EN/IO0 removed, HDR-SERVICE 1x3, carrier sheet and CAD, J-MCU at y 14.9
Checkpoint committed by the coordinator to protect uncommitted work.

Gate-Red: carrier and RH board mid-layout, CAD outputs and sims not rebuilt

Co-Authored-By: Claude Opus 5.5 <noreply@anthropic.com>
Claude-Session: https://claude.ai/code/session_01LmB4muFXnoLprWX4JzuJ5A
Parts:
- removed C-EN: 1uF, Capacitor_SMD:C_0805_2012Metric, symbol Device:C
- HDR-SERVICE: value 1x5 -> 1x3; footprint Connector_PinHeader_2.54mm:PinHeader_1x05_P2.54mm_Vertical -> Connector_PinHeader_2.54mm:PinHeader_1x03_P2.54mm_Vertical; symbol Connector_Generic:Conn_01x05 -> Connector_Generic:Conn_01x03; LCSC C32713271 -> C32713269; MPN HX PZ2.54-1x5P ZZ -> HX PZ2.54-1x3P ZZ; Note FIVE PINS (ADR 0018): 1 TXD, 2 RXD, 3 GND, 4 EN, 5 IO0 - th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 -> THREE PINS: 1 TXD, 2 RXD, 3 GND - the UART and its ground. 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; Pins 1=1 2=2 3=3 4=4 5=5 -> 1=1 2=2 3=3
Connections:
- removed net EN: HDR-SERVICE.4 (Pin_4)
- removed net IO0: HDR-SERVICE.5 (Pin_5)
Other:
- note added: "FROM THE HAND-WRITTEN NETLIST THIS SHEET REPLACES (verbatim; the part notes are on each part's Note field): AUTHORITATIVE for connectivity. This circuit is one header, the conductors to it and R-TXD-SER in TXD (Espressif's guidelines, #14 A3); EN and IO0 left it 2026-10-03 (program over USB only), and the drawing in the page is a REPRESENTATION of this file. Whatever is plugged into the service h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"
- note removed: "FROM THE HAND-WRITTEN NETLIST THIS SHEET REPLACES (verbatim; the part notes are on each part's Note field): AUTHORITATIVE for connectivity. This circuit is one header, the conductors to it, R-TXD-SER in TXD and C-EN on EN (Espressif's guidelines, #14 A2/A3), and the drawing in the page is a REPRESENTATION of this file. Whatever is plugged into the service header is not part of the instrument, so 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"
Changed lines of the file:
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@@
     (comment 4 "Ports are hierarchical labels (Dir, From/To, Figure); the main board places this sheet")
   )
-  (symbol (lib_id "Connector_Generic:Conn_01x05") (at 40.64 50.8 0) (unit 1)
+  (symbol (lib_id "Connector_Generic:Conn_01x03") (at 40.64 48.26 0) (unit 1)
     (in_bom yes) (on_board yes) (dnp no)
     (property "Reference" "HDR-SERVICE" (at 40.64 43.18 0) (effects (font (size 1.27 1.27))))
-    (property "Value" "1x5" (at 40.64 58.42 0) (effects (font (size 1.27 1.27))))
-    (property "Footprint" "Connector_PinHeader_2.54mm:PinHeader_1x05_P2.54mm_Vertical" (at 40.64 50.8 0) (effects (font (size 1.27 1.27)) hide))
-    (property "Datasheet" "" (at 40.64 50.8 0) (effects (font (size 1.27 1.27)) hide))
-    (property "Row" "HDR-SERVICE" (at 40.64 50.8 0) (effects (font (size 1.27 1.27)) hide))
-    (property "Pins" "1=1 2=2 3=3 4=4 5=5" (at 40.64 50.8 0) (effects (font (size 1.27 1.27)) hide))
-    (property "Note" "FIVE PINS (ADR 0018): 1 TXD, 2 RXD, 3 GND, 4 EN, 5 IO0 - the ground between the UART pair and the control pair. EN and IO0 are pulled up on the Matrix; drive them to ground only" (at 40.64 50.8 0) (effects (font (size 1.27 1.27)) hide))
-    (property "Pins_source" "pin n is header position n (service-uart.md)" (at 40.64 50.8 0) (effects (font (size 1.27 1.27)) hide))
-    (property "Manufacturer" "hanxia" (at 40.64 50.8 0) (effects (font (size 1.27 1.27)) hide))
-    (property "MPN" "HX PZ2.54-1x5P ZZ" (at 40.64 50.8 0) (effects (font (size 1.27 1.27)) hide))
-    (property "LCSC" "C32713271" (at 40.64 50.8 0) (effects (font (size 1.27 1.27)) hide))
-    (property "Assembly" "hand" (at 40.64 50.8 0) (effects (font (size 1.27 1.27)) hide))
+    (property "Value" "1x3" (at 40.64 53.34 0) (effects (font (size 1.27 1.27))))
+    (property "Footprint" "Connector_PinHeader_2.54mm:PinHeader_1x03_P2.54mm_Vertical" (at 40.64 48.26 0) (effects (font (size 1.27 1.27)) hide))
+    (property "Datasheet" "" (at 40.64 48.26 0) (effects (font (size 1.27 1.27)) hide))
+    (property "Row" "HDR-SERVICE" (at 40.64 48.26 0) (effects (font (size 1.27 1.27)) hide))
+    (property "Pins" "1=1 2=2 3=3" (at 40.64 48.26 0) (effects (font (size 1.27 1.27)) hide))
+    (property "Note" "THREE PINS: 1 TXD, 2 RXD, 3 GND - the UART and its ground. EN and IO0 were pins 4 and 5 until the owner chose to program and recover the Matrix over its own USB-C only (2026-10-03, ADR 0021 amendment 2026-10-03): its BOOT and RESET buttons do both with the lid off" (at 40.64 48.26 0) (effects (font (size 1.27 1.27)) hide))
+    (property "Pins_source" "pin n is header position n (service-uart.md)" (at 40.64 48.26 0) (effects (font (size 1.27 1.27)) hide))
+    (property "Manufacturer" "hanxia" (at 40.64 48.26 0) (effects (font (size 1.27 1.27)) hide))
+    (property "MPN" "HX PZ2.54-1x3P ZZ" (at 40.64 48.26 0) (effects (font (size 1.27 1.27)) hide))
+    (property "LCSC" "C32713269" (at 40.64 48.26 0) (effects (font (size 1.27 1.27)) hide))
+    (property "Assembly" "hand" (at 40.64 48.26 0) (effects (font (size 1.27 1.27)) hide))
     (pin "1")
     (pin "2")
     (pin "3")
-    (pin "4")
-    (pin "5")
     (instances (project "main-board" (path "/b12a49ac-ffa0-5078-b2ba-e15d161f1936/993f4837-2260-5646-9a14-8beddecedd97" (reference "J2") (unit 1))) (project "service-uart" (path "/cef56e05-f716-52bd-88f7-88ccc70bb739" (reference "HDR-SERVICE") (unit 1))))
   )
@@
     (property "From" "module/power-entry" (at 33.02 50.8 0) (effects (font (size 1.27 1.27)) hide))
     (property "Figure" "dig-gnd-topology" (at 33.02 50.8 0) (effects (font (size 1.27 1.27)) hide)))
-  (wire (pts (xy 35.56 53.34) (xy 33.02 53.34)) (stroke (width 0) (type default)))
-  (hierarchical_label "EN" (shape input) (at 33.02 53.34 180) (effects (font (size 1.27 1.27)) (justify right))
-    (property "Dir" "in" (at 33.02 53.34 0) (effects (font (size 1.27 1.27)) hide))
-    (property "From" "carrier/carrier" (at 33.02 53.34 0) (effects (font (size 1.27 1.27)) hide)))
-  (wire (pts (xy 35.56 55.88) (xy 33.02 55.88)) (stroke (width 0) (type default)))
-  (hierarchical_label "IO0" (shape input) (at 33.02 55.88 180) (effects (font (size 1.27 1.27)) (justify right))
-    (property "Dir" "in" (at 33.02 55.88 0) (effects (font (size 1.27 1.27)) hide))
-    (property "From" "carrier/carrier" (at 33.02 55.88 0) (effects (font (size 1.27 1.27)) hide)))
-  (text "FROM THE HAND-WRITTEN NETLIST THIS SHEET REPLACES (verbatim; the part notes are on each part's Note field):\n\nAUTHORITATIVE for connectivity. This circuit is one header, the conductors to it, R-TXD-SER in TXD and C-EN on\nEN (Espressif's guidelines, #14 A2/A3), and the drawing in the page is a REPRESENTATION of this file. Whatever is plugged into the service header is not part of the\ninstrument, so hardware/nets.yaml marks that end with `external_driver:` rather than inventing a driver or\ncalling the net undriven." (at 205.74 38.099999999999994 0) (effects (font (size 1.27 1.27)) (justify left top)))
+  (text "FROM THE HAND-WRITTEN NETLIST THIS SHEET REPLACES (verbatim; the part notes are on each part's Note field):\n\nAUTHORITATIVE for connectivity. This circuit is one header, the conductors to it and R-TXD-SER in TXD (Espressif's guidelines, #14 A3);\nEN and IO0 left it 2026-10-03 (program over USB only), and the drawing in the page is a REPRESENTATION of this file. Whatever is plugged into the service header is not part of the\ninstrument, so hardware/nets.yaml marks that end with `external_driver:` rather than inventing a driver or\ncalling the net undriven." (at 205.74 38.099999999999994 0) (effects (font (size 1.27 1.27)) (justify left top)))
   (symbol (lib_id "Device:R") (at 101.60 50.80 0) (unit 1)
     (in_bom yes) (on_board yes) (dnp no)
@@
   (wire (pts (xy 101.60 54.61) (xy 101.60 57.15)) (stroke (width 0) (type default)))
   (label "TXD_HDR" (at 101.60 57.15 270) (fields_autoplaced) (effects (font (size 1.27 1.27)) (justify right bottom)))
-  (symbol (lib_id "Device:C") (at 127.00 50.80 0) (unit 1)
-    (in_bom yes) (on_board yes) (dnp no)
-    (property "Reference" "C-EN" (at 129.54 49.53 0) (effects (font (size 1.27 1.27)) (justify left)))
-    (property "Value" "1uF" (at 129.54 52.07 0) (effects (font (size 1.27 1.27)) (justify left)))
-    (property "Footprint" "Capacitor_SMD:C_0805_2012Metric" (at 127.00 50.80 0) (effects (font (size 1.27 1.27)) hide))
-    (property "Datasheet" "" (at 127.00 50.80 0) (effects (font (size 1.27 1.27)) hide))
-    (property "Row" "C-EN" (at 127.00 50.80 0) (effects (font (size 1.27 1.27)) hide))
-    (property "Pins" "1=1 2=2" (at 127.00 50.80 0) (effects (font (size 1.27 1.27)) hide))
-    (property "Note" "EN's (CHIP_PU's) delay capacitor (#14 A2, #11 F7): Espressif advises 'an RC delay circuit at the CHIP_PU pin ... usually R = 10 kohm and C = 1 uF' [ds logic/ESP-HARDWARE-DESIGN-GUIDELINES-ESP32S3.pdf p.11]. The Matrix fits the R (R8, 10k to its 3V3) and no C, and EN runs down the ribbon and across this board to HDR-SERVICE. 1 uF against R8 is 10 ms, past the 50 us t_STBL [ds ESP32-S3-datasheet-v2.2.pdf Table 2-13]. At J-MCU pin 24, returned to J-MCU's grounds. Key1, a jumper or an adapter's open-collector reset still pulls it low at once" (at 127.00 50.80 0) (effects (font (size 1.27 1.27)) hide))
-    (property "Pins_source" "a two-terminal capacitor" (at 127.00 50.80 0) (effects (font (size 1.27 1.27)) hide))
-    (property "Manufacturer" "Samsung Electro-Mechanics" (at 127.00 50.80 0) (effects (font (size 1.27 1.27)) hide))
-    (property "MPN" "CL21B105KBFNNNE" (at 127.00 50.80 0) (effects (font (size 1.27 1.27)) hide))
-    (property "LCSC" "C28323" (at 127.00 50.80 0) (effects (font (size 1.27 1.27)) hide))
-    (property "Assembly" "machine" (at 127.00 50.80 0) (effects (font (size 1.27 1.27)) hide))
-    (pin "1")
-    (pin "2")
-    (instances (project "main-board" (path "/b12a49ac-ffa0-5078-b2ba-e15d161f1936/993f4837-2260-5646-9a14-8beddecedd97" (reference "C41") (unit 1))) (project "service-uart" (path "/cef56e05-f716-52bd-88f7-88ccc70bb739" (reference "C-EN") (unit 1))))
-  )
-  (wire (pts (xy 127.00 46.99) (xy 127.00 44.45)) (stroke (width 0) (type default)))
-  (hierarchical_label "EN" (shape input) (at 127.00 44.45 90) (effects (font (size 1.27 1.27)) (justify left))
-    (property "Dir" "in" (at 127.00 44.45 0) (effects (font (size 1.27 1.27)) hide))
-    (property "From" "carrier/carrier" (at 127.00 44.45 0) (effects (font (size 1.27 1.27)) hide)))
-  (wire (pts (xy 127.00 54.61) (xy 127.00 57.15)) (stroke (width 0) (type default)))
-  (hierarchical_label "PWR_GND" (shape passive) (at 127.00 57.15 270) (effects (font (size 1.27 1.27)) (justify right))
-    (property "Dir" "ref" (at 127.00 57.15 0) (effects (font (size 1.27 1.27)) hide))
-    (property "From" "module/power-entry" (at 127.00 57.15 0) (effects (font (size 1.27 1.27)) hide))
-    (property "Figure" "dig-gnd-topology" (at 127.00 57.15 0) (effects (font (size 1.27 1.27)) hide)))
   (sheet_instances (path "/" (page "1")))
 )

Commit message: #40 J2: HDR-SERVICE surface mount - hanxia HX PZ2.54-1x3P TP-YQ (C41417360); no tails, so no bottom-plate window
Owner, 2026-10-06: "I think I would prefer to have it a surface mount part if that's
easy to do".
- Part: hanxia HX PZ2.54-1x3P TP-YQ, LCSC C41417360 (47,410 at LCSC, 49,531 at JLC,
  Extended), the staggered-foot family of HDR-MATRIX's 1x10. Drawing banked
  (datasheets/connectors/HANXIA-HX-PZ2.54-1x3P-TP-YQ.pdf, fragment
  .manifest-R57-issue40-j2-smd.csv; MANIFEST.csv regenerated).
- Footprint woody:PinHeader_1x03_P2.54mm_Vertical_SMD_Hanxia_PZ2.54-TP-YQ, the drawing's
  recommended pads (1.02 x 3.20 at 6.40 outside, Type A); hardware/lib/README.md row.
- service-uart sheet J2 fields (footprint, MPN, LCSC), BOM fragment row (package SMD,
  part), bom.csv regenerated; netlists re-exported (unchanged); sheet renders redone.
  Assembly stays hand, as HDR-MATRIX's.
- Body CAD: HDR-SERVICE out of tht_tails, so its bottom-plate window (and the corner
  notch) is gone; boards.service_hdr_tail removed; boards.service_hdr_h 6.0 from the
  drawing (was 8.5 from memory). Rebuilt: drc, pcb-geometry (standoffs unchanged: only
  the window line goes), plate-bottom DXF, the fab plate-bottom DXF and PDF, the other
  cut DXFs (bytes unchanged). Not rebuilt: renders, photos, clash.
- main-board README and layout.yaml comments; J2's height entry 6.0 from the drawing.
- J7's 3D stand-in noted in hardware/lib/README.md (no SM4-TB model in KiCad 9).

Gate-Red: staleness 84 cad (the body's renders, photos and clash, fingerprint-stale after the woody_body.scad / body.yaml edit, not rebuilt by instruction; some inherited) + 1 sim (inherited module-iso coverage row); kicad check: main-board.kicad_pcb still has J2's through-hole footprint until the board half (scratch j2smd.kicad_pcb) is brought in, so its parity fails until then

Co-Authored-By: Claude Opus 5.5 <noreply@anthropic.com>
Claude-Session: https://claude.ai/code/session_01LmB4muFXnoLprWX4JzuJ5A
Parts:
- HDR-SERVICE: footprint Connector_PinHeader_2.54mm:PinHeader_1x03_P2.54mm_Vertical -> woody:PinHeader_1x03_P2.54mm_Vertical_SMD_Hanxia_PZ2.54-TP-YQ; LCSC C32713269 -> C41417360; MPN HX PZ2.54-1x3P ZZ -> HX PZ2.54-1x3P TP-YQ
Changed lines of the file:
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@@
     (property "Reference" "HDR-SERVICE" (at 40.64 43.18 0) (effects (font (size 1.27 1.27))))
     (property "Value" "1x3" (at 40.64 53.34 0) (effects (font (size 1.27 1.27))))
-    (property "Footprint" "Connector_PinHeader_2.54mm:PinHeader_1x03_P2.54mm_Vertical" (at 40.64 48.26 0) (effects (font (size 1.27 1.27)) hide))
+    (property "Footprint" "woody:PinHeader_1x03_P2.54mm_Vertical_SMD_Hanxia_PZ2.54-TP-YQ" (at 40.64 48.26 0) (effects (font (size 1.27 1.27)) hide))
     (property "Datasheet" "" (at 40.64 48.26 0) (effects (font (size 1.27 1.27)) hide))
     (property "Row" "HDR-SERVICE" (at 40.64 48.26 0) (effects (font (size 1.27 1.27)) hide))
@@
     (property "Pins_source" "pin n is header position n (service-uart.md)" (at 40.64 48.26 0) (effects (font (size 1.27 1.27)) hide))
     (property "Manufacturer" "hanxia" (at 40.64 48.26 0) (effects (font (size 1.27 1.27)) hide))
-    (property "MPN" "HX PZ2.54-1x3P ZZ" (at 40.64 48.26 0) (effects (font (size 1.27 1.27)) hide))
-    (property "LCSC" "C32713269" (at 40.64 48.26 0) (effects (font (size 1.27 1.27)) hide))
+    (property "MPN" "HX PZ2.54-1x3P TP-YQ" (at 40.64 48.26 0) (effects (font (size 1.27 1.27)) hide))
+    (property "LCSC" "C41417360" (at 40.64 48.26 0) (effects (font (size 1.27 1.27)) hide))
     (property "Assembly" "hand" (at 40.64 48.26 0) (effects (font (size 1.27 1.27)) hide))
     (pin "1")
